File: KiCad/ModeltrainWagonLight/Modelwagonlight.sch (KiCad schematic (older format))
At the start: 10 parts

Commit message: Added ModeltrainWagonLight and schematic/pcb drawn --> prototype
Parts:
- removed D5: Zener, symbol D_Zener
- removed D6, D7: LED, symbol LED
- added C2: 100nF, Capacitors_SMD:C_0805_HandSoldering, symbol C
- added C3: 2.2uF, Capacitors_SMD:C_0805_HandSoldering, symbol C
- added J1, J2: Conn_01x02, Pin_Headers:Pin_Header_Angled_1x02_Pitch1.00mm, symbol Conn_01x02
- added R3: 100R, Resistors_SMD:R_0805_HandSoldering, symbol R
- added U1: NCP1117-ADJ_SOT223, TO_SOT_Packages_SMD:SOT-223-3_TabPin2, symbol NCP1117-ADJ_SOT223
- C1: value 220nF -> 1uF; footprint (none) -> Capacitors_SMD:C_0805_HandSoldering
- D1, D2, D3, D4: footprint (none) -> Diodes_SMD:D_SOD-323
- R1: value R -> 100R; footprint (none) -> Resistors_SMD:R_0805_HandSoldering
- R2: value R -> 100K; footprint (none) -> Resistors_SMD:R_0805_HandSoldering
Connections:
- net labels removed: AC
- wire segments 23 -> 27
Other:
- note added: "05mA --> 1V/0.005 = 200 Ohm\n10mA --> 1V/0.010 = 100 Ohm\n15mA --> 1V/0.015 = 67 Ohm\n20mA --> 1V/0.020 = 50 Ohm\n(0.5mA is minimum requirement \nfor regulation)"
- note added: "100K = 1V output"
- note added: "2.2uF is recommendation from datasheet \non output capacity to prevent oscillations\n"
- note added: "Dropout Voltage @ Iload = 10 mA --> 1.22V typ\nDropout Voltage @ Iload = 200 mA --> 1.3V typ"
- note added: "The amount of Led's depends on the supplied voltage,\nnormal operation from PWM amplifier is 17V minus 2V \ndue to rectifiers is 15V. For a red led a voltage of typ 1.2V\nis required, therfore maximum of 12 led's is achievable"
- note removed: "Current drawn from track 15V 20kHz PWM"
- note removed: "If VD5 = 5V1 and VD6/7 = 1.2V (one red led)\n\nVled = 2 x 1.2V\nIled --> 1mA?\nR2 = (VD5 - VLed) / ILed = (5.1 - 2.4) / 0.001 = 2k7 Ohm\n\nVR1 = Vsup - VD5 = 15 - 5.1 = 9.9V\nID5 --> 1mA?\nIR1 = Iled + ID5\nR1 = VR1 / IR1 = 9.9 / 0.002 = 4k95 Ohm\n\nPR1 = VR1 x IR1 = 9.9 x 0.002 = 20mW --> OK\nPD5 = VD5 x ID5 = 9.9 x 0.001 = 10mW --> OK\nPR2 = VR2 x IR2 = 2.7 x 0.001 = 3mW --> OK\n"
- moved on the sheet: C1, R1, R2
Changed lines of the file:
@@
 LIBS:contrib
 LIBS:valves
+LIBS:Modelwagonlight-cache
 EELAYER 25 0
 EELAYER END
@@
 F 0 "D2" H 5100 4400 50  0000 C CNN
 F 1 "1n4148" H 5100 4200 50  0000 C CNN
-F 2 "" H 5100 4300 50  0001 C CNN
+F 2 "Diodes_SMD:D_SOD-323" H 5100 4300 50  0001 C CNN
 F 3 "" H 5100 4300 50  0001 C CNN
 	1    5100 4300
@@
 F 0 "D1" H 5100 4050 50  0000 C CNN
 F 1 "1n4148" H 5100 3850 50  0000 C CNN
-F 2 "" H 5100 3950 50  0001 C CNN
+F 2 "Diodes_SMD:D_SOD-323" H 5100 3950 50  0001 C CNN
 F 3 "" H 5100 3950 50  0001 C CNN
 	1    5100 3950
@@
 F 0 "D4" H 5100 5100 50  0000 C CNN
 F 1 "1n4148" H 5100 4900 50  0000 C CNN
-F 2 "" H 5100 5000 50  0001 C CNN
+F 2 "Diodes_SMD:D_SOD-323" H 5100 5000 50  0001 C CNN
 F 3 "" H 5100 5000 50  0001 C CNN
 	1    5100 5000
@@
 F 0 "D3" H 5100 4750 50  0000 C CNN
 F 1 "1n4148" H 5100 4550 50  0000 C CNN
-F 2 "" H 5100 4650 50  0001 C CNN
+F 2 "Diodes_SMD:D_SOD-323" H 5100 4650 50  0001 C CNN
 F 3 "" H 5100 4650 50  0001 C CNN
 	1    5100 4650
@@
 $EndComp
 $Comp
-L D_Zener D5
-U 1 1 5A9521EF
-P 6300 4250
-F 0 "D5" H 6300 4350 50  0000 C CNN
-F 1 "Zener" H 6300 4150 50  0000 C CNN
-F 2 "" H 6300 4250 50  0001 C CNN
-F 3 "" H 6300 4250 50  0001 C CNN
-	1    6300 4250
-	0    1    1    0
-$EndComp
-$Comp
 L R R1
 U 1 1 5A952272
-P 5900 3950
-F 0 "R1" V 5980 3950 50  0000 C CNN
-F 1 "R" V 5900 3950 50  0000 C CNN
-F 2 "" V 5830 3950 50  0001 C CNN
-F 3 "" H 5900 3950 50  0001 C CNN
-	1    5900 3950
+P 5600 3950
+F 0 "R1" V 5680 3950 50  0000 C CNN
+F 1 "100R" V 5600 3950 50  0000 C CNN
+F 2 "Resistors_SMD:R_0805_HandSoldering" V 5530 3950 50  0001 C CNN
+F 3 "" H 5600 3950 50  0001 C CNN
+	1    5600 3950
 	0    -1   -1   0
-$EndComp
-$Comp
-L LED D7
-U 1 1 5A9522B7
-P 7750 3950
-F 0 "D7" H 7750 4050 50  0000 C CNN
-F 1 "LED" H 7750 3850 50  0000 C CNN
-F 2 "" H 7750 3950 50  0001 C CNN
-F 3 "" H 7750 3950 50  0001 C CNN
-	1    7750 3950
-	-1   0    0    1
-$EndComp
-$Comp
-L LED D6
-U 1 1 5A9524FB
-P 7250 3950
-F 0 "D6" H 7250 4050 50  0000 C CNN
-F 1 "LED" H 7250 3850 50  0000 C CNN
-F 2 "" H 7250 3950 50  0001 C CNN
-F 3 "" H 7250 3950 50  0001 C CNN
-	1    7250 3950
-	-1   0    0    1
 $EndComp
 $Comp
 L R R2
 U 1 1 5A9526BF
-P 6750 3950
-F 0 "R2" V 6830 3950 50  0000 C CNN
-F 1 "R" V 6750 3950 50  0000 C CNN
-F 2 "" V 6680 3950 50  0001 C CNN
-F 3 "" H 6750 3950 50  0001 C CNN
-	1    6750 3950
-	0    -1   -1   0
-$EndComp
-Wire Wire Line
-	5250 3950 5750 3950
-Wire Wire Line
-	6050 3950 6600 3950
-Wire Wire Line
-	6300 3950 6300 4100
-Connection ~ 6300 3950
-Wire Wire Line
-	6900 3950 7100 3950
-Wire Wire Line
-	7400 3950 7600 3950
-Wire Wire Line
-	7900 3950 7950 3950
-Wire Wire Line
-	7950 3950 7950 4650
-Wire Wire Line
-	7950 4650 5250 4650
-Wire Wire Line
-	6300 4400 6300 4650
+P 7300 4450
+F 0 "R2" V 7380 4450 50  0000 C CNN
+F 1 "100K" V 7300 4450 50  0000 C CNN
+F 2 "Resistors_SMD:R_0805_HandSoldering" V 7230 4450 50  0001 C CNN
+F 3 "" H 7300 4450 50  0001 C CNN
+	1    7300 4450
+	-1   0    0    1
+$EndComp
+Wire Wire Line
+	5250 3950 5450 3950
+Wire Wire Line
+	5250 4650 8350 4650
 Wire Wire Line
 	5300 5000 5250 5000
@@
 Connection ~ 5300 3950
 Wire Wire Line
-	3500 3950 4950 3950
-Wire Wire Line
 	4700 3950 4700 4650
 Wire Wire Line
 	4700 4650 4950 4650
-$Comp
-L AC #PWR1
-U 1 1 5A952F27
-P 3500 3900
-F 0 "#PWR1" H 3500 3800 50  0001 C CNN
-F 1 "AC" H 3500 4150 50  0000 C CNN
-F 2 "" H 3500 3900 50  0001 C CNN
-F 3 "" H 3500 3900 50  0001 C CNN
-	1    3500 3900
-	1    0    0    -1
-$EndComp
-$Comp
-L AC #PWR2
-U 1 1 5A952FC9
-P 3500 4350
-F 0 "#PWR2" H 3500 4250 50  0001 C CNN
-F 1 "AC" H 3500 4600 50  0000 C CNN
-F 2 "" H 3500 4350 50  0001 C CNN
-F 3 "" H 3500 4350 50  0001 C CNN
-	1    3500 4350
-	-1   0    0    1
-$EndComp
 Connection ~ 4700 3950
-Text Notes 2600 4150 0    60   ~ 0
-Current drawn from track 15V 20kHz PWM
-Wire Wire Line
-	3500 3950 3500 3900
-Connection ~ 6300 4650
 Wire Wire Line
 	5250 4300 5300 4300
@@
 	5300 4300 5300 3950
 Wire Wire Line
-	3500 4300 4950 4300
-Wire Wire Line
 	4850 4300 4850 5000
 Wire Wire Line
 	4850 5000 4950 5000
-Wire Wire Line
-	3500 4300 3500 4350
 Connection ~ 4850 4300
 $Comp
 L C C1
 U 1 1 5A953B73
-P 5550 4300
-F 0 "C1" H 5575 4400 50  0000 L CNN
-F 1 "220nF" H 5575 4200 50  0000 L CNN
-F 2 "" H 5588 4150 50  0001 C CNN
-F 3 "" H 5550 4300 50  0001 C CNN
-	1    5550 4300
-	1    0    0    -1
-$EndComp
-Wire Wire Line
-	5550 4150 5550 3950
-Connection ~ 5550 3950
-Wire Wire Line
-	5550 4450 5550 4650
-Connection ~ 5550 4650
-Text Notes 4550 3700 0    60   ~ 0
-If VD5 = 5V1 and VD6/7 = 1.2V (one red led)\n\nVled = 2 x 1.2V\nIled --> 1mA?\nR2 = (VD5 - VLed) / ILed = (5.1 - 2.4) / 0.001 = 2k7 Ohm\n\nVR1 = Vsup - VD5 = 15 - 5.1 = 9.9V\nID5 --> 1mA?\nIR1 = Iled + ID5\nR1 = VR1 / IR1 = 9.9 / 0.002 = 4k95 Ohm\n\nPR1 = VR1 x IR1 = 9.9 x 0.002 = 20mW --> OK\nPD5 = VD5 x ID5 = 9.9 x 0.001 = 10mW --> OK\nPR2 = VR2 x IR2 = 2.7 x 0.001 = 3mW --> OK\n
+P 5900 4300
+F 0 "C1" H 5925 4400 50  0000 L CNN
+F 1 "1uF" H 5925 4200 50  0000 L CNN
+F 2 "Capacitors_SMD:C_0805_HandSoldering" H 5938 4150 50  0001 C CNN
+F 3 "" H 5900 4300 50  0001 C CNN
+	1    5900 4300
+	1    0    0    -1
+$EndComp
+Wire Wire Line
+	4250 3950 4950 3950
+Wire Wire Line
+	4450 4300 4950 4300
+$Comp
+L NCP1117-ADJ_SOT223 U1
+U 1 1 5AB3A09A
+P 7300 3950
+F 0 "U1" H 7150 4075 50  0000 C CNN
+F 1 "NCP1117-ADJ_SOT223" H 7300 4075 50  0000 L CNN
+F 2 "TO_SOT_Packages_SMD:SOT-223-3_TabPin2" H 7300 4150 50  0001 C CNN
+F 3 "" H 7400 3700 50  0001 C CNN
+	1    7300 3950
+	1    0    0    -1
+$EndComp
+Wire Wire Line
+	7300 4250 7300 4300
+Wire Wire Line
+	7300 4600 7300 4650
+Connection ~ 7300 4650
+$Comp
+L R R3
+U 1 1 5AB3A528
+P 8350 4250
+F 0 "R3" V 8430 4250 50  0000 C CNN
+F 1 "100R" V 8350 4250 50  0000 C CNN
+F 2 "Resistors_SMD:R_0805_HandSoldering" V 8280 4250 50  0001 C CNN
+F 3 "" H 8350 4250 50  0001 C CNN
+	1    8350 4250
+	-1   0    0    1
+$EndComp
+Wire Wire Line
+	7600 3950 8350 3950
+Wire Wire Line
+	8350 3950 8350 4100
+Text Notes 6900 4800 0    60   ~ 0
+100K = 1V output
+Text Notes 8450 4300 0    60   ~ 0
+05mA --> 1V/0.005 = 200 Ohm\n10mA --> 1V/0.010 = 100 Ohm\n15mA --> 1V/0.015 = 67 Ohm\n20mA --> 1V/0.020 = 50 Ohm\n(0.5mA is minimum requirement \nfor regulation)
+Text Notes 7100 3600 0    60   ~ 0
+Dropout Voltage @ Iload = 10   mA --> 1.22V typ\nDropout Voltage @ Iload = 200 mA --> 1.3V typ
+$Comp
+L C C2
+U 1 1 5AB3CFB6
+P 7500 4450
+F 0 "C2" H 7525 4550 50  0000 L CNN
+F 1 "100nF" H 7525 4350 50  0000 L CNN
+F 2 "Capacitors_SMD:C_0805_HandSoldering" H 7538 4300 50  0001 C CNN
+F 3 "" H 7500 4450 50  0001 C CNN
+	1    7500 4450
+	1    0    0    -1
+$EndComp
+Connection ~ 7500 4650
+Wire Wire Line
+	7300 4300 7500 4300
+Wire Wire Line
+	8350 4650 8350 4400
+Wire Wire Line
+	5900 4150 5900 3950
+Connection ~ 5900 3950
+Wire Wire Line
+	5900 4450 5900 4650
+Connection ~ 5900 4650
+$Comp
+L C C3
+U 1 1 5AB3DBE0
+P 7950 4300
+F 0 "C3" H 7975 4400 50  0000 L CNN
+F 1 "2.2uF" H 7975 4200 50  0000 L CNN
+F 2 "Capacitors_SMD:C_0805_HandSoldering" H 7988 4150 50  0001 C CNN
+F 3 "" H 7950 4300 50  0001 C CNN
+	1    7950 4300
+	1    0    0    -1
+$EndComp
+Wire Wire Line
+	7950 4150 7950 3950
+Connection ~ 7950 3950
+Wire Wire Line
+	7950 4450 7950 4650
+Connection ~ 7950 4650
+Text Notes 7950 4900 0    60   ~ 0
+2.2uF is recommendation from datasheet \non output capacity to prevent oscillations\n
+Text Notes 5850 3300 0    60   ~ 0
+The amount of Led's depends on the supplied voltage,\nnormal operation from PWM amplifier is 17V minus 2V \ndue to rectifiers is 15V. For a red led a voltage of typ 1.2V\nis required, therfore maximum of 12 led's is achievable
+Wire Wire Line
+	7500 4600 7500 4650
+$Comp
+L Conn_01x02 J1
+U 1 1 5AB3E9A3
+P 4050 3950
+F 0 "J1" H 4050 4050 50  0000 C CNN
+F 1 "Conn_01x02" H 4050 3750 50  0000 C CNN
+F 2 "Pin_Headers:Pin_Header_Angled_1x02_Pitch1.00mm" H 4050 3950 50  0001 C CNN
+F 3 "" H 4050 3950 50  0001 C CNN
+	1    4050 3950
+	-1   0    0    -1
+$EndComp
+$Comp
+L Conn_01x02 J2
+U 1 1 5AB3EB44
+P 6400 3750
+F 0 "J2" H 6400 3850 50  0000 C CNN
+F 1 "Conn_01x02" H 6400 3550 50  0000 C CNN
+F 2 "Pin_Headers:Pin_Header_Angled_1x02_Pitch1.00mm" H 6400 3750 50  0001 C CNN
+F 3 "" H 6400 3750 50  0001 C CNN
+	1    6400 3750
+	0    -1   -1   0
+$EndComp
+Wire Wire Line
+	5750 3950 6400 3950
+Wire Wire Line
+	6500 3950 7000 3950
+Wire Wire Line
+	4250 4050 4450 4050
+Wire Wire Line
+	4450 4050 4450 4300
 $EndSCHEMATC
