File: KiCad/TrackControllerClockDistrTest/ClockDistrTest.sch (KiCad schematic (older format))
At the start: 36 parts

Commit message: Updated libraries, drawing ClockDistrTest schematic and PCB
Parts:
- removed U? (x2): MAX1487E, symbol MAX1487E
- added C13, C14, C15, C16, C17: C, Capacitor_SMD:C_1206_3216Metric, symbol ClockDistrTest-rescue:C
- added D1: DIODE, Diode_THT:D_DO-15_P10.16mm_Horizontal, symbol pspice:DIODE
- added D2: LED, LED_THT:LED_D5.0mm, symbol Device:LED
- added J10, J11, J12, J8, J9: Conn_01x02_Male, Connector_PinHeader_2.54mm:PinHeader_1x02_P2.54mm_Vertical, symbol ClockDistrTest-rescue:Conn_01x02_Male
- added R10, R4, R6, R7, R9: 1K, Resistor_SMD:R_1206_3216Metric, symbol ClockDistrTest-rescue:R
- added R11: 300, Resistor_SMD:R_1206_3216Metric, symbol ClockDistrTest-rescue:R
- added R5, R8: 120E, Resistor_SMD:R_1206_3216Metric, symbol ClockDistrTest-rescue:R
- added U4, U9: MAX14783E, Package_SO:SOIC-8_3.9x4.9mm_P1.27mm, symbol Interface_UART:MAX14783E
- added U5, U6, U7, U8: MAX3284E, Package_TO_SOT_SMD:SOT-23-6, symbol Interface_UART:MAX3284E
- C1, C10, C11, C12, C2, C3, C4, C5, C6, C7, C8, C9: renamed from C?; footprint Capacitors_SMD:C_1206 -> Capacitor_SMD:C_1206_3216Metric; symbol C -> ClockDistrTest-rescue:C
- J1, J2, J3, J4, J5, J6, J7: renamed from J?; footprint (none) -> Connector_PinHeader_2.54mm:PinHeader_1x02_P2.54mm_Vertical; symbol Conn_01x02_Male -> ClockDistrTest-rescue:Conn_01x02_Male
- R1, R2, R3: renamed from R?; footprint Resistors_SMD:R_1206 -> Resistor_SMD:R_1206_3216Metric; symbol R -> ClockDistrTest-rescue:R
- U1: renamed from U?; footprint (none) -> Package_DIP:DIP-16_W7.62mm; symbol 4049 -> ClockDistrTest-rescue:4049
- U2: renamed from U?; footprint Housings_SOIC:SOIC-8_3.9x4.9mm_Pitch1.27mm -> Package_SO:SOIC-8_3.9x4.9mm_P1.27mm; symbol NB3N511 -> ClockDistrTest-rescue:NB3N511
- U3: renamed from U?; footprint TO_SOT_Packages_THT:TO-220_Vertical -> Package_TO_SOT_THT:TO-220-3_Horizontal_TabDown; symbol LM7805_TO220 -> ClockDistrTest-rescue:LM7805_TO220
- X1: renamed from X?; symbol SG-531 -> ClockDistrTest-rescue:SG-531
- Y1, Y2: renamed from Y?; footprint (none) -> Crystal:Crystal_HC49-U_Vertical; symbol Crystal -> ClockDistrTest-rescue:Crystal
Connections:
- net labels added: A, B, RS422-A, RS422-B
- wire segments 80 -> 206
Other:
- moved on the sheet: R3

Commit message: Update ClockDistrTest.sch, had symbol update?
Parts:
- added J13, J14, J15, J16, J17, J18, J19, J20, J21, J22: Conn_01x02_Male, Connector_PinHeader_2.54mm:PinHeader_1x02_P2.54mm_Vertical, symbol ClockDistrTest-rescue:Conn_01x02_Male-ClockDistrTest-rescue
- C1, C10, C11, C12, C13, C14, C15, C16, C17, C2, C3, C4, C5, C6, C7, C8, C9: symbol ClockDistrTest-rescue:C -> ClockDistrTest-rescue:C-ClockDistrTest-rescue
- J1, J10, J11, J12, J2, J3, J4, J5, J6, J7, J8, J9: symbol ClockDistrTest-rescue:Conn_01x02_Male -> ClockDistrTest-rescue:Conn_01x02_Male-ClockDistrTest-rescue
- R1, R10, R11, R2, R3, R4, R5, R6, R7, R8, R9: symbol ClockDistrTest-rescue:R -> ClockDistrTest-rescue:R-ClockDistrTest-rescue
- U1: symbol ClockDistrTest-rescue:4049 -> ClockDistrTest-rescue:4049-ClockDistrTest-rescue
- U2: symbol ClockDistrTest-rescue:NB3N511 -> ClockDistrTest-rescue:NB3N511-ClockDistrTest-rescue
- U3: symbol ClockDistrTest-rescue:LM7805_TO220 -> ClockDistrTest-rescue:LM7805_TO220-ClockDistrTest-rescue
- X1: symbol ClockDistrTest-rescue:SG-531 -> ClockDistrTest-rescue:SG-531-ClockDistrTest-rescue
- Y1, Y2: symbol ClockDistrTest-rescue:Crystal -> ClockDistrTest-rescue:Crystal-ClockDistrTest-rescue
Connections:
- net labels added: A1, A2, A3, A4, B1, B2, B3, B4
- net labels removed: A, B
- wire segments 206 -> 222
Other:
- moved on the sheet: J12, R10, R3, R4, R5, R6, R7, R8, R9, U4, U9

Commit message: intermediate update on schematic
Parts:
- removed R10, R3: 1K, Resistor_SMD:R_1206_3216Metric, symbol ClockDistrTest-rescue:R-ClockDistrTest-rescue
- added C17, C18, C21, C22, C25: 22u, Capacitor_SMD:C_1206_3216Metric, symbol ClockDistrTest-rescue:C-ClockDistrTest-rescue
- added C20, C23, C24, C26: 0.1u, Capacitor_SMD:C_1206_3216Metric, symbol ClockDistrTest-rescue:C-ClockDistrTest-rescue
- added R1, R13, R14, R18, R2, R5, R7, R8, R9: 10E, Resistor_SMD:R_1206_3216Metric, symbol ClockDistrTest-rescue:R-ClockDistrTest-rescue
- C1: value C -> 12p
- C15: value C -> 22u
- C16: value C -> 0.1u
- C19: renamed from C17; value C -> 0.1u
- C2: renamed from C13; value C -> 22u
- C3: renamed from C2; value C -> 12p
- C4: renamed from C14; value C -> 0.1u
- C6: renamed from C10; value C -> 22u
- C7: renamed from C9; value C -> 0.1u
- renumbered C6 to C10, C12 to C11, C11 to C12, C7 to C13, C8 to C14, C3 to C5, C4 to C8, C5 to C9, J15 to J10, J16 to J11, J17 to J12, J18 to J13, J8 to J14, J9 to J15, J19 to J16, J20 to J17, J21 to J18, J22 to J19, J3 to J2, J10 to J20, J11 to J21, J12 to J22, J2 to J3, J13 to J8, J14 to J9, R4 to R10, R5 to R11, R6 to R12, R7 to R15, R8 to R16, R9 to R17, R1 to R3, R2 to R4, R11 to R6
Connections:
- wire segments 222 -> 276
Other:
- moved on the sheet: C11, C12, C15, C16, C19, C2, C4, C6, C7, J2, J20, J21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

Commit message: Updated schematic
Parts:
- removed J5, J6, J7: Conn_01x02_Male, Connector_PinHeader_2.54mm:PinHeader_1x02_P2.54mm_Vertical, symbol ClockDistrTest-rescue:Conn_01x02_Male-ClockDistrTest-rescue
Connections:
- wire segments 276 -> 267
Changed lines of the file:
@@
-	0    1    1    0
-$EndComp
-$Comp
-L ClockDistrTest-rescue:Conn_01x02_Male-ClockDistrTest-rescue J5
-U 1 1 5AD684BA
-P 4500 5400
-F 0 "J5" H 4500 5500 50  0000 C CNN
-F 1 "Conn_01x02_Male" V 4350 5200 50  0000 C CNN
-F 2 "Connector_PinHeader_2.54mm:PinHeader_1x02_P2.54mm_Vertical" H 4500 5400 50  0001 C CNN
-F 3 "" H 4500 5400 50  0001 C CNN
-	1    4500 5400
 	0    1    1    0
 $EndComp
@@
 	3050 4050 4400 4050
 Wire Wire Line
-	4100 5600 4400 5600
-Wire Wire Line
 	4500 4150 4500 4050
 Connection ~ 4850 4150
-Wire Wire Line
-	4850 5600 4500 5600
 $Comp
 L ClockDistrTest-rescue:+5V-ClockDistrTest-rescue #PWR016
@@
 	1    3150 3500
 	1    0    0    -1
-$EndComp
-$Comp
-L ClockDistrTest-rescue:Conn_01x02_Male-ClockDistrTest-rescue J6
-U 1 1 5AD6C486
-P 4500 5850
-F 0 "J6" H 4500 5950 50  0000 C CNN
-F 1 "Conn_01x02_Male" V 4750 6200 50  0000 C CNN
-F 2 "Connector_PinHeader_2.54mm:PinHeader_1x02_P2.54mm_Vertical" H 4500 5850 50  0001 C CNN
-F 3 "" H 4500 5850 50  0001 C CNN
-	1    4500 5850
-	0    1    1    0
-$EndComp
-$Comp
-L ClockDistrTest-rescue:Conn_01x02_Male-ClockDistrTest-rescue J7
-U 1 1 5AD6C60A
-P 4500 6300
-F 0 "J7" H 4500 6400 50  0000 C CNN
-F 1 "Conn_01x02_Male" V 4800 6600 50  0000 C CNN
-F 2 "Connector_PinHeader_2.54mm:PinHeader_1x02_P2.54mm_Vertical" H 4500 6300 50  0001 C CNN
-F 3 "" H 4500 6300 50  0001 C CNN
-	1    4500 6300
-	0    1    1    0
 $EndComp
 $Comp
@@
 $EndComp
 Wire Wire Line
-	4100 6050 4400 6050
-Wire Wire Line
-	4100 6500 4400 6500
-Wire Wire Line
 	4100 6950 4350 6950
 Wire Wire Line
-	4850 6050 4500 6050
-Connection ~ 4850 5600
-Wire Wire Line
-	4850 6500 4500 6500
-Connection ~ 4850 6050
-Wire Wire Line
 	4850 6950 4450 6950
-Connection ~ 4850 6500
 Wire Wire Line
 	2100 900  2350 900
@@
 Wire Wire Line
 	4850 4150 4500 4150
-Wire Wire Line
-	4850 4150 4850 5600
-Wire Wire Line
-	4850 5600 4850 6050
-Wire Wire Line
-	4850 6050 4850 6500
-Wire Wire Line
-	4850 6500 4850 6950
 $Comp
 L Interface_UART:MAX14783E U4
@@
 Wire Wire Line
 	3750 3150 4200 3150
+Wire Wire Line
+	4850 4150 4850 6950
 $EndSCHEMATC

Commit message: Finalized ClockDistrTest.sch generated plot files.
Parts:
- C11, C13, C9: value C -> 0.1u
- C12, C14, C8: value C -> 22u
- C15, C2, C25: value 22u -> 0.1u
- C16, C26, C4: value 0.1u -> 22u
Changed lines of the file:
@@
 P 3550 1200
 F 0 "C13" H 3575 1300 50  0000 L CNN
-F 1 "C" H 3575 1100 50  0000 L CNN
+F 1 "0.1u" H 3575 1100 50  0000 L CNN
 F 2 "Capacitor_SMD:C_1206_3216Metric" H 3588 1050 50  0001 C CNN
 F 3 "" H 3550 1200 50  0001 C CNN
@@
 P 3850 1200
 F 0 "C14" H 3875 1300 50  0000 L CNN
-F 1 "C" H 3875 1100 50  0000 L CNN
+F 1 "22u" H 3875 1100 50  0000 L CNN
 F 2 "Capacitor_SMD:C_1206_3216Metric" H 3888 1050 50  0001 C CNN
 F 3 "" H 3850 1200 50  0001 C CNN
@@
 P 2350 1200
 F 0 "C9" H 2375 1300 50  0000 L CNN
-F 1 "C" H 2375 1100 50  0000 L CNN
+F 1 "0.1u" H 2375 1100 50  0000 L CNN
 F 2 "Capacitor_SMD:C_1206_3216Metric" H 2388 1050 50  0001 C CNN
 F 3 "" H 2350 1200 50  0001 C CNN
@@
 P 2100 1200
 F 0 "C8" H 2125 1300 50  0000 L CNN
-F 1 "C" H 2125 1100 50  0000 L CNN
+F 1 "22u" H 2125 1100 50  0000 L CNN
 F 2 "Capacitor_SMD:C_1206_3216Metric" H 2138 1050 50  0001 C CNN
 F 3 "" H 2100 1200 50  0001 C CNN
@@
 P 3350 3500
 F 0 "C12" H 3375 3600 50  0000 L CNN
-F 1 "C" H 3375 3400 50  0000 L CNN
+F 1 "22u" H 3375 3400 50  0000 L CNN
 F 2 "Capacitor_SMD:C_1206_3216Metric" H 3388 3350 50  0001 C CNN
 F 3 "" H 3350 3500 50  0001 C CNN
@@
 P 3150 3500
 F 0 "C11" H 3175 3600 50  0000 L CNN
-F 1 "C" H 3175 3400 50  0000 L CNN
+F 1 "0.1u" H 3175 3400 50  0000 L CNN
 F 2 "Capacitor_SMD:C_1206_3216Metric" H 3188 3350 50  0001 C CNN
 F 3 "" H 3150 3500 50  0001 C CNN
@@
 P 1150 5600
 F 0 "C2" H 1175 5700 50  0000 L CNN
-F 1 "22u" H 1175 5500 50  0000 L CNN
+F 1 "0.1u" H 1175 5500 50  0000 L CNN
 F 2 "Capacitor_SMD:C_1206_3216Metric" H 1188 5450 50  0001 C CNN
 F 3 "" H 1150 5600 50  0001 C CNN
@@
 P 1350 5600
 F 0 "C4" H 1375 5700 50  0000 L CNN
-F 1 "0.1u" H 1375 5500 50  0000 L CNN
+F 1 "22u" H 1375 5500 50  0000 L CNN
 F 2 "Capacitor_SMD:C_1206_3216Metric" H 1388 5450 50  0001 C CNN
 F 3 "" H 1350 5600 50  0001 C CNN
@@
 P 5700 1500
 F 0 "C15" H 5725 1600 50  0000 L CNN
-F 1 "22u" H 5725 1400 50  0000 L CNN
+F 1 "0.1u" H 5725 1400 50  0000 L CNN
 F 2 "Capacitor_SMD:C_1206_3216Metric" H 5738 1350 50  0001 C CNN
 F 3 "" H 5700 1500 50  0001 C CNN
@@
 P 5900 1500
 F 0 "C16" H 5925 1600 50  0000 L CNN
-F 1 "0.1u" H 5925 1400 50  0000 L CNN
+F 1 "22u" H 5925 1400 50  0000 L CNN
 F 2 "Capacitor_SMD:C_1206_3216Metric" H 5938 1350 50  0001 C CNN
 F 3 "" H 5900 1500 50  0001 C CNN
@@
 P 9950 1500
 F 0 "C25" H 9975 1600 50  0000 L CNN
-F 1 "22u" H 9975 1400 50  0000 L CNN
+F 1 "0.1u" H 9975 1400 50  0000 L CNN
 F 2 "Capacitor_SMD:C_1206_3216Metric" H 9988 1350 50  0001 C CNN
 F 3 "" H 9950 1500 50  0001 C CNN
@@
 P 10150 1500
 F 0 "C26" H 10175 1600 50  0000 L CNN
-F 1 "0.1u" H 10175 1400 50  0000 L CNN
+F 1 "22u" H 10175 1400 50  0000 L CNN
 F 2 "Capacitor_SMD:C_1206_3216Metric" H 10188 1350 50  0001 C CNN
 F 3 "" H 10150 1500 50  0001 C CNN
