File: KiCad/TrackAmplifier/TrackAmplifier.sch (KiCad schematic (older format))
At the start: 6 parts

Commit message: Updated Amplifier schematic (concept)
Parts:
- removed C?: 1uF, symbol C
- removed C?: 22uF, symbol CP
- removed U?: PIC16F18854-ISO, symbol PIC16F18854-ISO
- removed U?: LMD18200D, symbol LMD18200D
- added C? (x12): 22u, Capacitor_SMD:C_1206_3216Metric, symbol TrackAmplifier-rescue:C
- added C? (x12): 100n, Capacitor_SMD:C_1206_3216Metric, symbol TrackAmplifier-rescue:C
- added C?: 100u, Capacitor_THT:CP_Radial_D6.3mm_P2.50mm, symbol Device:CP
- added C?: 3000u, Capacitor_THT:CP_Radial_D6.3mm_P2.50mm, symbol Device:CP
- added C? (x2): 10n, Capacitor_SMD:C_1206_3216Metric, symbol TrackAmplifier-rescue:C
- added C? (x2): 1u, Capacitor_SMD:C_1206_3216Metric, symbol TrackAmplifier-rescue:C
- added D? (x3): 1n4148, Diode_SMD:D_1206_3216Metric, symbol Device:D
- added D? (x4): LED, LED_SMD:LED_1206_3216Metric, symbol Device:LED
- added FL? (x2): EMI_Filter_CMode, symbol Device:EMI_Filter_CommonMode
- added J?: Conn_01x06, symbol Connector_Generic:Conn_01x06
- added Q?: 2N7002, Package_TO_SOT_SMD:SOT-23, symbol Transistor_FET:2N7002
- added R? (x7): 10E, symbol Device:R
- added R? (x5): 4K7, symbol Device:R
- added R?: 10K, Resistor_SMD:R_1206_3216Metric, symbol Device:R
- added R?: 100E, symbol Device:R
- added R? (x3): 1K, Resistor_SMD:R_1206_3216Metric, symbol Device:R
- added R? (x4): 10E, Resistor_SMD:R_1206_3216Metric, symbol Device:R
- added R? (x2): 100E, Resistor_SMD:R_1206_3216Metric, symbol Device:R
- added R? (x2): 0.2E, symbol Device:R
- added R?: 3K3, Resistor_SMD:R_1206_3216Metric, symbol Device:R
- added R? (x4): 330E, Resistor_SMD:R_1206_3216Metric, symbol Device:R
- added R?: 100K, Resistor_SMD:R_1206_3216Metric, symbol Device:R
- added U? (x4): ST485EBDR, Package_SO:SOIC-8_3.9x4.9mm_P1.27mm, symbol Interface_UART:ST485EBDR
- added U?: LM78M05_TO252, Package_TO_SOT_SMD:TO-252-2, symbol Regulator_Linear:LM78M05_TO252
- added U?: LMD18200, Package_TO_SOT_THT:TO-220-11_Horizontal_TabDown_StaggeredType1_Py2.54mm, symbol Driver_Motor:LMD18200
- added U?: PIC16F18854-SO, Package_SO:SOIC-28W_7.5x17.9mm_P1.27mm, symbol MCU_Microchip_PIC16:PIC16F18854-SO
- added U? (x2): INA326, Package_SO:MSOP-8_3x3mm_P0.65mm, symbol Amplifier_Instrumentation:INA326
- C?: footprint (none) -> Capacitor_SMD:C_1206_3216Metric; symbol C -> TrackAmplifier-rescue:C
- J?: symbol DB15_Male_MountingHoles -> TrackAmplifier-rescue:DB15_Male_MountingHoles
Connections:
- net labels added: +5V, BMF, BRK, CSEN, CSEN_FLT, DIR, GNDD, ICSPCLK, ICSPDAT, ID, ID_R, OCC, OCC1, OCC2, PWM, PWM1, PWM2, PWMO1, PWMO2, RST, RX, RX_A, RX_B, Reset_A, Reset_B, SYNC, Sync_A, Sync_B, THFLG, TX, TX_A, TX_B, TX_ENA, VBUS, VPP, ~MCLR
- wire segments 14 -> 385
Other:
- note added: "377uA/A --> 4A meauring range\n5V / (377^-6 x 4) -->\n3K3"
- note added: "Default Drivers Open\nBRAKE = H\nPWM = L\nDIR = X"
- note added: "Disconnected receiver inputs\nor idle bus will have RO high.\nInvert for uController reset"
- note added: "Resistor on backplane \nwill determine ID voltage"
- note added: "~MCLR~ Vil = 0.2V Vih = 0.7V\nLVP is possible, HVP only\nwhen "RESET" transceiver \ninput A < B"
- moved on the sheet: C?, J?

Commit message: Update TrackAmplifier.sch
Parts:
- removed FL?: EMI_Filter_CMode, symbol Device:EMI_Filter_CommonMode
- added R3, R5: 10E, Resistor_SMD:R_1206_3216Metric, symbol Device:R
- FL1: renamed from FL?; footprint (none) -> Inductor_THT:Choke_EPCOS_B82722-A2302-N1-22.3x22.7mm
- J1: renamed from J?; footprint (none) -> Connector_Dsub:DSUB-15_Male_Horizontal_P2.77x2.84mm_EdgePinOffset4.94mm_Housed_MountingHolesOffset7.48mm
- J2: renamed from J?; footprint (none) -> Connector_PinHeader_2.54mm:PinHeader_1x06_P2.54mm_Vertical
- R1, R10, R11, R12, R14, R16, R17, R19, R2, R22, R4, R6, R7, R8, R9: renamed from R?; footprint (none) -> Resistor_SMD:R_1206_3216Metric
- gave numbers to parts that had none: 64
Connections:
- wire segments 385 -> 381

Commit message: Updated TrackAmplifier.sch and started layout. todo: - verify ina use - verify ref use and connections
Parts:
- added C32: 22u, Capacitor_SMD:C_1206_3216Metric, symbol TrackAmplifier-rescue:C
- added C33: 100n, Capacitor_SMD:C_1206_3216Metric, symbol TrackAmplifier-rescue:C
- added D8: LED, LED_SMD:LED_1206_3216Metric, symbol Device:LED
- added MK1: Mounting_Hole, MountingHole:MountingHole_3.7mm, symbol Mechanical:Mounting_Hole
- added R34: 10E, Resistor_SMD:R_1206_3216Metric, symbol Device:R
- added R35: 330E, Resistor_SMD:R_1206_3216Metric, symbol Device:R
- added U10: REF3025, Package_TO_SOT_SMD:SOT-23, symbol Reference_Voltage:REF3025
- C6: value 3000u -> 22u; footprint Capacitor_THT:CP_Radial_D6.3mm_P2.50mm -> Capacitor_THT:CP_Axial_L21.0mm_D8.0mm_P28.00mm_Horizontal
- J2: footprint Connector_PinHeader_2.54mm:PinHeader_1x06_P2.54mm_Vertical -> Connector_PinHeader_2.54mm:PinHeader_1x06_P2.54mm_Horizontal
- R16, R17: footprint Resistor_SMD:R_1206_3216Metric -> Resistor_THT:R_Axial_DIN0411_L9.9mm_D3.6mm_P12.70mm_Horizontal
Connections:
- net labels added: REF
- wire segments 381 -> 401
- no-connect marks 0 -> 5
Other:
- note added: "length pcb = 104.7mm\nwidth pcb = 52mm\nheart conn to far pcb edge = 35mm\n\nConnector heart distance = 75mm\nConnector plate = 39.3mm\nSpace between connector plates = 35.4mm"
- moved on the sheet: C30
