File: KiCad/TrackAmplifier/TrackAmplifier.sch (KiCad schematic (older format))
At the start: 96 parts, among them J1 DB15_Male_MountingHoles, J2 Conn_01x06, Q1 2N7002, U1 ST485EBDR, U10 REF3025, U11 LM35-LP, U2 ST485EBDR, U3 LM78M05_TO252, U4 LMD18200, U5 ST485EBDR, U6 ST485EBDR, U7 INA326, U8 INA326, U9 PIC16F18854-SO

Commit message: updated schematic
Parts:
- added C36: 220n, Capacitor_SMD:C_1206_3216Metric, symbol TrackAmplifier-rescue:C
- added D10, D9: 1n4148, Diode_SMD:D_1206_3216Metric, symbol Device:D
- added F1: Polyfuse, Fuse:Fuse_Bourns_MF-SM_7.98x5.44mm, symbol Device:Polyfuse
- added R17: 10k, Resistor_SMD:R_1206_3216Metric, symbol Device:R
- added R38: 10E, Resistor_SMD:R_1206_3216Metric, symbol Device:R
- C6: value 22u -> 470u; footprint Capacitor_THT:CP_Axial_L21.0mm_D8.0mm_P28.00mm_Horizontal -> Capacitor_THT:CP_Radial_D10.0mm_P5.00mm
- R16: value 0.02 -> 0.025
Connections:
- net labels added: Vlm
- net labels removed: Vbus_flt+
- wire segments 398 -> 410
Other:
- note added: "http://nl.farnell.com/epcos/b41858c7477m000/cap-alu-elec-aec-q200-470uf-35v/dp/2750201"
- note removed: "Package_TO_SOT_THT:TO-220-11_Horizontal_TabDown_StaggeredType1_Py2.54mm"
Changed lines of the file:
@@
 P 1850 5900
 F 0 "C6" H 1900 5800 50  0000 L CNN
-F 1 "22u" H 1600 5950 50  0000 L CNN
-F 2 "Capacitor_THT:CP_Axial_L21.0mm_D8.0mm_P28.00mm_Horizontal" H 1888 5750 50  0001 C CNN
+F 1 "470u" H 1550 5950 50  0000 L CNN
+F 2 "Capacitor_THT:CP_Radial_D10.0mm_P5.00mm" H 1888 5750 50  0001 C CNN
 F 3 "~" H 1850 5900 50  0001 C CNN
 	1    1850 5900
@@
 Wire Wire Line
 	9000 1150 9200 1150
-Text GLabel 7200 2150 0    50   Input ~ 0
+Text GLabel 7200 1750 0    50   Input ~ 0
 ID
 $Comp
@@
 	1650 750  1650 800
 Text GLabel 900  800  0    50   Input ~ 0
-Vbus_flt+
+Vbus_flt
 Text Notes 7350 6450 0    50   ~ 0
 377uA/A --> 4A meauring range\n5V / (377^-6 x 4) -->\n3K3
@@
 Wire Wire Line
 	9800 5350 10100 5350
-Text GLabel 1700 5700 0    50   Input ~ 0
+Text GLabel 950  5900 0    50   Input ~ 0
 Vbus_flt
 Wire Wire Line
-	1700 5700 1850 5700
-Connection ~ 1850 5700
-Wire Wire Line
 	9500 2150 9500 2250
 Wire Wire Line
@@
 Wire Wire Line
 	7350 2050 7200 2050
-Wire Wire Line
-	7200 2150 7350 2150
 $Comp
 L Reference_Voltage:REF3025 U10
@@
 Connection ~ 5500 1450
 Wire Wire Line
-	7350 1750 7300 1750
-Wire Wire Line
-	6750 1750 6750 1150
+	6750 1850 6750 1150
 Wire Wire Line
 	6750 1150 6650 1150
-Wire Wire Line
-	7350 1850 7300 1850
-Wire Wire Line
-	7300 1850 7300 1750
-Connection ~ 7300 1750
-Wire Wire Line
-	7300 1750 6750 1750
-Text GLabel 6700 1750 0    50   Output ~ 0
+Text GLabel 6600 1850 0    50   Output ~ 0
 VREF
 Wire Wire Line
-	6700 1750 6750 1750
-Connection ~ 6750 1750
+	6600 1850 6750 1850
 Text GLabel 5450 2350 2    50   Input ~ 0
 VREF
@@
 $EndComp
 Text GLabel 8450 4750 0    50   Output ~ 0
-Vbus_flt+
+Vbus_flt
 Text GLabel 8450 4550 0    50   Output ~ 0
 GND
@@
 	9200 6150 9200 5850
 Connection ~ 9200 5850
-Text Notes 3000 7700 0    50   ~ 0
-Package_TO_SOT_THT:TO-220-11_Horizontal_TabDown_StaggeredType1_Py2.54mm
 Wire Wire Line
 	2850 5700 2850 6200
@@
 P 4850 6750
 F 0 "R16" V 4675 6750 50  0000 C CNN
-F 1 "0.02" V 4750 6750 50  0000 C CNN
+F 1 "0.025" V 4750 6750 50  0000 C CNN
 F 2 "Resistor_SMD:R_Shunt_2512_6332Metric_0.005-0.2" V 4780 6750 50  0001 C CNN
 F 3 "~" H 4850 6750 50  0001 C CNN
@@
 Wire Wire Line
 	4950 6500 4950 6600
+$Comp
+L Device:Polyfuse F1
+U 1 1 5AF3A43B
+P 1250 5900
+F 0 "F1" V 1150 5900 50  0000 C CNN
+F 1 "Polyfuse" V 1350 5900 50  0000 C CNN
+F 2 "Fuse:Fuse_Bourns_MF-SM_7.98x5.44mm" H 1300 5700 50  0001 L CNN
+F 3 "~" H 1250 5900 50  0001 C CNN
+	1    1250 5900
+	0    1    1    0
+$EndComp
+Wire Wire Line
+	1100 5900 950  5900
+Wire Wire Line
+	1400 5900 1450 5900
+Wire Wire Line
+	1450 5900 1450 5700
+Wire Wire Line
+	1450 5700 1850 5700
+Connection ~ 1850 5700
+$Comp
+L Device:R R38
+U 1 1 5AFB301E
+P 6950 1850
+F 0 "R38" V 7030 1850 50  0000 C CNN
+F 1 "10E" V 6950 1850 50  0000 C CNN
+F 2 "Resistor_SMD:R_1206_3216Metric" V 6880 1850 50  0001 C CNN
+F 3 "~" H 6950 1850 50  0001 C CNN
+	1    6950 1850
+	0    -1   -1   0
+$EndComp
+Connection ~ 6750 1850
+Wire Wire Line
+	6750 1850 6800 1850
+Wire Wire Line
+	7100 1850 7350 1850
+Wire Wire Line
+	7200 1750 7350 1750
+Text GLabel 5900 5700 2    50   Output ~ 0
+Vlm
+$Comp
+L TrackAmplifier-rescue:C C36
+U 1 1 5B1E8513
+P 5800 5900
+F 0 "C36" H 5825 6000 50  0000 L CNN
+F 1 "220n" H 5825 5800 50  0000 L CNN
+F 2 "Capacitor_SMD:C_1206_3216Metric" H 5838 5750 50  0001 C CNN
+F 3 "" H 5800 5900 50  0001 C CNN
+	1    5800 5900
+	-1   0    0    1
+$EndComp
+$Comp
+L TrackAmplifier-rescue:GND #PWR038
+U 1 1 5B1E851A
+P 5800 6100
+F 0 "#PWR038" H 5800 5850 50  0001 C CNN
+F 1 "GND" H 5800 5950 50  0000 C CNN
+F 2 "" H 5800 6100 50  0001 C CNN
+F 3 "" H 5800 6100 50  0001 C CNN
+	1    5800 6100
+	-1   0    0    -1
+$EndComp
+$Comp
+L Device:D D9
+U 1 1 5B1E8528
+P 5300 5500
+F 0 "D9" H 5300 5600 50  0000 C CNN
+F 1 "1n4148" H 5300 5400 50  0000 C CNN
+F 2 "Diode_SMD:D_1206_3216Metric" H 5300 5500 50  0001 C CNN
+F 3 "~" H 5300 5500 50  0001 C CNN
+	1    5300 5500
+	0    1    1    0
+$EndComp
+$Comp
+L Device:D D10
+U 1 1 5B1E852F
+P 5300 5900
+F 0 "D10" H 5300 6000 50  0000 C CNN
+F 1 "1n4148" H 5300 5800 50  0000 C CNN
+F 2 "Diode_SMD:D_1206_3216Metric" H 5300 5900 50  0001 C CNN
+F 3 "~" H 5300 5900 50  0001 C CNN
+	1    5300 5900
+	0    1    1    0
+$EndComp
+$Comp
+L TrackAmplifier-rescue:GND #PWR017
+U 1 1 5B1E8536
+P 5300 6100
+F 0 "#PWR017" H 5300 5850 50  0001 C CNN
+F 1 "GND" H 5300 5950 50  0000 C CNN
+F 2 "" H 5300 6100 50  0001 C CNN
+F 3 "" H 5300 6100 50  0001 C CNN
+	1    5300 6100
+	-1   0    0    -1
+$EndComp
+$Comp
+L power:+5V #PWR010
+U 1 1 5B1E853C
+P 5300 5300
+F 0 "#PWR010" H 5300 5150 50  0001 C CNN
+F 1 "+5V" H 5300 5440 50  0000 C CNN
+F 2 "" H 5300 5300 50  0001 C CNN
+F 3 "" H 5300 5300 50  0001 C CNN
+	1    5300 5300
+	1    0    0    -1
+$EndComp
+Wire Wire Line
+	5300 5300 5300 5350
+Wire Wire Line
+	5300 5650 5300 5700
+Wire Wire Line
+	5300 6100 5300 6050
+Connection ~ 5300 5700
+Wire Wire Line
+	5300 5700 5300 5750
+Wire Wire Line
+	5800 6100 5800 6050
+$Comp
+L Device:R R17
+U 1 1 5B2136D1
+P 5000 5700
+F 0 "R17" V 5080 5700 50  0000 C CNN
+F 1 "10k" V 5000 5700 50  0000 C CNN
+F 2 "Resistor_SMD:R_1206_3216Metric" V 4930 5700 50  0001 C CNN
+F 3 "~" H 5000 5700 50  0001 C CNN
+	1    5000 5700
+	0    1    1    0
+$EndComp
+Wire Wire Line
+	2850 5700 4850 5700
+Connection ~ 2850 5700
+Wire Wire Line
+	5150 5700 5300 5700
+Wire Wire Line
+	5800 5700 5800 5750
+Wire Wire Line
+	5300 5700 5800 5700
+Wire Wire Line
+	5900 5700 5800 5700
+Connection ~ 5800 5700
+Text GLabel 7200 2150 0    50   Input ~ 0
+Vlm
+Wire Wire Line
+	7200 2150 7350 2150
+Text Notes 1200 8200 0    50   ~ 0
+http://nl.farnell.com/epcos/b41858c7477m000/cap-alu-elec-aec-q200-470uf-35v/dp/2750201
 $EndSCHEMATC

Commit message: update schematic
Parts:
- added R39: 50k, Resistor_SMD:R_1206_3216Metric, symbol Device:R
- F1: value Polyfuse -> 3.0A
- R26, R27, R28, R29, R35: footprint Resistor_SMD:R_1206_3216Metric -> Resistor_SMD:R_0603_1608Metric
Connections:
- wire segments 410 -> 413
Other:
- moved on the sheet: C36
Changed lines of the file:
@@
 U 1 1 5AF827EA
 P 1850 5900
-F 0 "C6" H 1900 5800 50  0000 L CNN
+F 0 "C6" H 1700 5800 50  0000 L CNN
 F 1 "470u" H 1550 5950 50  0000 L CNN
 F 2 "Capacitor_THT:CP_Radial_D10.0mm_P5.00mm" H 1888 5750 50  0001 C CNN
@@
 F 0 "R26" V 8750 2150 50  0000 C CNN
 F 1 "330E" V 8700 1950 50  0000 C CNN
-F 2 "Resistor_SMD:R_1206_3216Metric" V 8630 1950 50  0001 C CNN
+F 2 "Resistor_SMD:R_0603_1608Metric" V 8630 1950 50  0001 C CNN
 F 3 "~" H 8700 1950 50  0001 C CNN
 	1    8700 1950
@@
 F 0 "R27" V 8750 2250 50  0000 C CNN
 F 1 "330E" V 8700 2050 50  0000 C CNN
-F 2 "Resistor_SMD:R_1206_3216Metric" V 8630 2050 50  0001 C CNN
+F 2 "Resistor_SMD:R_0603_1608Metric" V 8630 2050 50  0001 C CNN
 F 3 "~" H 8700 2050 50  0001 C CNN
 	1    8700 2050
@@
 F 0 "R28" V 8750 2350 50  0000 C CNN
 F 1 "330E" V 8700 2150 50  0000 C CNN
-F 2 "Resistor_SMD:R_1206_3216Metric" V 8630 2150 50  0001 C CNN
+F 2 "Resistor_SMD:R_0603_1608Metric" V 8630 2150 50  0001 C CNN
 F 3 "~" H 8700 2150 50  0001 C CNN
 	1    8700 2150
@@
 F 0 "R29" V 8750 2550 50  0000 C CNN
 F 1 "330E" V 8700 2350 50  0000 C CNN
-F 2 "Resistor_SMD:R_1206_3216Metric" V 8630 2350 50  0001 C CNN
+F 2 "Resistor_SMD:R_0603_1608Metric" V 8630 2350 50  0001 C CNN
 F 3 "~" H 8700 2350 50  0001 C CNN
 	1    8700 2350
@@
 F 0 "R35" V 8650 2050 50  0000 C CNN
 F 1 "330E" V 8700 2250 50  0000 C CNN
-F 2 "Resistor_SMD:R_1206_3216Metric" V 8630 2250 50  0001 C CNN
+F 2 "Resistor_SMD:R_0603_1608Metric" V 8630 2250 50  0001 C CNN
 F 3 "~" H 8700 2250 50  0001 C CNN
 	1    8700 2250
@@
 	-1   0    0    -1
 $EndComp
+Text GLabel 8450 4550 0    50   Output ~ 0
+Vbus_flt
 Text GLabel 8450 4750 0    50   Output ~ 0
-Vbus_flt
-Text GLabel 8450 4550 0    50   Output ~ 0
 GND
 Text GLabel 900  1300 0    50   Input ~ 0
@@
 	9200 4550 9200 4650
 Connection ~ 9200 4650
-Wire Wire Line
-	8450 4550 8600 4550
-Wire Wire Line
-	8600 4750 8450 4750
 $Comp
 L Device:R R36
@@
 L power:GNDD #PWR0104
 U 1 1 5AF2B1F8
-P 9200 6150
-F 0 "#PWR0104" H 9200 5900 50  0001 C CNN
-F 1 "GNDD" H 9200 6025 50  0000 C CNN
-F 2 "" H 9200 6150 50  0001 C CNN
-F 3 "" H 9200 6150 50  0001 C CNN
-	1    9200 6150
-	1    0    0    -1
-$EndComp
-Wire Wire Line
-	9200 6150 9200 5850
-Connection ~ 9200 5850
+P 9250 6150
+F 0 "#PWR0104" H 9250 5900 50  0001 C CNN
+F 1 "GNDD" H 9250 6025 50  0000 C CNN
+F 2 "" H 9250 6150 50  0001 C CNN
+F 3 "" H 9250 6150 50  0001 C CNN
+	1    9250 6150
+	1    0    0    -1
+$EndComp
 Wire Wire Line
 	2850 5700 2850 6200
@@
 P 1250 5900
 F 0 "F1" V 1150 5900 50  0000 C CNN
-F 1 "Polyfuse" V 1350 5900 50  0000 C CNN
+F 1 "3.0A" V 1350 5900 50  0000 C CNN
 F 2 "Fuse:Fuse_Bourns_MF-SM_7.98x5.44mm" H 1300 5700 50  0001 L CNN
 F 3 "~" H 1250 5900 50  0001 C CNN
@@
 Wire Wire Line
 	7200 1750 7350 1750
-Text GLabel 5900 5700 2    50   Output ~ 0
+Text GLabel 6250 5700 2    50   Output ~ 0
 Vlm
 $Comp
 L TrackAmplifier-rescue:C C36
 U 1 1 5B1E8513
-P 5800 5900
-F 0 "C36" H 5825 6000 50  0000 L CNN
-F 1 "220n" H 5825 5800 50  0000 L CNN
-F 2 "Capacitor_SMD:C_1206_3216Metric" H 5838 5750 50  0001 C CNN
-F 3 "" H 5800 5900 50  0001 C CNN
-	1    5800 5900
+P 6150 5900
+F 0 "C36" H 6175 6000 50  0000 L CNN
+F 1 "220n" H 6175 5800 50  0000 L CNN
+F 2 "Capacitor_SMD:C_1206_3216Metric" H 6188 5750 50  0001 C CNN
+F 3 "" H 6150 5900 50  0001 C CNN
+	1    6150 5900
 	-1   0    0    1
 $EndComp
@@
 L TrackAmplifier-rescue:GND #PWR038
 U 1 1 5B1E851A
-P 5800 6100
-F 0 "#PWR038" H 5800 5850 50  0001 C CNN
-F 1 "GND" H 5800 5950 50  0000 C CNN
-F 2 "" H 5800 6100 50  0001 C CNN
-F 3 "" H 5800 6100 50  0001 C CNN
-	1    5800 6100
+P 6150 6100
+F 0 "#PWR038" H 6150 5850 50  0001 C CNN
+F 1 "GND" H 6150 5950 50  0000 C CNN
+F 2 "" H 6150 6100 50  0001 C CNN
+F 3 "" H 6150 6100 50  0001 C CNN
+	1    6150 6100
 	-1   0    0    -1
 $EndComp
@@
 L Device:D D9
 U 1 1 5B1E8528
-P 5300 5500
-F 0 "D9" H 5300 5600 50  0000 C CNN
-F 1 "1n4148" H 5300 5400 50  0000 C CNN
-F 2 "Diode_SMD:D_1206_3216Metric" H 5300 5500 50  0001 C CNN
-F 3 "~" H 5300 5500 50  0001 C CNN
-	1    5300 5500
+P 5650 5500
+F 0 "D9" H 5650 5600 50  0000 C CNN
+F 1 "1n4148" H 5650 5400 50  0000 C CNN
+F 2 "Diode_SMD:D_1206_3216Metric" H 5650 5500 50  0001 C CNN
+F 3 "~" H 5650 5500 50  0001 C CNN
+	1    5650 5500
 	0    1    1    0
 $EndComp
@@
 L Device:D D10
 U 1 1 5B1E852F
-P 5300 5900
-F 0 "D10" H 5300 6000 50  0000 C CNN
-F 1 "1n4148" H 5300 5800 50  0000 C CNN
-F 2 "Diode_SMD:D_1206_3216Metric" H 5300 5900 50  0001 C CNN
-F 3 "~" H 5300 5900 50  0001 C CNN
-	1    5300 5900
+P 5650 5900
+F 0 "D10" H 5650 6000 50  0000 C CNN
+F 1 "1n4148" H 5650 5800 50  0000 C CNN
+F 2 "Diode_SMD:D_1206_3216Metric" H 5650 5900 50  0001 C CNN
+F 3 "~" H 5650 5900 50  0001 C CNN
+	1    5650 5900
 	0    1    1    0
 $EndComp
@@
 L TrackAmplifier-rescue:GND #PWR017
 U 1 1 5B1E8536
-P 5300 6100
-F 0 "#PWR017" H 5300 5850 50  0001 C CNN
-F 1 "GND" H 5300 5950 50  0000 C CNN
-F 2 "" H 5300 6100 50  0001 C CNN
-F 3 "" H 5300 6100 50  0001 C CNN
-	1    5300 6100
+P 5650 6100
+F 0 "#PWR017" H 5650 5850 50  0001 C CNN
+F 1 "GND" H 5650 5950 50  0000 C CNN
+F 2 "" H 5650 6100 50  0001 C CNN
+F 3 "" H 5650 6100 50  0001 C CNN
+	1    5650 6100
 	-1   0    0    -1
 $EndComp
@@
 L power:+5V #PWR010
 U 1 1 5B1E853C
-P 5300 5300
-F 0 "#PWR010" H 5300 5150 50  0001 C CNN
-F 1 "+5V" H 5300 5440 50  0000 C CNN
-F 2 "" H 5300 5300 50  0001 C CNN
-F 3 "" H 5300 5300 50  0001 C CNN
-	1    5300 5300
-	1    0    0    -1
-$EndComp
-Wire Wire Line
-	5300 5300 5300 5350
-Wire Wire Line
-	5300 5650 5300 5700
-Wire Wire Line
-	5300 6100 5300 6050
-Connection ~ 5300 5700
-Wire Wire Line
-	5300 5700 5300 5750
-Wire Wire Line
-	5800 6100 5800 6050
+P 5650 5300
+F 0 "#PWR010" H 5650 5150 50  0001 C CNN
+F 1 "+5V" H 5650 5440 50  0000 C CNN
+F 2 "" H 5650 5300 50  0001 C CNN
+F 3 "" H 5650 5300 50  0001 C CNN
+	1    5650 5300
+	1    0    0    -1
+$EndComp
+Wire Wire Line
+	5650 5300 5650 5350
+Wire Wire Line
+	5650 5650 5650 5700
+Wire Wire Line
+	5650 6100 5650 6050
+Connection ~ 5650 5700
+Wire Wire Line
+	5650 5700 5650 5750
+Wire Wire Line
+	6150 6100 6150 6050
 $Comp
 L Device:R R17
@@
 Connection ~ 2850 5700
 Wire Wire Line
-	5150 5700 5300 5700
-Wire Wire Line
-	5800 5700 5800 5750
-Wire Wire Line
-	5300 5700 5800 5700
-Wire Wire Line
-	5900 5700 5800 5700
-Connection ~ 5800 5700
+	6150 5700 6150 5750
+Wire Wire Line
+	5650 5700 6150 5700
+Wire Wire Line
+	6250 5700 6150 5700
+Connection ~ 6150 5700
 Text GLabel 7200 2150 0    50   Input ~ 0
 Vlm
@@
 Text Notes 1200 8200 0    50   ~ 0
 http://nl.farnell.com/epcos/b41858c7477m000/cap-alu-elec-aec-q200-470uf-35v/dp/2750201
+$Comp
+L Device:R R39
+U 1 1 5AF71650
+P 5250 5900
+F 0 "R39" V 5330 5900 50  0000 C CNN
+F 1 "50k" V 5250 5900 50  0000 C CNN
+F 2 "Resistor_SMD:R_1206_3216Metric" V 5180 5900 50  0001 C CNN
+F 3 "~" H 5250 5900 50  0001 C CNN
+	1    5250 5900
+	-1   0    0    1
+$EndComp
+$Comp
+L TrackAmplifier-rescue:GND #PWR048
+U 1 1 5AF7179B
+P 5250 6100
+F 0 "#PWR048" H 5250 5850 50  0001 C CNN
+F 1 "GND" H 5250 5950 50  0000 C CNN
+F 2 "" H 5250 6100 50  0001 C CNN
+F 3 "" H 5250 6100 50  0001 C CNN
+	1    5250 6100
+	-1   0    0    -1
+$EndComp
+Wire Wire Line
+	5150 5700 5250 5700
+Wire Wire Line
+	5250 5750 5250 5700
+Connection ~ 5250 5700
+Wire Wire Line
+	5250 5700 5650 5700
+Wire Wire Line
+	5250 6050 5250 6100
+Wire Wire Line
+	9250 6150 9250 5950
+Connection ~ 9250 5950
+Wire Wire Line
+	8450 4550 8600 4550
+Wire Wire Line
+	8450 4750 8600 4750
 $EndSCHEMATC

Commit message: updated PCB
Parts:
- C30: value 22u -> 220n
- R26, R27, R28, R29, R35: footprint Resistor_SMD:R_0603_1608Metric -> Resistor_SMD:R_1206_3216Metric
Changed lines of the file:
@@
 P 9700 1350
 F 0 "C30" H 9725 1450 50  0000 L CNN
-F 1 "22u" H 9725 1250 50  0000 L CNN
+F 1 "220n" H 9800 1350 50  0000 L CNN
 F 2 "Capacitor_SMD:C_1206_3216Metric" H 9738 1200 50  0001 C CNN
 F 3 "" H 9700 1350 50  0001 C CNN
@@
 F 0 "R26" V 8750 2150 50  0000 C CNN
 F 1 "330E" V 8700 1950 50  0000 C CNN
-F 2 "Resistor_SMD:R_0603_1608Metric" V 8630 1950 50  0001 C CNN
+F 2 "Resistor_SMD:R_1206_3216Metric" V 8630 1950 50  0001 C CNN
 F 3 "~" H 8700 1950 50  0001 C CNN
 	1    8700 1950
@@
 F 0 "R27" V 8750 2250 50  0000 C CNN
 F 1 "330E" V 8700 2050 50  0000 C CNN
-F 2 "Resistor_SMD:R_0603_1608Metric" V 8630 2050 50  0001 C CNN
+F 2 "Resistor_SMD:R_1206_3216Metric" V 8630 2050 50  0001 C CNN
 F 3 "~" H 8700 2050 50  0001 C CNN
 	1    8700 2050
@@
 F 0 "R28" V 8750 2350 50  0000 C CNN
 F 1 "330E" V 8700 2150 50  0000 C CNN
-F 2 "Resistor_SMD:R_0603_1608Metric" V 8630 2150 50  0001 C CNN
+F 2 "Resistor_SMD:R_1206_3216Metric" V 8630 2150 50  0001 C CNN
 F 3 "~" H 8700 2150 50  0001 C CNN
 	1    8700 2150
@@
 F 0 "R29" V 8750 2550 50  0000 C CNN
 F 1 "330E" V 8700 2350 50  0000 C CNN
-F 2 "Resistor_SMD:R_0603_1608Metric" V 8630 2350 50  0001 C CNN
+F 2 "Resistor_SMD:R_1206_3216Metric" V 8630 2350 50  0001 C CNN
 F 3 "~" H 8700 2350 50  0001 C CNN
 	1    8700 2350
@@
 F 0 "R35" V 8650 2050 50  0000 C CNN
 F 1 "330E" V 8700 2250 50  0000 C CNN
-F 2 "Resistor_SMD:R_0603_1608Metric" V 8630 2250 50  0001 C CNN
+F 2 "Resistor_SMD:R_1206_3216Metric" V 8630 2250 50  0001 C CNN
 F 3 "~" H 8700 2250 50  0001 C CNN
 	1    8700 2250
