File: KiCad/TrackAmplifier/TrackAmplifier.sch (KiCad schematic (older format))
At the start: 103 parts, among them J1 DB15_Male_MountingHoles, J2 Conn_01x06, Q1 2N7002, U1 ST485EBDR, U10 REF3025, U11 LM35-LP, U2 ST485EBDR, U3 LM78M05_TO252, U4 LMD18200, U5 ST485EBDR, U6 ST485EBDR, U7 INA326, U8 INA326, U9 PIC16F18854-SO

Commit message: TrackAmplifier.kicad_pcb finished To do: - Check and fit test
Parts:
- added C37: 100n, Capacitor_SMD:C_1206_3216Metric, symbol TrackAmplifier-rescue:C
- added R40: 4k7, Resistor_SMD:R_1206_3216Metric, symbol Device:R
- R30: value 1K -> 10k
Connections:
- net labels added: THFLG
- wire segments 413 -> 421
- no-connect marks 6 -> 4
Other:
- note added: "Disconnected receiver inputs\nor idle bus will have RO high.\nInvert for continuous uController reset"
- note removed: "Disconnected receiver inputs\nor idle bus will have RO high.\nInvert for uController reset"
- moved on the sheet: C30, Q1
Changed lines of the file:
@@
 	9250 4550 9250 4750
 Wire Wire Line
-	10100 5950 9250 5950
-Wire Wire Line
 	10100 4650 9200 4650
-Wire Wire Line
-	9200 5850 10100 5850
 $Comp
 L TrackAmplifier-rescue:C C7
@@
 Wire Wire Line
 	1850 4250 1000 4250
-Connection ~ 1000 3950
 Text GLabel 1400 3600 0    50   Input ~ 0
 Sync_B
@@
 Text GLabel 9800 5250 0    50   Output ~ 0
 RX_A
+Text GLabel 9800 5550 0    50   Input ~ 0
+TX_B
 Text GLabel 9800 5450 0    50   Input ~ 0
-TX_B
-Text GLabel 9800 5550 0    50   Input ~ 0
 TX_A
 $Comp
@@
 Text GLabel 5800 6950 2    50   Output ~ 0
 PWMO2
-Text GLabel 9800 5650 0    50   Input ~ 0
+Text GLabel 9800 5850 0    50   Input ~ 0
 PWMO1
-Text GLabel 9800 5750 0    50   Input ~ 0
+Text GLabel 9800 5950 0    50   Input ~ 0
 PWMO2
-Wire Wire Line
-	9800 5750 10100 5750
 Wire Wire Line
 	4050 3200 4050 3250
@@
 Text GLabel 2350 3600 2    50   Output ~ 0
 SYNC
-Text GLabel 3100 2000 2    50   Input ~ 0
+Text GLabel 3500 2000 2    50   Input ~ 0
 RST
 Wire Wire Line
@@
 Text GLabel 8500 2650 2    50   Input ~ 0
 TEMP
+Text GLabel 8500 2950 2    50   Output ~ 0
+PWM
 Text GLabel 8500 2750 2    50   Output ~ 0
-PWM
-Text GLabel 8500 2950 2    50   Output ~ 0
 DIR
 Text GLabel 8500 2850 2    50   Output ~ 0
@@
 L Transistor_FET:2N7002 Q1
 U 1 1 5B357979
-P 2900 2300
-F 0 "Q1" H 3100 2375 50  0000 L CNN
-F 1 "2N7002" H 3100 2300 50  0000 L CNN
-F 2 "Package_TO_SOT_SMD:SOT-23" H 3100 2225 50  0001 L CIN
-F 3 "https://www.fairchildsemi.com/datasheets/2N/2N7002.pdf" H 2900 2300 50  0001 L CNN
-	1    2900 2300
+P 3300 2300
+F 0 "Q1" H 3500 2375 50  0000 L CNN
+F 1 "2N7002" H 3500 2300 50  0000 L CNN
+F 2 "Package_TO_SOT_SMD:SOT-23" H 3500 2225 50  0001 L CIN
+F 3 "https://www.fairchildsemi.com/datasheets/2N/2N7002.pdf" H 3300 2300 50  0001 L CNN
+	1    3300 2300
 	1    0    0    -1
 $EndComp
@@
 L TrackAmplifier-rescue:GND #PWR012
 U 1 1 5B3BB8BC
-P 3000 2600
-F 0 "#PWR012" H 3000 2350 50  0001 C CNN
-F 1 "GND" H 3000 2450 50  0000 C CNN
-F 2 "" H 3000 2600 50  0001 C CNN
-F 3 "" H 3000 2600 50  0001 C CNN
-	1    3000 2600
-	-1   0    0    -1
-$EndComp
-Wire Wire Line
-	3000 2600 3000 2500
-Wire Wire Line
-	3100 2000 3000 2000
-Wire Wire Line
-	3000 2000 3000 2100
+P 3400 2600
+F 0 "#PWR012" H 3400 2350 50  0001 C CNN
+F 1 "GND" H 3400 2450 50  0000 C CNN
+F 2 "" H 3400 2600 50  0001 C CNN
+F 3 "" H 3400 2600 50  0001 C CNN
+	1    3400 2600
+	-1   0    0    -1
+$EndComp
+Wire Wire Line
+	3400 2600 3400 2500
+Wire Wire Line
+	3500 2000 3400 2000
+Wire Wire Line
+	3400 2000 3400 2100
 $Comp
 L Device:D D7
@@
 ~MCLR~ Vil = 0.2V Vih = 0.7V\nLVP is possible, HVP only\nwhen "RESET" transceiver \ninput A < B
 Text Notes 2150 1900 0    50   ~ 0
-Disconnected receiver inputs\nor idle bus will have RO high.\nInvert for uController reset
-Wire Wire Line
-	9800 5650 10100 5650
+Disconnected receiver inputs\nor idle bus will have RO high.\nInvert for continuous uController reset
 Wire Wire Line
 	9800 4750 10100 4750
-Wire Wire Line
-	10100 5450 9800 5450
-Wire Wire Line
-	9800 5550 10100 5550
 $Comp
 L power:GNDD #PWR046
@@
 L TrackAmplifier-rescue:C C30
 U 1 1 5B65E3B2
-P 9700 1350
-F 0 "C30" H 9725 1450 50  0000 L CNN
-F 1 "220n" H 9800 1350 50  0000 L CNN
-F 2 "Capacitor_SMD:C_1206_3216Metric" H 9738 1200 50  0001 C CNN
-F 3 "" H 9700 1350 50  0001 C CNN
-	1    9700 1350
+P 9500 1350
+F 0 "C30" H 9525 1450 50  0000 L CNN
+F 1 "220n" H 9550 1250 50  0000 L CNN
+F 2 "Capacitor_SMD:C_1206_3216Metric" H 9538 1200 50  0001 C CNN
+F 3 "" H 9500 1350 50  0001 C CNN
+	1    9500 1350
 	-1   0    0    1
 $EndComp
@@
 L TrackAmplifier-rescue:GND #PWR040
 U 1 1 5B66EA4C
-P 9700 1550
-F 0 "#PWR040" H 9700 1300 50  0001 C CNN
-F 1 "GND" H 9700 1400 50  0000 C CNN
-F 2 "" H 9700 1550 50  0001 C CNN
-F 3 "" H 9700 1550 50  0001 C CNN
-	1    9700 1550
+P 9500 1550
+F 0 "#PWR040" H 9500 1300 50  0001 C CNN
+F 1 "GND" H 9500 1400 50  0000 C CNN
+F 2 "" H 9500 1550 50  0001 C CNN
+F 3 "" H 9500 1550 50  0001 C CNN
+	1    9500 1550
 	-1   0    0    -1
 $EndComp
@@
 L Device:R R30
 U 1 1 5B6A0D19
-P 9450 1150
-F 0 "R30" V 9530 1150 50  0000 C CNN
-F 1 "1K" V 9450 1150 50  0000 C CNN
-F 2 "Resistor_SMD:R_1206_3216Metric" V 9380 1150 50  0001 C CNN
-F 3 "~" H 9450 1150 50  0001 C CNN
-	1    9450 1150
+P 9700 1150
+F 0 "R30" V 9780 1150 50  0000 C CNN
+F 1 "10k" V 9700 1150 50  0000 C CNN
+F 2 "Resistor_SMD:R_1206_3216Metric" V 9630 1150 50  0001 C CNN
+F 3 "~" H 9700 1150 50  0001 C CNN
+	1    9700 1150
 	0    1    1    0
 $EndComp
@@
 	9200 1550 9200 1500
 Wire Wire Line
-	9300 1150 9200 1150
+	9550 1150 9500 1150
 Connection ~ 9200 1150
 Wire Wire Line
@@
 	9850 3900 9850 3950
 Wire Wire Line
-	9600 1150 9700 1150
-Wire Wire Line
-	9700 1150 9700 1200
-Wire Wire Line
-	9700 1150 9900 1150
-Connection ~ 9700 1150
-Wire Wire Line
 	4850 3750 4950 3750
 $Comp
@@
 	9500 2150 9500 2250
 Wire Wire Line
-	8500 2950 8350 2950
-Wire Wire Line
-	8350 2850 8500 2850
-Wire Wire Line
-	8500 2750 8350 2750
-Wire Wire Line
 	8350 2650 8500 2650
 Wire Wire Line
@@
 Connection ~ 5500 1450
 Wire Wire Line
-	6750 1850 6750 1150
+	6750 1850 6750 1550
 Wire Wire Line
 	6750 1150 6650 1150
-Text GLabel 6600 1850 0    50   Output ~ 0
+Text GLabel 6650 1550 0    50   Output ~ 0
 VREF
-Wire Wire Line
-	6600 1850 6750 1850
 Text GLabel 5450 2350 2    50   Input ~ 0
 VREF
@@
 VREF
 Wire Wire Line
-	9700 1550 9700 1500
+	9500 1550 9500 1500
 NoConn ~ 7350 2250
 NoConn ~ 7350 2350
-NoConn ~ 7350 2450
 NoConn ~ 4450 3550
 NoConn ~ 10600 2600
@@
 Text Notes 1200 8100 0    50   ~ 0
 http://nl.farnell.com/epcos/b82722a2202n001/filter-common-mode-choke-2-2mh/dp/1223076?ost=B82722A2202N001&scope=partnumberlookahead&exaMfpn=true&searchref=searchlookahead&ddkey=http%3Anl-NL%2FElement14_Netherlands%2Fw%2Fsearch
-Wire Wire Line
-	1850 4350 1000 4350
 $Comp
 L TrackAmplifier-rescue:C C35
@@
 Connection ~ 1000 4950
 Connection ~ 1000 5350
-Wire Wire Line
-	1000 3950 1000 4350
 $Comp
 L Sensor_Temperature:LM35-LP U11
@@
 Connection ~ 1650 1300
 Wire Wire Line
-	9200 4650 9200 5850
+	9200 4650 9200 5650
 Wire Wire Line
 	9000 4750 9250 4750
 Connection ~ 9250 4750
 Wire Wire Line
-	9250 4750 9250 5950
+	9250 4750 9250 5750
 Wire Wire Line
 	9000 4550 9200 4550
@@
 Connection ~ 2650 2300
 Wire Wire Line
-	2650 2300 2700 2300
+	2650 2300 3000 2300
 $Comp
 L TrackAmplifier-rescue:GND #PWR05
@@
 Wire Wire Line
 	2350 5700 2850 5700
-NoConn ~ 2650 7400
 Wire Wire Line
 	2750 7450 2750 7400
@@
 	0    -1   -1   0
 $EndComp
-Connection ~ 6750 1850
 Wire Wire Line
 	6750 1850 6800 1850
@@
 	5250 6050 5250 6100
 Wire Wire Line
-	9250 6150 9250 5950
-Connection ~ 9250 5950
-Wire Wire Line
 	8450 4550 8600 4550
 Wire Wire Line
 	8450 4750 8600 4750
+Text GLabel 2650 7450 3    50   Output ~ 0
+THFLG
+Wire Wire Line
+	2650 7400 2650 7450
+Text GLabel 6350 2500 3    50   Output ~ 0
+THFLG
+Wire Wire Line
+	6650 1550 6750 1550
+Connection ~ 6750 1550
+Wire Wire Line
+	6750 1550 6750 1150
+$Comp
+L power:+5V #PWR049
+U 1 1 5AFAD006
+P 6350 2050
+F 0 "#PWR049" H 6350 1900 50  0001 C CNN
+F 1 "+5V" H 6350 2190 50  0000 C CNN
+F 2 "" H 6350 2050 50  0001 C CNN
+F 3 "" H 6350 2050 50  0001 C CNN
+	1    6350 2050
+	1    0    0    -1
+$EndComp
+$Comp
+L Device:R R40
+U 1 1 5AFAD0DF
+P 6350 2250
+F 0 "R40" V 6430 2250 50  0000 C CNN
+F 1 "4k7" V 6350 2250 50  0000 C CNN
+F 2 "Resistor_SMD:R_1206_3216Metric" V 6280 2250 50  0001 C CNN
+F 3 "~" H 6350 2250 50  0001 C CNN
+	1    6350 2250
+	1    0    0    -1
+$EndComp
+Wire Wire Line
+	6350 2050 6350 2100
+Wire Wire Line
+	6350 2400 6350 2450
+Wire Wire Line
+	7350 2450 6350 2450
+Connection ~ 6350 2450
+Wire Wire Line
+	6350 2450 6350 2500
+$Comp
+L TrackAmplifier-rescue:C C37
+U 1 1 5B05E585
+P 3000 2550
+F 0 "C37" H 3025 2650 50  0000 L CNN
+F 1 "100n" H 3025 2450 50  0000 L CNN
+F 2 "Capacitor_SMD:C_1206_3216Metric" H 3038 2400 50  0001 C CNN
+F 3 "" H 3000 2550 50  0001 C CNN
+	1    3000 2550
+	-1   0    0    1
+$EndComp
+Wire Wire Line
+	3000 2400 3000 2300
+Connection ~ 3000 2300
+Wire Wire Line
+	3000 2300 3100 2300
+Wire Wire Line
+	3000 2700 2650 2700
+Connection ~ 2650 2700
+Wire Wire Line
+	1000 4250 1000 3950
+Connection ~ 1000 3950
+Wire Wire Line
+	9850 1150 9900 1150
+Wire Wire Line
+	9500 1200 9500 1150
+Connection ~ 9500 1150
+Wire Wire Line
+	9500 1150 9200 1150
+Wire Wire Line
+	10100 5650 9200 5650
+Wire Wire Line
+	10100 5750 9250 5750
+Connection ~ 9250 5750
+Wire Wire Line
+	9250 5750 9250 6150
+Wire Wire Line
+	9800 5850 10100 5850
+Wire Wire Line
+	10100 5950 9800 5950
+Wire Wire Line
+	9800 5450 10100 5450
+Wire Wire Line
+	10100 5550 9800 5550
+Wire Wire Line
+	8350 2750 8500 2750
+Wire Wire Line
+	8500 2850 8350 2850
+Wire Wire Line
+	8350 2950 8500 2950
 $EndSCHEMATC

Commit message: Updated chematic and pcb according to fit test
Connections:
- wire segments 421 -> 420
Changed lines of the file:
@@
 	1    0    0    1
 $EndComp
-Wire Wire Line
-	10100 4550 9250 4550
-Wire Wire Line
-	9250 4550 9250 4750
-Wire Wire Line
-	10100 4650 9200 4650
 $Comp
 L TrackAmplifier-rescue:C C7
@@
 Wire Wire Line
 	3600 3850 3650 3850
-Text GLabel 9800 4950 0    50   Output ~ 0
+Text GLabel 9800 5550 0    50   Output ~ 0
 Reset_B
-Text GLabel 9800 4850 0    50   Output ~ 0
+Text GLabel 9800 5650 0    50   Output ~ 0
 Reset_A
+Text GLabel 9800 5350 0    50   Output ~ 0
+Sync_B
+Text GLabel 9800 5450 0    50   Output ~ 0
+Sync_A
 Text GLabel 9800 5150 0    50   Output ~ 0
-Sync_B
-Text GLabel 9800 5050 0    50   Output ~ 0
-Sync_A
-Text GLabel 9800 5350 0    50   Output ~ 0
 RX_B
 Text GLabel 9800 5250 0    50   Output ~ 0
 RX_A
-Text GLabel 9800 5550 0    50   Input ~ 0
+Text GLabel 9800 4950 0    50   Input ~ 0
 TX_B
-Text GLabel 9800 5450 0    50   Input ~ 0
+Text GLabel 9800 5050 0    50   Input ~ 0
 TX_A
 $Comp
@@
 Text GLabel 5800 6950 2    50   Output ~ 0
 PWMO2
-Text GLabel 9800 5850 0    50   Input ~ 0
+Text GLabel 9800 4650 0    50   Input ~ 0
 PWMO1
-Text GLabel 9800 5950 0    50   Input ~ 0
+Text GLabel 9800 4550 0    50   Input ~ 0
 PWMO2
 Wire Wire Line
@@
 Wire Wire Line
 	10450 3500 10600 3500
-Text GLabel 9800 4750 0    50   Input ~ 0
+Text GLabel 9800 5750 0    50   Input ~ 0
 ID_R
 Text GLabel 9900 1400 3    50   Output ~ 0
@@
 Text Notes 2150 1900 0    50   ~ 0
 Disconnected receiver inputs\nor idle bus will have RO high.\nInvert for continuous uController reset
-Wire Wire Line
-	9800 4750 10100 4750
 $Comp
 L power:GNDD #PWR046
@@
 	1    0    0    -1
 $EndComp
-Wire Wire Line
-	9800 4850 10100 4850
-Wire Wire Line
-	9800 4950 10100 4950
-Wire Wire Line
-	9800 5050 10100 5050
-Wire Wire Line
-	9800 5150 10100 5150
-Wire Wire Line
-	9800 5250 10100 5250
-Wire Wire Line
-	9800 5350 10100 5350
 Text GLabel 950  5900 0    50   Input ~ 0
 Vbus_flt
@@
 Connection ~ 1650 1300
 Wire Wire Line
-	9200 4650 9200 5650
-Wire Wire Line
 	9000 4750 9250 4750
 Connection ~ 9250 4750
 Wire Wire Line
-	9250 4750 9250 5750
-Wire Wire Line
 	9000 4550 9200 4550
-Wire Wire Line
-	9200 4550 9200 4650
-Connection ~ 9200 4650
 $Comp
 L Device:R R36
@@
 	9500 1150 9200 1150
 Wire Wire Line
-	10100 5650 9200 5650
-Wire Wire Line
-	10100 5750 9250 5750
-Connection ~ 9250 5750
-Wire Wire Line
-	9250 5750 9250 6150
-Wire Wire Line
-	9800 5850 10100 5850
-Wire Wire Line
-	10100 5950 9800 5950
+	8350 2750 8500 2750
+Wire Wire Line
+	8500 2850 8350 2850
+Wire Wire Line
+	8350 2950 8500 2950
+Wire Wire Line
+	10100 5850 9200 5850
+Wire Wire Line
+	10100 4850 9200 4850
+Connection ~ 9200 4850
+Wire Wire Line
+	9200 4850 9200 5850
+Wire Wire Line
+	9200 4550 9200 4850
+Wire Wire Line
+	9250 4750 9250 5950
+Wire Wire Line
+	10100 5950 9250 5950
+Connection ~ 9250 5950
+Wire Wire Line
+	9250 5950 9250 6150
+Wire Wire Line
+	10100 4750 9250 4750
+Wire Wire Line
+	9800 4550 10100 4550
+Wire Wire Line
+	10100 4650 9800 4650
+Wire Wire Line
+	9800 5750 10100 5750
+Wire Wire Line
+	9800 5650 10100 5650
+Wire Wire Line
+	9800 5550 10100 5550
+Wire Wire Line
+	9800 4950 10100 4950
+Wire Wire Line
+	9800 5050 10100 5050
+Wire Wire Line
+	10100 5150 9800 5150
+Wire Wire Line
+	9800 5250 10100 5250
+Wire Wire Line
+	10100 5350 9800 5350
 Wire Wire Line
 	9800 5450 10100 5450
-Wire Wire Line
-	10100 5550 9800 5550
-Wire Wire Line
-	8350 2750 8500 2750
-Wire Wire Line
-	8500 2850 8350 2850
-Wire Wire Line
-	8350 2950 8500 2950
 $EndSCHEMATC

Commit message: Proto TrackAmplifier done!
Parts:
- added C38: 22u, Capacitor_SMD:C_1206_3216Metric, symbol TrackAmplifier-rescue:C
- U1, U2, U5, U6: symbol Interface_UART:ST485EBDR -> TrackAmplifier-rescue:ST485EBDR-Interface_UART
- U4: symbol Driver_Motor:LMD18200 -> TrackAmplifier-rescue:LMD18200-Driver_Motor
- U9: symbol MCU_Microchip_PIC16:PIC16F18854-SO -> TrackAmplifier-rescue:PIC16F18854-SO-MCU_Microchip_PIC16
Connections:
- wire segments 420 -> 423
Other:
- moved on the sheet: C34, C35
Changed lines of the file:
@@
 $EndComp
 $Comp
-L Interface_UART:ST485EBDR U1
+L TrackAmplifier-rescue:ST485EBDR-Interface_UART U1
 U 1 1 5AE19840
 P 1850 2400
@@
 	2350 2600 2350 2500
 $Comp
-L Interface_UART:ST485EBDR U2
+L TrackAmplifier-rescue:ST485EBDR-Interface_UART U2
 U 1 1 5AE58D1D
 P 1850 3700
@@
 	2350 3900 2350 3800
 $Comp
-L Interface_UART:ST485EBDR U6
+L TrackAmplifier-rescue:ST485EBDR-Interface_UART U6
 U 1 1 5AE5B3FC
 P 4050 5000
@@
 	4550 5200 4550 5100
 $Comp
-L Interface_UART:ST485EBDR U5
+L TrackAmplifier-rescue:ST485EBDR-Interface_UART U5
 U 1 1 5AE5F184
 P 4050 3650
@@
 TX_A
 $Comp
-L Driver_Motor:LMD18200 U4
+L TrackAmplifier-rescue:LMD18200-Driver_Motor U4
 U 1 1 5AE92F98
 P 2750 6800
@@
 Connection ~ 4050 3200
 $Comp
-L MCU_Microchip_PIC16:PIC16F18854-SO U9
+L TrackAmplifier-rescue:PIC16F18854-SO-MCU_Microchip_PIC16 U9
 U 1 1 5AEBDEF2
 P 7850 2350
@@
 	7500 4200 7550 4200
 Connection ~ 7500 4200
-Text GLabel 7200 2050 0    50   Input ~ 0
+Text GLabel 7200 1850 0    50   Input ~ 0
 OCC
 Wire Wire Line
@@
 Wire Wire Line
 	7200 1950 7350 1950
-Wire Wire Line
-	7350 2050 7200 2050
 $Comp
 L Reference_Voltage:REF3025 U10
@@
 Connection ~ 5500 1450
 Wire Wire Line
-	6750 1850 6750 1550
-Wire Wire Line
 	6750 1150 6650 1150
 Text GLabel 6650 1550 0    50   Output ~ 0
@@
 L TrackAmplifier-rescue:C C35
 U 1 1 5AEECD74
-P 1000 5150
-F 0 "C35" H 1025 5250 50  0000 L CNN
-F 1 "100n" H 1025 5050 50  0000 L CNN
-F 2 "Capacitor_SMD:C_1206_3216Metric" H 1038 5000 50  0001 C CNN
-F 3 "" H 1000 5150 50  0001 C CNN
-	1    1000 5150
+P 1000 5000
+F 0 "C35" H 1025 5100 50  0000 L CNN
+F 1 "100n" H 1025 4900 50  0000 L CNN
+F 2 "Capacitor_SMD:C_1206_3216Metric" H 1038 4850 50  0001 C CNN
+F 3 "" H 1000 5000 50  0001 C CNN
+	1    1000 5000
 	-1   0    0    1
 $EndComp
@@
 L TrackAmplifier-rescue:C C34
 U 1 1 5AEECD7B
-P 750 5150
-F 0 "C34" H 775 5250 50  0000 L CNN
-F 1 "22u" H 775 5050 50  0000 L CNN
-F 2 "Capacitor_SMD:C_1206_3216Metric" H 788 5000 50  0001 C CNN
-F 3 "" H 750 5150 50  0001 C CNN
-	1    750  5150
+P 750 5000
+F 0 "C34" H 775 5100 50  0000 L CNN
+F 1 "22u" H 775 4900 50  0000 L CNN
+F 2 "Capacitor_SMD:C_1206_3216Metric" H 788 4850 50  0001 C CNN
+F 3 "" H 750 5000 50  0001 C CNN
+	1    750  5000
 	-1   0    0    1
 $EndComp
@@
 L power:+5V #PWR0101
 U 1 1 5AEECD82
-P 750 4550
-F 0 "#PWR0101" H 750 4400 50  0001 C CNN
-F 1 "+5V" H 750 4690 50  0000 C CNN
-F 2 "" H 750 4550 50  0001 C CNN
-F 3 "" H 750 4550 50  0001 C CNN
-	1    750  4550
+P 750 4400
+F 0 "#PWR0101" H 750 4250 50  0001 C CNN
+F 1 "+5V" H 750 4540 50  0000 C CNN
+F 2 "" H 750 4400 50  0001 C CNN
+F 3 "" H 750 4400 50  0001 C CNN
+	1    750  4400
 	1    0    0    -1
 $EndComp
@@
 L TrackAmplifier-rescue:GND #PWR0102
 U 1 1 5AEECD88
-P 750 5400
-F 0 "#PWR0102" H 750 5150 50  0001 C CNN
-F 1 "GND" H 750 5250 50  0000 C CNN
-F 2 "" H 750 5400 50  0001 C CNN
-F 3 "" H 750 5400 50  0001 C CNN
-	1    750  5400
+P 750 5250
+F 0 "#PWR0102" H 750 5000 50  0001 C CNN
+F 1 "GND" H 750 5100 50  0000 C CNN
+F 2 "" H 750 5250 50  0001 C CNN
+F 3 "" H 750 5250 50  0001 C CNN
+	1    750  5250
 	-1   0    0    -1
 $EndComp
@@
 L Device:R R11
 U 1 1 5AEECD8E
-P 750 4750
-F 0 "R11" V 830 4750 50  0000 C CNN
-F 1 "10E" V 750 4750 50  0000 C CNN
-F 2 "Resistor_SMD:R_1206_3216Metric" V 680 4750 50  0001 C CNN
-F 3 "~" H 750 4750 50  0001 C CNN
-	1    750  4750
-	-1   0    0    1
-$EndComp
-Wire Wire Line
-	750  4550 750  4600
-Wire Wire Line
-	750  4900 750  4950
-Wire Wire Line
-	750  5300 750  5350
-Wire Wire Line
-	750  4950 1000 4950
-Wire Wire Line
-	1000 4950 1000 5000
-Connection ~ 750  4950
-Wire Wire Line
-	750  4950 750  5000
-Wire Wire Line
-	750  5350 1000 5350
-Wire Wire Line
-	1000 5350 1000 5300
-Connection ~ 750  5350
-Wire Wire Line
-	750  5350 750  5400
-Connection ~ 1000 4950
-Connection ~ 1000 5350
+P 750 4600
+F 0 "R11" V 830 4600 50  0000 C CNN
+F 1 "10E" V 750 4600 50  0000 C CNN
+F 2 "Resistor_SMD:R_1206_3216Metric" V 680 4600 50  0001 C CNN
+F 3 "~" H 750 4600 50  0001 C CNN
+	1    750  4600
+	-1   0    0    1
+$EndComp
+Wire Wire Line
+	750  4400 750  4450
+Wire Wire Line
+	750  4750 750  4800
+Wire Wire Line
+	750  5150 750  5200
+Wire Wire Line
+	750  4800 1000 4800
+Wire Wire Line
+	1000 4800 1000 4850
+Connection ~ 750  4800
+Wire Wire Line
+	750  4800 750  4850
+Wire Wire Line
+	750  5200 1000 5200
+Wire Wire Line
+	1000 5200 1000 5150
+Connection ~ 750  5200
+Wire Wire Line
+	750  5200 750  5250
+Connection ~ 1000 4800
+Connection ~ 1000 5200
 $Comp
 L Sensor_Temperature:LM35-LP U11
 U 1 1 5AEEC2F8
-P 1500 5200
-F 0 "U11" H 1250 5450 50  0000 C CNN
-F 1 "LM35-LP" H 1550 5450 50  0000 L CNN
-F 2 "Package_TO_SOT_THT:TO-92" H 1550 4950 50  0001 L CNN
-F 3 "http://www.ti.com/lit/ds/symlink/lm35.pdf" H 1500 5200 50  0001 C CNN
-	1    1500 5200
-	1    0    0    -1
-$EndComp
-Wire Wire Line
-	1500 5500 1500 5600
-Wire Wire Line
-	1500 5600 1000 5600
-Wire Wire Line
-	1000 5600 1000 5350
-Wire Wire Line
-	1500 4900 1500 4800
-Wire Wire Line
-	1500 4800 1000 4800
-Wire Wire Line
-	1000 4800 1000 4950
-Text GLabel 2350 5200 2    50   Output ~ 0
+P 1500 5050
+F 0 "U11" H 1250 5300 50  0000 C CNN
+F 1 "LM35-LP" H 1550 5300 50  0000 L CNN
+F 2 "Package_TO_SOT_THT:TO-92" H 1550 4800 50  0001 L CNN
+F 3 "http://www.ti.com/lit/ds/symlink/lm35.pdf" H 1500 5050 50  0001 C CNN
+	1    1500 5050
+	1    0    0    -1
+$EndComp
+Wire Wire Line
+	1500 5350 1500 5450
+Wire Wire Line
+	1500 5450 1000 5450
+Wire Wire Line
+	1000 5450 1000 5200
+Wire Wire Line
+	1500 4750 1500 4650
+Wire Wire Line
+	1500 4650 1000 4650
+Wire Wire Line
+	1000 4650 1000 4800
+Text GLabel 2350 5050 2    50   Output ~ 0
 TEMP
 $Comp
@@
 L Device:R R37
 U 1 1 5AF19CD4
-P 2100 5200
-F 0 "R37" V 2180 5200 50  0000 C CNN
-F 1 "10E" V 2100 5200 50  0000 C CNN
-F 2 "Resistor_SMD:R_1206_3216Metric" V 2030 5200 50  0001 C CNN
-F 3 "~" H 2100 5200 50  0001 C CNN
-	1    2100 5200
+P 2100 5050
+F 0 "R37" V 2180 5050 50  0000 C CNN
+F 1 "10E" V 2100 5050 50  0000 C CNN
+F 2 "Resistor_SMD:R_1206_3216Metric" V 2030 5050 50  0001 C CNN
+F 3 "~" H 2100 5050 50  0001 C CNN
+	1    2100 5050
 	0    -1   -1   0
 $EndComp
 Wire Wire Line
-	1900 5200 1950 5200
-Wire Wire Line
-	2250 5200 2350 5200
+	1900 5050 1950 5050
+Wire Wire Line
+	2250 5050 2300 5050
 Wire Wire Line
 	5050 2700 5050 2750
@@
 L Device:R R38
 U 1 1 5AFB301E
-P 6950 1850
-F 0 "R38" V 7030 1850 50  0000 C CNN
-F 1 "10E" V 6950 1850 50  0000 C CNN
-F 2 "Resistor_SMD:R_1206_3216Metric" V 6880 1850 50  0001 C CNN
-F 3 "~" H 6950 1850 50  0001 C CNN
-	1    6950 1850
-	0    -1   -1   0
-$EndComp
-Wire Wire Line
-	6750 1850 6800 1850
-Wire Wire Line
-	7100 1850 7350 1850
+P 6750 1750
+F 0 "R38" V 6830 1750 50  0000 C CNN
+F 1 "10E" V 6750 1750 50  0000 C CNN
+F 2 "Resistor_SMD:R_1206_3216Metric" V 6680 1750 50  0001 C CNN
+F 3 "~" H 6750 1750 50  0001 C CNN
+	1    6750 1750
+	1    0    0    -1
+$EndComp
 Wire Wire Line
 	7200 1750 7350 1750
@@
 Wire Wire Line
 	6650 1550 6750 1550
-Connection ~ 6750 1550
 Wire Wire Line
 	6750 1550 6750 1150
@@
 Wire Wire Line
 	9800 5450 10100 5450
+Wire Wire Line
+	7200 1850 7350 1850
+Wire Wire Line
+	6750 1600 6750 1550
+Connection ~ 6750 1550
+Wire Wire Line
+	7350 2050 6750 2050
+Wire Wire Line
+	6750 2050 6750 1900
+$Comp
+L TrackAmplifier-rescue:C C38
+U 1 1 5B022B32
+P 2300 5250
+F 0 "C38" H 2325 5350 50  0000 L CNN
+F 1 "22u" H 2325 5150 50  0000 L CNN
+F 2 "Capacitor_SMD:C_1206_3216Metric" H 2338 5100 50  0001 C CNN
+F 3 "" H 2300 5250 50  0001 C CNN
+	1    2300 5250
+	-1   0    0    1
+$EndComp
+$Comp
+L TrackAmplifier-rescue:GND #PWR050
+U 1 1 5B04E1AB
+P 2300 5450
+F 0 "#PWR050" H 2300 5200 50  0001 C CNN
+F 1 "GND" H 2300 5300 50  0000 C CNN
+F 2 "" H 2300 5450 50  0001 C CNN
+F 3 "" H 2300 5450 50  0001 C CNN
+	1    2300 5450
+	-1   0    0    -1
+$EndComp
+Wire Wire Line
+	2300 5050 2300 5100
+Connection ~ 2300 5050
+Wire Wire Line
+	2300 5050 2350 5050
+Wire Wire Line
+	2300 5400 2300 5450
 $EndSCHEMATC
