File: KiCad/TrackAmplifier/TrackAmplifier.sch (KiCad schematic (older format))
At the start: 106 parts, among them J1 DB15_Male_MountingHoles, J2 Conn_01x06, Q1 2N7002, U1 ST485EBDR, U10 REF3025, U11 LM35-LP, U2 ST485EBDR, U3 LM78M05_TO252, U4 LMD18200, U5 ST485EBDR, U6 ST485EBDR, U7 INA326, U8 INA326, U9 PIC16F18854-SO

Commit message: updating with Farnell orderno
Parts:
- C10, C7: Farnell (none) -> 2395785
- D1: Farnell (none) -> 1581232
- D2: Farnell (none) -> 1581231
- D3: Farnell (none) -> 1581229
- D4, D8: Farnell (none) -> 1581233
- J1: Farnell (none) -> 2294292
- Q1: Farnell (none) -> 2317616
- R3: Farnell (none) -> 1653053
- U1, U2, U5, U6: Farnell (none) -> 1467755
- U10: Farnell (none) -> 1234684
- U11: Farnell (none) -> 1469236
- U3: Farnell (none) -> 2854542
- U4: Farnell (none) -> 1468979
- U7, U8: Farnell (none) -> 2764750
- U9: Farnell (none) -> 2696647
Other:
- note added: "BL"
- note added: "GR"
- note added: "RD"
- note added: "YE"
Changed lines of the file:
@@
 F 2 "Connector_Dsub:DSUB-15_Male_Horizontal_P2.77x2.84mm_EdgePinOffset4.94mm_Housed_MountingHolesOffset7.48mm" H 10400 5250 50  0001 C CNN
 F 3 "" H 10400 5250 50  0001 C CNN
+F 4 "2294292" H 10400 5250 50  0001 C CNN "Farnell"
 	1    10400 5250
 	1    0    0    1
@@
 F 1 "100n" H 1975 950 50  0000 L CNN
 F 2 "Capacitor_SMD:C_1206_3216Metric" H 1988 900 50  0001 C CNN
-F 3 "" H 1950 1050 50  0001 C CNN
+F 3 "http://www.farnell.com/datasheets/2049140.pdf?_ga=2.261496907.792852979.1526285019-1651149783.1519657816" H 1950 1050 50  0001 C CNN
+F 4 "2395785" H 1950 1050 50  0001 C CNN "Farnell"
 	1    1950 1050
 	-1   0    0    1
@@
 F 2 "Package_SO:SOIC-8_3.9x4.9mm_P1.27mm" H 1850 1500 50  0001 C CNN
 F 3 "http://www.st.com/resource/en/datasheet/st485eb.pdf" H 1850 2450 50  0001 C CNN
+F 4 "1467755" H 1850 2400 50  0001 C CNN "Farnell"
 	1    1850 2400
 	-1   0    0    -1
@@
 F 2 "Package_TO_SOT_SMD:TO-252-2" H 2350 1025 50  0001 C CIN
 F 3 "http://www.fairchildsemi.com/ds/LM/LM78M05.pdf" H 2350 750 50  0001 C CNN
+F 4 "2854542" H 2350 800 50  0001 C CNN "Farnell"
 	1    2350 800
 	1    0    0    -1
@@
 F 1 "100n" H 2925 950 50  0000 L CNN
 F 2 "Capacitor_SMD:C_1206_3216Metric" H 2938 900 50  0001 C CNN
-F 3 "" H 2900 1050 50  0001 C CNN
+F 3 "http://www.farnell.com/datasheets/2049140.pdf?_ga=2.50946415.792852979.1526285019-1651149783.1519657816" H 2900 1050 50  0001 C CNN
+F 4 "2395785" H 2900 1050 50  0001 C CNN "Farnell"
 	1    2900 1050
 	-1   0    0    1
@@
 F 2 "Package_SO:SOIC-8_3.9x4.9mm_P1.27mm" H 1850 2800 50  0001 C CNN
 F 3 "http://www.st.com/resource/en/datasheet/st485eb.pdf" H 1850 3750 50  0001 C CNN
+F 4 "1467755" H 1850 3700 50  0001 C CNN "Farnell"
 	1    1850 3700
 	-1   0    0    -1
@@
 F 2 "Package_SO:SOIC-8_3.9x4.9mm_P1.27mm" H 4050 4100 50  0001 C CNN
 F 3 "http://www.st.com/resource/en/datasheet/st485eb.pdf" H 4050 5050 50  0001 C CNN
+F 4 "1467755" H 4050 5000 50  0001 C CNN "Farnell"
 	1    4050 5000
 	-1   0    0    -1
@@
 F 2 "Package_SO:SOIC-8_3.9x4.9mm_P1.27mm" H 4050 2750 50  0001 C CNN
 F 3 "http://www.st.com/resource/en/datasheet/st485eb.pdf" H 4050 3700 50  0001 C CNN
+F 4 "1467755" H 4050 3650 50  0001 C CNN "Farnell"
 	1    4050 3650
 	-1   0    0    -1
@@
 F 2 "Package_TO_SOT_THT:TO-220-11_20.02x17.50mm_P3.4x5.08mm_StaggerOdd_Lead8.45mm_Tab-Down" H 2750 5900 50  0001 C CNN
 F 3 "http://www.ti.com/lit/ds/symlink/lmd18200.pdf" H 2650 6800 50  0001 C CNN
+F 4 "1468979" H 2750 6800 50  0001 C CNN "Farnell"
 	1    2750 6800
 	1    0    0    -1
@@
 F 2 "Package_SO:SOIC-28W_7.5x17.9mm_P1.27mm" H 7850 1250 50  0001 C CNN
 F 3 "http://ww1.microchip.com/downloads/en/DeviceDoc/PIC16(L)F18854%20Data%20Sheet_DS40001826C.pdf" H 8150 1750 50  0001 C CNN
+F 4 "2696647" H 7850 2350 50  0001 C CNN "Farnell"
 	1    7850 2350
 	1    0    0    -1
@@
 F 2 "Package_TO_SOT_SMD:SOT-23" H 3500 2225 50  0001 L CIN
 F 3 "https://www.fairchildsemi.com/datasheets/2N/2N7002.pdf" H 3300 2300 50  0001 L CNN
+F 4 "2317616" H 3300 2300 50  0001 C CNN "Farnell"
 	1    3300 2300
 	1    0    0    -1
@@
 F 2 "Package_SO:MSOP-8_3x3mm_P0.65mm" H 4950 1750 50  0001 L CNN
 F 3 "http://www.ti.com/lit/ds/symlink/ina326.pdf" H 5050 1750 50  0001 C CNN
+F 4 "2764750" H 4950 1750 50  0001 C CNN "Farnell"
 	1    4950 1750
 	1    0    0    -1
@@
 F 2 "Package_SO:MSOP-8_3x3mm_P0.65mm" H 6550 4200 50  0001 L CNN
 F 3 "http://www.ti.com/lit/ds/symlink/ina326.pdf" H 6650 4200 50  0001 C CNN
+F 4 "2764750" H 6550 4200 50  0001 C CNN "Farnell"
 	1    6550 4200
 	1    0    0    -1
@@
 F 2 "LED_SMD:LED_1206_3216Metric" H 9150 1950 50  0001 C CNN
 F 3 "~" H 9150 1950 50  0001 C CNN
+F 4 "1581232" H 9150 1950 50  0001 C CNN "Farnell"
 	1    9150 1950
 	-1   0    0    1
@@
 F 2 "LED_SMD:LED_1206_3216Metric" H 9150 2050 50  0001 C CNN
 F 3 "~" H 9150 2050 50  0001 C CNN
+F 4 "1581231" H 9150 2050 50  0001 C CNN "Farnell"
 	1    9150 2050
 	-1   0    0    1
@@
 F 2 "LED_SMD:LED_1206_3216Metric" H 9150 2150 50  0001 C CNN
 F 3 "~" H 9150 2150 50  0001 C CNN
+F 4 "1581229" H 9150 2150 50  0001 C CNN "Farnell"
 	1    9150 2150
 	-1   0    0    1
@@
 F 2 "LED_SMD:LED_1206_3216Metric" H 9150 2250 50  0001 C CNN
 F 3 "~" H 9150 2250 50  0001 C CNN
+F 4 "1581233" H 9150 2250 50  0001 C CNN "Farnell"
 	1    9150 2250
 	-1   0    0    1
@@
 F 1 "10E" V 1100 800 50  0000 C CNN
 F 2 "Resistor_SMD:R_1206_3216Metric" V 1030 800 50  0001 C CNN
-F 3 "~" H 1100 800 50  0001 C CNN
+F 3 "http://www.farnell.com/datasheets/2310790.pdf?_ga=2.157221117.792852979.1526285019-1651149783.1519657816" H 1100 800 50  0001 C CNN
+F 4 "1653053" V 1100 800 50  0001 C CNN "Farnell"
 	1    1100 800
 	0    -1   -1   0
@@
 F 2 "Package_TO_SOT_SMD:SOT-23" H 6350 700 50  0001 C CIN
 F 3 "http://www.ti.com/lit/ds/symlink/ref3033.pdf" H 6450 800 50  0001 C CIN
+F 4 "1234684" H 6350 1150 50  0001 C CNN "Farnell"
 	1    6350 1150
 	1    0    0    -1
@@
 F 2 "LED_SMD:LED_1206_3216Metric" H 9150 2350 50  0001 C CNN
 F 3 "~" H 9150 2350 50  0001 C CNN
+F 4 "1581233" H 9150 2350 50  0001 C CNN "Farnell"
 	1    9150 2350
 	-1   0    0    1
@@
 F 2 "Package_TO_SOT_THT:TO-92" H 1550 4800 50  0001 L CNN
 F 3 "http://www.ti.com/lit/ds/symlink/lm35.pdf" H 1500 5050 50  0001 C CNN
+F 4 "1469236" H 1500 5050 50  0001 C CNN "Farnell"
 	1    1500 5050
 	1    0    0    -1
@@
 Wire Wire Line
 	2300 5400 2300 5450
+Text Notes 9550 2000 0    50   ~ 0
+GR
+Text Notes 9550 2100 0    50   ~ 0
+YE
+Text Notes 9550 2200 0    50   ~ 0
+RD
+Text Notes 9550 2300 0    50   ~ 0
+BL
+Text Notes 9550 2400 0    50   ~ 0
+BL
 $EndSCHEMATC

Commit message: Updated schematic with component values and order nr
Parts:
- C1, C11, C12, C19, C2, C26, C29, C32, C34, C8: value 22u -> 2.2u
- C10: Manufacturer nr (none) -> VJ1206Y104KXBAT
- C13, C5: value 22u -> 2.2u; Farnell (none) -> 1759451; Manufacturer nr (none) -> MC1206F225Z250CT
- C16: value 100u -> 220u; Farnell (none) -> 2346568; Manufacturer nr (none) -> 16PX220MEFC6.3X11
- C17, C18: Farnell (none) -> 9406549; Manufacturer nr (none) -> MCU1206R103KCT
- C21, C25: value 100n -> np
- C22, C28: value 1u -> 100n
- C30, C36: value 220n -> 2.2u
- C6: Farnell (none) -> 2750201
- C7: Manufactufrer nr (none) -> VJ1206Y104KXBAT
- D1: Manufacturer nr (none) -> MCL-S250GC
- D10, D5, D6, D7, D9: Farnell (none) -> 2677464
- D2: Manufacturer nr (none) -> MCL-S250YC
- D3: Manufacturer nr (none) -> MCL-S250SRC
- D4, D8: Manufacturer nr (none) -> MCL-S250SBLC
- FL1, FL2: Farnell (none) -> 1223076; Manufacturer nr (none) -> B82722A2202N001
- Q1: Manufacturer nr (none) -> 2N7002ET1G
- R13: value 10E -> 402k; Farnell (none) -> 2139646; Manufacturer nr (none) -> CRCW1206402KFKEA
- R15: value 10E -> 39k; Farnell (none) -> 2139553; Manufacturer nr (none) -> CRCW120639K0FKEA
- R16: value 0.025 -> 0.025E; Farnell (none) -> 1107432; Manufacturer nr (none) -> WSK2512R0250FEA
- R17: value 10k -> 4k99; Farnell (none) -> 1470015; Manufacturer nr (none) -> CRCW12064K99FKEA
- R20: value 10E -> 2k00; Farnell (none) -> 1469985; Manufacturer nr (none) -> CRCW12062K00FKEA
- R21: value 10E -> 5M11; Farnell (none) -> 2139776; Manufacturer nr (none) -> CRCW12065M11FKEA
- R24: Farnell (none) -> 1653122; Manufacturer nr (none) -> CRCW12063K30FKEA
- R3: Manufacturer nr (none) -> CRCW120610R0FKEB
- R31: Farnell (none) -> 1469975; Manufacturer nr (none) -> CRCW1206100KFKEA
- R36: Farnell (none) -> 1469970; Manufacturer nr (none) -> CRCW120610K0FKEA
- R39: value 50k -> 1k; Farnell (none) -> 1653077; Manufacturer nr (none) -> CRCW12061K00JNEA
- R40: Farnell (none) -> 1470014; Manufacturer nr (none) -> CRCW12064K75FKEA
- R8: Farnell (none) -> 2616760; Manufacturer nr (none) -> CRCW1206100RJNEA
- U1, U2, U5, U6: Manufacturer nr (none) -> ST485EBDR
- U4: Manufacturer nr (none) -> LMD18200T
- U7, U8: Manufacturer nr (none) -> INA326EA/2K5
- U9: Manufacturer nr (none) -> PIC16F18854-I/SO
Other:
- note removed: "http://nl.farnell.com/epcos/b41858c7477m000/cap-alu-elec-aec-q200-470uf-35v/dp/2750201"
- note removed: "http://nl.farnell.com/epcos/b82722a2202n001/filter-common-mode-choke-2-2mh/dp/1223076?ost=B82722A2202N001&scope=partnumberlookahead&exaMfpn=true&searchref=searchlookahead&ddkey=http%3Anl-NL%2FElement14_Netherlands%2Fw%2Fsearch"
