File: KiCad/TrackAmplifier/TrackAmplifier.sch (KiCad schematic (older format))
At the start: 106 parts, among them J1 DB15_Male_MountingHoles, J2 Conn_01x06, Q1 2N7002, U1 ST485EBDR, U10 REF3025, U11 LM35-LP, U2 ST485EBDR, U3 LM78M05_TO252, U4 LMD18200, U5 ST485EBDR, U6 ST485EBDR, U7 INA326, U8 INA326, U9 PIC16F18854-SO

Commit message: Updated with component ordering
Parts:
- C23, C38: value 22u -> 2.2u
- C29, C30: value 2.2u -> 100n
- C7: Manufactufrer nr VJ1206Y104KXBAT -> (none); Manufacturer nr (none) -> VJ1206Y104KXBAT
- F1: value 3.0A -> 2.5A; Farnell (none) -> 9350268; Manufacturer nr (none) -> MF-SM250-2
- J1: Manufacturer nr (none) -> 182-015-113R531
- J2: Farnell (none) -> 3418327; Manufacturer nr (none) -> 826629-6
- MK1: Farnell (none) -> -; Manufacturer nr (none) -> -
- Q1: value 2N7002 -> BVSS123LT1G; Farnell 2317616 -> 2727944; Manufacturer nr 2N7002ET1G -> BVSS123LT1G
- R14, R4, R6, R7: value 4K7 -> 4k7
- R25: value 1K -> 4k7
- R26, R27: value 330E -> 301E; Farnell (none) -> 2139391; Manufacturer nr (none) -> CRCW1206301RFKEA
- R28: Farnell (none) -> 1470008; Manufacturer nr (none) -> CRCW1206330RFKEA
- R29, R35: value 330E -> 301E; Farnell (none) -> 2139391; Manufacturer nr (none) -> CRCW1206162RFKEA
- R30: value 10k -> 1k
- R33: value 1K -> 402k
- U10: Manufacturer nr (none) -> REF3025AIDBZTG4
- U11: Manufacturer nr (none) -> LM35DZ/NOPB
- U3: Manufacturer nr (none) -> LM78M05CDTX/NOPB
Other:
- note added: "Resistor on backplane \nwill determine ID voltage\n\nIf with potmeter:\nFarnell: 1141389"
- note added: "SMD Vishay resistors:\nhttp://nl.farnell.com/w/c/passive-components/resistors-fixed-value/chip-smd-resistors?brand=vishay&resistor-case-style=1206-3216-metric-&packaging=each|cuttape&range=inc-in-stock|exc-delivery-surcharge|exc-obs"
- note removed: "BL"
- note removed: "Resistor on backplane \nwill determine ID voltage"
Changed lines of the file:
@@
 F 1 "DB15_Male_MountingHoles" H 10400 6125 50  0000 C CNN
 F 2 "Connector_Dsub:DSUB-15_Male_Horizontal_P2.77x2.84mm_EdgePinOffset4.94mm_Housed_MountingHolesOffset7.48mm" H 10400 5250 50  0001 C CNN
-F 3 "" H 10400 5250 50  0001 C CNN
+F 3 "-" H 10400 5250 50  0001 C CNN
 F 4 "2294292" H 10400 5250 50  0001 C CNN "Farnell"
+F 5 "182-015-113R531" H 10400 5250 50  0001 C CNN "Manufacturer nr"
 	1    10400 5250
 	1    0    0    1
@@
 F 3 "http://www.farnell.com/datasheets/2049140.pdf?_ga=2.261496907.792852979.1526285019-1651149783.1519657816" H 1950 1050 50  0001 C CNN
 F 4 "2395785" H 1950 1050 50  0001 C CNN "Farnell"
-F 5 "VJ1206Y104KXBAT" H 1950 1050 50  0001 C CNN "Manufactufrer nr"
+F 5 "VJ1206Y104KXBAT" H 1950 1050 50  0001 C CNN "Manufacturer nr"
 	1    1950 1050
 	-1   0    0    1
@@
 F 3 "http://www.fairchildsemi.com/ds/LM/LM78M05.pdf" H 2350 750 50  0001 C CNN
 F 4 "2854542" H 2350 800 50  0001 C CNN "Farnell"
+F 5 "LM78M05CDTX/NOPB" H 2350 800 50  0001 C CNN "Manufacturer nr"
 	1    2350 800
 	1    0    0    -1
@@
 F 1 "Conn_01x06" H 10800 1900 50  0000 C CNN
 F 2 "Connector_PinHeader_2.54mm:PinHeader_1x06_P2.54mm_Vertical" H 10800 2300 50  0001 C CNN
-F 3 "~" H 10800 2300 50  0001 C CNN
+F 3 "http://www.farnell.com/datasheets/32535.pdf?_ga=2.160907771.792852979.1526285019-1651149783.1519657816" H 10800 2300 50  0001 C CNN
+F 4 "3418327" H 10800 2300 50  0001 C CNN "Farnell"
+F 5 "826629-6" H 10800 2300 50  0001 C CNN "Manufacturer nr"
 	1    10800 2300
 	1    0    0    -1
@@
 P 1700 7200
 F 0 "R6" V 1780 7200 50  0000 C CNN
-F 1 "4K7" V 1700 7200 50  0000 C CNN
+F 1 "4k7" V 1700 7200 50  0000 C CNN
 F 2 "Resistor_SMD:R_1206_3216Metric" V 1630 7200 50  0001 C CNN
 F 3 "~" H 1700 7200 50  0001 C CNN
@@
 P 1250 6700
 F 0 "R4" V 1330 6700 50  0000 C CNN
-F 1 "4K7" V 1250 6700 50  0000 C CNN
+F 1 "4k7" V 1250 6700 50  0000 C CNN
 F 2 "Resistor_SMD:R_1206_3216Metric" V 1180 6700 50  0001 C CNN
 F 3 "~" H 1250 6700 50  0001 C CNN
@@
 P 1900 7200
 F 0 "R7" V 1980 7200 50  0000 C CNN
-F 1 "4K7" V 1900 7200 50  0000 C CNN
+F 1 "4k7" V 1900 7200 50  0000 C CNN
 F 2 "Resistor_SMD:R_1206_3216Metric" V 1830 7200 50  0001 C CNN
 F 3 "~" H 1900 7200 50  0001 C CNN
@@
 P 4850 3950
 F 0 "R14" V 4930 3950 50  0000 C CNN
-F 1 "4K7" V 4850 3950 50  0000 C CNN
+F 1 "4k7" V 4850 3950 50  0000 C CNN
 F 2 "Resistor_SMD:R_1206_3216Metric" V 4780 3950 50  0001 C CNN
 F 3 "~" H 4850 3950 50  0001 C CNN
@@
 P 3300 2300
 F 0 "Q1" H 3500 2375 50  0000 L CNN
-F 1 "2N7002" H 3500 2300 50  0000 L CNN
+F 1 "BVSS123LT1G" H 3500 2300 50  0000 L CNN
 F 2 "Package_TO_SOT_SMD:SOT-23" H 3500 2225 50  0001 L CIN
-F 3 "https://www.fairchildsemi.com/datasheets/2N/2N7002.pdf" H 3300 2300 50  0001 L CNN
-F 4 "2317616" H 3300 2300 50  0001 C CNN "Farnell"
-F 5 "2N7002ET1G" H 3300 2300 50  0001 C CNN "Manufacturer nr"
+F 3 "http://www.farnell.com/datasheets/2255231.pdf?_ga=2.44068322.792852979.1526285019-1651149783.1519657816" H 3300 2300 50  0001 L CNN
+F 4 "2727944" H 3300 2300 50  0001 C CNN "Farnell"
+F 5 "BVSS123LT1G" H 3300 2300 50  0001 C CNN "Manufacturer nr"
 	1    3300 2300
 	1    0    0    -1
@@
 P 9900 950
 F 0 "R33" V 9980 950 50  0000 C CNN
-F 1 "1K" V 9900 950 50  0000 C CNN
+F 1 "402k" V 9900 950 50  0000 C CNN
 F 2 "Resistor_SMD:R_1206_3216Metric" V 9830 950 50  0001 C CNN
 F 3 "~" H 9900 950 50  0001 C CNN
@@
 P 9500 1350
 F 0 "C30" H 9525 1450 50  0000 L CNN
-F 1 "2.2u" H 9550 1250 50  0000 L CNN
+F 1 "100n" H 9550 1250 50  0000 L CNN
 F 2 "Capacitor_SMD:C_1206_3216Metric" H 9538 1200 50  0001 C CNN
 F 3 "" H 9500 1350 50  0001 C CNN
@@
 $EndComp
 Connection ~ 9900 1150
-Text Notes 10000 1250 0    50   ~ 0
-Resistor on backplane \nwill determine ID voltage
+Text Notes 10200 1350 0    50   ~ 0
+Resistor on backplane \nwill determine ID voltage\n\nIf with potmeter:\nFarnell: 1141389
 $Comp
 L Device:R R30
@@
 P 9700 1150
 F 0 "R30" V 9780 1150 50  0000 C CNN
-F 1 "10k" V 9700 1150 50  0000 C CNN
+F 1 "1k" V 9700 1150 50  0000 C CNN
 F 2 "Resistor_SMD:R_1206_3216Metric" V 9630 1150 50  0001 C CNN
 F 3 "~" H 9700 1150 50  0001 C CNN
@@
 P 6100 3450
 F 0 "C23" H 6125 3550 50  0000 L CNN
-F 1 "22u" H 6125 3350 50  0000 L CNN
+F 1 "2.2u" H 6125 3350 50  0000 L CNN
 F 2 "Capacitor_SMD:C_1206_3216Metric" H 6138 3300 50  0001 C CNN
 F 3 "" H 6100 3450 50  0001 C CNN
@@
 P 7900 5550
 F 0 "R25" V 7980 5550 50  0000 C CNN
-F 1 "1K" V 7900 5550 50  0000 C CNN
+F 1 "4k7" V 7900 5550 50  0000 C CNN
 F 2 "Resistor_SMD:R_1206_3216Metric" V 7830 5550 50  0001 C CNN
 F 3 "~" H 7900 5550 50  0001 C CNN
@@
 P 8150 5750
 F 0 "C29" H 8175 5850 50  0000 L CNN
-F 1 "2.2u" H 8175 5650 50  0000 L CNN
+F 1 "100n" H 8175 5650 50  0000 L CNN
 F 2 "Capacitor_SMD:C_1206_3216Metric" H 8188 5600 50  0001 C CNN
 F 3 "" H 8150 5750 50  0001 C CNN
@@
 P 8700 1950
 F 0 "R26" V 8750 2150 50  0000 C CNN
-F 1 "330E" V 8700 1950 50  0000 C CNN
+F 1 "301E" V 8700 1950 50  0000 C CNN
 F 2 "Resistor_SMD:R_1206_3216Metric" V 8630 1950 50  0001 C CNN
-F 3 "~" H 8700 1950 50  0001 C CNN
+F 3 "http://www.farnell.com/datasheets/2310790.pdf?_ga=2.18263423.792852979.1526285019-1651149783.1519657816" H 8700 1950 50  0001 C CNN
+F 4 "2139391" V 8700 1950 50  0001 C CNN "Farnell"
+F 5 "CRCW1206301RFKEA" V 8700 1950 50  0001 C CNN "Manufacturer nr"
 	1    8700 1950
 	0    -1   -1   0
@@
 P 8700 2050
 F 0 "R27" V 8750 2250 50  0000 C CNN
-F 1 "330E" V 8700 2050 50  0000 C CNN
+F 1 "301E" V 8700 2050 50  0000 C CNN
 F 2 "Resistor_SMD:R_1206_3216Metric" V 8630 2050 50  0001 C CNN
-F 3 "~" H 8700 2050 50  0001 C CNN
+F 3 "http://www.farnell.com/datasheets/2310790.pdf?_ga=2.55968109.792852979.1526285019-1651149783.1519657816" H 8700 2050 50  0001 C CNN
+F 4 "2139391" V 8700 2050 50  0001 C CNN "Farnell"
+F 5 "CRCW1206301RFKEA" V 8700 2050 50  0001 C CNN "Manufacturer nr"
 	1    8700 2050
 	0    -1   -1   0
@@
 F 1 "330E" V 8700 2150 50  0000 C CNN
 F 2 "Resistor_SMD:R_1206_3216Metric" V 8630 2150 50  0001 C CNN
-F 3 "~" H 8700 2150 50  0001 C CNN
+F 3 "http://www.farnell.com/datasheets/2310790.pdf?_ga=2.55968109.792852979.1526285019-1651149783.1519657816" H 8700 2150 50  0001 C CNN
+F 4 "1470008" V 8700 2150 50  0001 C CNN "Farnell"
+F 5 "CRCW1206330RFKEA" V 8700 2150 50  0001 C CNN "Manufacturer nr"
 	1    8700 2150
 	0    -1   -1   0
@@
 P 8700 2350
 F 0 "R29" V 8750 2550 50  0000 C CNN
-F 1 "330E" V 8700 2350 50  0000 C CNN
+F 1 "301E" V 8700 2350 50  0000 C CNN
 F 2 "Resistor_SMD:R_1206_3216Metric" V 8630 2350 50  0001 C CNN
-F 3 "~" H 8700 2350 50  0001 C CNN
+F 3 "http://www.farnell.com/datasheets/2310790.pdf?_ga=2.48325984.792852979.1526285019-1651149783.1519657816" H 8700 2350 50  0001 C CNN
+F 4 "2139391" V 8700 2350 50  0001 C CNN "Farnell"
+F 5 "CRCW1206162RFKEA" V 8700 2350 50  0001 C CNN "Manufacturer nr"
 	1    8700 2350
 	0    -1   -1   0
@@
 F 1 "Mounting_Hole" H 6400 7505 50  0000 L CNN
 F 2 "MountingHole:MountingHole_3.7mm_Pad_Via" H 6300 7550 50  0001 C CNN
-F 3 "" H 6300 7550 50  0001 C CNN
+F 3 "-" H 6300 7550 50  0001 C CNN
+F 4 "-" H 6300 7550 50  0001 C CNN "Farnell"
+F 5 "-" H 6300 7550 50  0001 C CNN "Manufacturer nr"
 	1    6300 7550
 	1    0    0    -1
@@
 F 3 "http://www.ti.com/lit/ds/symlink/ref3033.pdf" H 6450 800 50  0001 C CIN
 F 4 "1234684" H 6350 1150 50  0001 C CNN "Farnell"
+F 5 "REF3025AIDBZTG4" H 6350 1150 50  0001 C CNN "Manufacturer nr"
 	1    6350 1150
 	1    0    0    -1
@@
 P 8700 2250
 F 0 "R35" V 8650 2050 50  0000 C CNN
-F 1 "330E" V 8700 2250 50  0000 C CNN
+F 1 "301E" V 8700 2250 50  0000 C CNN
 F 2 "Resistor_SMD:R_1206_3216Metric" V 8630 2250 50  0001 C CNN
-F 3 "~" H 8700 2250 50  0001 C CNN
+F 3 "http://www.farnell.com/datasheets/2310790.pdf?_ga=2.48325984.792852979.1526285019-1651149783.1519657816" H 8700 2250 50  0001 C CNN
+F 4 "2139391" V 8700 2250 50  0001 C CNN "Farnell"
+F 5 "CRCW1206162RFKEA" V 8700 2250 50  0001 C CNN "Manufacturer nr"
 	1    8700 2250
 	0    1    1    0
@@
 F 3 "http://www.ti.com/lit/ds/symlink/lm35.pdf" H 1500 5050 50  0001 C CNN
 F 4 "1469236" H 1500 5050 50  0001 C CNN "Farnell"
+F 5 "LM35DZ/NOPB" H 1500 5050 50  0001 C CNN "Manufacturer nr"
 	1    1500 5050
 	1    0    0    -1
@@
 P 1250 5900
 F 0 "F1" V 1150 5900 50  0000 C CNN
-F 1 "3.0A" V 1350 5900 50  0000 C CNN
+F 1 "2.5A" V 1350 5900 50  0000 C CNN
 F 2 "Fuse:Fuse_Bourns_MF-SM_7.98x5.44mm" H 1300 5700 50  0001 L CNN
-F 3 "~" H 1250 5900 50  0001 C CNN
+F 3 "http://www.farnell.com/datasheets/2038620.pdf?_ga=2.252661071.792852979.1526285019-1651149783.1519657816" H 1250 5900 50  0001 C CNN
+F 4 "9350268" V 1250 5900 50  0001 C CNN "Farnell"
+F 5 "MF-SM250-2" V 1250 5900 50  0001 C CNN "Manufacturer nr"
 	1    1250 5900
 	0    1    1    0
@@
 P 2300 5250
 F 0 "C38" H 2325 5350 50  0000 L CNN
-F 1 "22u" H 2325 5150 50  0000 L CNN
+F 1 "2.2u" H 2325 5150 50  0000 L CNN
 F 2 "Capacitor_SMD:C_1206_3216Metric" H 2338 5100 50  0001 C CNN
 F 3 "" H 2300 5250 50  0001 C CNN
@@
 RD
 Text Notes 9550 2300 0    50   ~ 0
-BL
+GR
 Text Notes 9550 2400 0    50   ~ 0
-BL
+GR
+Text Notes 750  8100 0    50   ~ 0
+SMD Vishay resistors:\nhttp://nl.farnell.com/w/c/passive-components/resistors-fixed-value/chip-smd-resistors?brand=vishay&resistor-case-style=1206-3216-metric-&packaging=each|cuttape&range=inc-in-stock|exc-delivery-surcharge|exc-obs
 $EndSCHEMATC

Commit message: Added new PCB: BackplanePCB Updating TrackAmplifier with new components to go to V2.0 (cheaper)
Parts:
- added C?: 2.2u, Capacitor_SMD:C_1206_3216Metric, symbol TrackAmplifier-rescue:C
- C10, C7: Farnell 2395785 -> 2760738; Manufacturer nr VJ1206Y104KXBAT -> C1206S104K5RACTU
- D1: value LED -> LED GR; footprint LED_SMD:LED_1206_3216Metric -> LED_SMD:LED_0603_1608Metric; Farnell 1581232 -> 2426215; Manufacturer nr MCL-S250GC -> KPH-1608SGC
- D2: value LED -> LED YE; footprint LED_SMD:LED_1206_3216Metric -> LED_SMD:LED_0603_1608Metric; Farnell 1581231 -> 2426218; Manufacturer nr MCL-S250YC -> KPH-1608YC
- D3: value LED -> LED RD; footprint LED_SMD:LED_1206_3216Metric -> LED_SMD:LED_0603_1608Metric; Farnell 1581229 -> 2426211; Manufacturer nr MCL-S250SRC -> KPH-1608EC
- D4, D8: value LED -> LED BL; footprint LED_SMD:LED_1206_3216Metric -> LED_SMD:LED_0603_1608Metric; Farnell 1581233 -> 2426212; Manufacturer nr MCL-S250SBLC -> KPH-1608QBC-D
- F1: footprint Fuse:Fuse_Bourns_MF-SM_7.98x5.44mm -> Fuse:Fuse_2920_7451Metric; Farnell 9350268 -> 2834923; Manufacturer nr MF-SM250-2 -> 0ZCF0250FF2C
- U10: value REF3025 -> MCP1525; Farnell 1234684 -> 9758500; Manufacturer nr REF3025AIDBZTG4 -> MCP1525T-I/TT
- U11: value LM35-LP -> MCP9701A-E/TO; Farnell 1469236 -> 1439484; Manufacturer nr LM35DZ/NOPB -> MCP9701-E/TO
- U3: value LM78M05_TO252 -> L78M05CDT-1-TO-251-3; footprint Package_TO_SOT_SMD:TO-252-2 -> Package_TO_SOT_THT:TO-251-3-1EP_Horizontal_TabDown; Farnell 2854542 -> 1077155; Manufacturer nr LM78M05CDTX/NOPB -> L78M05CDT-1
Connections:
- wire segments 423 -> 424
Other:
- note added: "2.0V"
- note added: "2.1V"
- note added: "2.2V"
- note added: "3.3V"
- note removed: "GR"
- note removed: "RD"
- note removed: "YE"

Commit message: New BackplanePCB_solder.pro for new sub-d PCB version instead of solder.
Other:
- note added: "length pcb = 104.7mm\nwidth pcb = 52mm\nheart conn to far pcb edge = 35mm\n\nConnector heart distance vertical = 75mm horizontal 50mm\nConnector plate = 39.3mm\nSpace between connector plates = 35.4mm"
- note removed: "length pcb = 104.7mm\nwidth pcb = 52mm\nheart conn to far pcb edge = 35mm\n\nConnector heart distance = 75mm\nConnector plate = 39.3mm\nSpace between connector plates = 35.4mm"
Changed lines of the file:
@@
 	1600 800  1650 800
 Text Notes 7550 7100 0    50   ~ 0
-length pcb = 104.7mm\nwidth pcb = 52mm\nheart conn to far pcb edge = 35mm\n\nConnector heart distance = 75mm\nConnector plate = 39.3mm\nSpace between connector plates = 35.4mm
+length pcb = 104.7mm\nwidth pcb = 52mm\nheart conn to far pcb edge = 35mm\n\nConnector heart distance vertical = 75mm horizontal 50mm\nConnector plate = 39.3mm\nSpace between connector plates = 35.4mm
 $Comp
 L Mechanical:Mounting_Hole MK1
