File: KiCad/TrackAmplifier/TrackAmplifier_LMD18200_up_right.kicad_pcb (KiCad board)
At the start: 2 copper layers, 105 x 70 mm, 99 parts, among them J1 DB15_Male_MountingHoles, J2 Conn_01x06, Q1 2N7002, U1 ST485EBDR, U10 REF3025, U11 LM35-LP, U2 ST485EBDR, U3 LM78M05_TO252, U4 LMD18200, U5 ST485EBDR, U6 ST485EBDR, U7 INA326, U8 INA326, U9 PIC16F18854-SO

Commit message: Updated schematic and pcb.
Parts:
- removed the REF** at (56.4, 57.8)
- added R17: 0.2E, Resistor_THT:R_Axial_DIN0411_L9.9mm_D3.6mm_P12.70mm_Horizontal, F.Cu at (120.1, 117.2)
- added R38: 0.2E, Resistor_THT:R_Axial_DIN0411_L9.9mm_D3.6mm_P12.70mm_Horizontal, F.Cu at (103.1, 112.9)
- added R39: 0.2E, Resistor_THT:R_Axial_DIN0411_L9.9mm_D3.6mm_P12.70mm_Horizontal, F.Cu at (103.1, 117.2)
- added REF**: CE-Logo_11.2x8mm_SilkScreen, Symbol:CE-Logo_11.2x8mm_SilkScreen, F.Cu at (56.4, 57.1)
- J2: footprint Connector_PinHeader_2.54mm:PinHeader_1x06_P2.54mm_Vertical -> Connector_PinHeader_2.54mm:PinHeader_1x06_P2.54mm_Horizontal; moved to B.Cu
- R16: value 0.02 -> 0.2E; footprint Resistor_SMD:R_Shunt_2512_6332Metric_0.005-0.2 -> Resistor_THT:R_Axial_DIN0411_L9.9mm_D3.6mm_P12.70mm_Horizontal
- moved R16 15.8 mm to (120.1, 112.9)
- moved C19 2.54 mm to (105.9, 100.3)
- moved C20 2.54 mm to (108.4, 100.3)
- moved C21 2.54 mm to (112.2, 105.4)
- moved C22 2.54 mm to (111.0, 100.3)
- moved C23 2.54 mm to (91.9, 100.3)
- moved C24 2.54 mm to (94.5, 100.3)
- moved C25 2.54 mm to (100.8, 105.4)
- moved C28 2.54 mm to (97.0, 100.3)
- moved R12 2.54 mm to (103.3, 100.3)
- moved R13 2.54 mm to (105.9, 105.4)
- moved R15 2.54 mm to (114.8, 105.4)
- moved R18 2.54 mm to (113.5, 100.3)
- moved R19 2.54 mm to (89.4, 100.3)
- moved R20 2.54 mm to (91.9, 105.4)
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Connections:
- C17 pad 2: PWM1 -> OCC1
- FL1 pad 1: Net-(FL1-Pad1) -> OCC2
- R16 pad 1: PWM1 -> OCC1
- R16 pad 2: OCC1 -> Net-(R16-Pad2)
- U4 pad 2: PWM1 -> OCC1
- U7 pad 3: PWM1 -> OCC1
