File: KiCad/TrackAmplifier/TrackAmplifier.kicad_pcb (KiCad board)
At the start: 2 copper layers, 105 x 70 mm, 108 parts, among them J1 DB15_Male_MountingHoles, J2 Conn_01x06, Q1 2N7002, U1 ST485EBDR, U10 REF3025, U11 LM35-LP, U2 ST485EBDR, U3 LM78M05_TO252, U4 LMD18200, U5 ST485EBDR, U6 ST485EBDR, U7 INA326, U8 INA326, U9 PIC16F18854-SO

Commit message: Proto TrackAmplifier done!
Parts:
- added C38: 22u, Capacitor_SMD:C_1206_3216Metric, F.Cu at (109.9, 96.5)
- moved R37 1.28 mm to (115.5, 96.5)
- moved REF** 1.02 mm to (114.5, 79.2)
- moved R38 1.02 mm to (93.2, 82.5)
- moved REF** 0.71 mm to (57.0, 112.2)
- moved REF** 0.50 mm to (56.8, 57.5)
Connections:
- U9 pad 3: Net-(R38-Pad2) -> OCC
- U9 pad 5: OCC -> Net-(R38-Pad2)
Routing:
- net GND: track 235.4 -> 270.0 mm, vias 37 -> 61
- net THFLG: track 86.1 -> 62.3 mm, vias 4 -> 2
- net GNDD: track 12.9 -> 26.4 mm
- net TX_ENA: track 44.1 -> 37.0 mm
- net Net-(R26-Pad1): track 51.9 -> 45.1 mm
- net Net-(R29-Pad1): track 49.3 -> 44.0 mm
- net +5V: track 288.0 -> 283.0 mm
- net Net-(R35-Pad2): track 48.2 -> 43.4 mm
- net Net-(R28-Pad1): track 48.4 -> 44.0 mm
- net Net-(R27-Pad1): track 48.5 -> 44.6 mm
- net OCC1: track 17.2 -> 21.1 mm
- net ICSPCLK: track 55.4 -> 51.7 mm
- net OCC: track 26.5 -> 29.4 mm, vias 2 -> 4
- net ICSPDAT: track 51.3 -> 48.9 mm
- net RST: track 56.8 -> 58.2 mm
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Other:
- board text added: "*"
- board text added: "**"
- board text added: "***"
- board text added: "****"
- board text added: "*****"
- board text added: "*****MF-SM_7.98x5.44mm"
- board text added: "****LM78M05_TO252"
- board text added: "***2N7002"
- board text added: "**REF3025"
- board text added: "*ST485 EBDR"
- board text added: "1"
- board text added: "10"
- board text added: "11"
- board text added: "15"
- board text added: "2"
- board text added: "8"
- board text added: "9"
- board text added: "C17"
- board text added: "C18"
- board text added: "C8"
- board text added: "C9"
- board text added: "EPCOS B82722A2202N001"
- board text added: "ICSP"
- board text added: "INA 326"
- board text added: "J1"
- board text added: "LM35"
- board text added: "LMD18200"
- board text added: "PIC16F18854"
- board text added: "WSK2512"
