File: KiCad/BackplanePCB_solder/BackplanePCB_solder.sch (KiCad schematic (older format))
At the start: 54 parts, among them J1 PowerBug_GND, J10 Conn_02x05_Odd_Even, J11 DB15_Female_MountingHoles, J12 DB15_Female_MountingHoles, J13 DB15_Female_MountingHoles, J14 DB15_Female_MountingHoles, J15 DB15_Female_MountingHoles, J16 Conn_01x03, J17 Conn_01x03, J18 Conn_01x03, J19 Conn_01x03, J2 Conn_01x03, J20 Conn_01x03, J21 Conn_01x03, J22 Conn_01x03, J23 Conn_01x03, J24 Conn_01x03, J25 Conn_01x03, J3 PowerBug+17V, J4 Conn_02x05_Odd_Even, J5 DB15_Female_MountingHoles, J6 DB15_Female_MountingHoles, J7 DB15_Female_MountingHoles, J8 DB15_Female_MountingHoles, J9 DB15_Female_MountingHoles

Commit message: updated with bias resistors.
Parts:
- added R25: 4k, Resistor_THT:R_Axial_DIN0207_L6.3mm_D2.5mm_P7.62mm_Horizontal, symbol Device:R
- added R26: 1k, Resistor_THT:R_Axial_DIN0207_L6.3mm_D2.5mm_P7.62mm_Horizontal, symbol Device:R
Connections:
- wire segments 335 -> 339
Other:
- note added: "Bus pre-load, to be soldered\nonly on 1 place for the whole\nbus!"
Changed lines of the file:
@@
 Entry Wire Line
 	800  6400 900  6500
-Wire Wire Line
-	900  6500 1300 6500
 Text Label 1100 6500 0    50   ~ 0
 +5V
@@
 Entry Wire Line
 	2550 6650 2650 6550
-Wire Wire Line
-	2550 6650 1700 6650
 Wire Wire Line
 	1700 6650 1700 6500
@@
 Wire Wire Line
 	6150 900  6150 950
-Wire Bus Line
-	800  6050 800  6400
+Wire Wire Line
+	900  6500 1300 6500
+Wire Wire Line
+	1700 6650 2550 6650
+$Comp
+L Device:R R25
+U 1 1 5B4410A9
+P 1450 6750
+F 0 "R25" V 1530 6750 50  0000 C CNN
+F 1 "4k" V 1450 6750 50  0000 C CNN
+F 2 "Resistor_THT:R_Axial_DIN0207_L6.3mm_D2.5mm_P7.62mm_Horizontal" V 1380 6750 50  0001 C CNN
+F 3 "~" H 1450 6750 50  0001 C CNN
+	1    1450 6750
+	0    1    1    0
+$EndComp
+$Comp
+L Device:R R26
+U 1 1 5B44116E
+P 1450 6950
+F 0 "R26" V 1530 6950 50  0000 C CNN
+F 1 "1k" V 1450 6950 50  0000 C CNN
+F 2 "Resistor_THT:R_Axial_DIN0207_L6.3mm_D2.5mm_P7.62mm_Horizontal" V 1380 6950 50  0001 C CNN
+F 3 "~" H 1450 6950 50  0001 C CNN
+	1    1450 6950
+	0    1    1    0
+$EndComp
+Entry Wire Line
+	2550 6750 2650 6650
+Entry Wire Line
+	800  6650 900  6750
+Text Label 1100 6950 0    50   ~ 0
+GND
+Text Label 1100 6750 0    50   ~ 0
++5V
+Text Label 2200 6950 0    50   ~ 0
+RX_B
+Text Label 2200 6750 0    50   ~ 0
+RX_A
+Entry Wire Line
+	800  6850 900  6950
+Entry Wire Line
+	2550 6950 2650 6850
+Wire Wire Line
+	900  6750 1300 6750
+Wire Wire Line
+	900  6950 1300 6950
+Wire Wire Line
+	1600 6750 2550 6750
+Wire Wire Line
+	1600 6950 2550 6950
 Wire Bus Line
 	5900 6050 5900 6550
 Wire Bus Line
-	2650 6050 2650 6550
+	800  6050 800  6900
 Wire Bus Line
 	3050 6050 3050 7550
@@
 	4950 6050 4950 7550
 Wire Bus Line
+	2650 6050 2650 7050
+Wire Bus Line
 	800  3750 800  6050
 Wire Bus Line
@@
 Wire Bus Line
 	2650 3750 2650 5800
+Text Notes 1050 7300 0    50   ~ 0
+Bus pre-load, to be soldered\nonly on 1 place for the whole\nbus!
 $EndSCHEMATC
