File: KiCad/TrackAmplifier2/TrackAmplifier.sch (KiCad schematic (older format))
At the start: 107 parts, among them J1 DB15_Male_MountingHoles, J2 Conn_01x06, Q1 BVSS123LT1G, U1 ST485EBDR, U10 MCP1525, U11 MCP9701A-E/TO, U2 ST485EBDR, U3 L78M05CDT-1-TO-251-3, U4 LMD18200, U5 ST485EBDR, U6 ST485EBDR, U7 INA326, U8 INA180A4, U9 PIC16F18854-SO

Commit message: Changed reset diode to resistor
Parts:
- removed D7: 1n4148, Diode_SMD:D_1206_3216Metric, symbol Device:D
- added R?: 470E, Resistor_SMD:R_1206_3216Metric, symbol Device:R
Changed lines of the file:
@@
 Wire Wire Line
 	3400 2000 3400 2100
-$Comp
-L Device:D D7
-U 1 1 5B3F6022
-P 10100 3500
-F 0 "D7" H 10100 3600 50  0000 C CNN
-F 1 "1n4148" H 10100 3400 50  0000 C CNN
-F 2 "Diode_SMD:D_1206_3216Metric" H 10100 3500 50  0001 C CNN
-F 3 "http://www.farnell.com/datasheets/2182681.pdf?_ga=2.208013010.1588585681.1526323724-1626853455.1515011571" H 10100 3500 50  0001 C CNN
-F 4 "2677464" H 10100 3500 50  0001 C CNN "Farnell"
-	1    10100 3500
-	-1   0    0    1
-$EndComp
 Text GLabel 10600 3500 2    50   Output ~ 0
 ~MCLR
@@
 Wire Wire Line
 	6950 4250 7050 4250
+$Comp
+L Device:R R?
+U 1 1 5B86EF97
+P 10100 3500
+F 0 "R?" V 10180 3500 50  0000 C CNN
+F 1 "470E" V 10100 3500 50  0000 C CNN
+F 2 "Resistor_SMD:R_1206_3216Metric" V 10030 3500 50  0001 C CNN
+F 3 "~" H 10100 3500 50  0001 C CNN
+	1    10100 3500
+	0    1    1    0
+$EndComp
 $EndSCHEMATC
