File: KiCad/TrackAmplifier2/TrackAmplifier.sch (KiCad schematic (older format))
At the start: 107 parts, among them J1 DB15_Male_MountingHoles, J2 Conn_01x06, Q1 BVSS123LT1G, U1 ST485EBDR, U10 MCP1525, U11 MCP9701A-E/TO, U2 ST485EBDR, U3 L78M05CDT-1-TO-251-3, U4 LMD18200, U5 ST485EBDR, U6 ST485EBDR, U7 INA326, U8 INA180A4, U9 PIC16F18854-SO

Commit message: Updating new schematic TrackAmplifier2 and added pdf's
Parts:
- added C40: 2.2u, Capacitor_SMD:C_1206_3216Metric, symbol TrackAmplifier-rescue:C
Connections:
- wire segments 413 -> 417
Other:
- note added: "Output capacitance on REF required between 1 and 10 uF"
Changed lines of the file:
@@
 	10700 4250 10700 4450
-$Comp
-L Amplifier_Instrumentation:INA326 U7
-U 1 1 5B58EFF0
-P 4950 1750
-F 0 "U7" H 5100 1875 50  0000 L CNN
-F 1 "INA326" H 5100 1625 50  0000 L CNN
-F 2 "Package_SO:MSOP-8_3x3mm_P0.65mm" H 4950 1750 50  0001 L CNN
-F 3 "http://www.ti.com/lit/ds/symlink/ina326.pdf" H 5050 1750 50  0001 C CNN
-F 4 "2764750" H 4950 1750 50  0001 C CNN "Farnell"
-F 5 "INA326EA/2K5" H 4950 1750 50  0001 C CNN "Manufacturer nr"
-	1    4950 1750
-	1    0    0    -1
-$EndComp
 $Comp
 L Device:EMI_Filter_CommonMode FL1
@@
 L TrackAmplifier-rescue:C C25
 U 1 1 5BAED16E
-P 5350 4800
-F 0 "C25" H 5375 4900 50  0000 L CNN
-F 1 "np" H 5375 4700 50  0000 L CNN
-F 2 "Capacitor_SMD:C_1206_3216Metric" H 5388 4650 50  0001 C CNN
-F 3 "" H 5350 4800 50  0001 C CNN
-	1    5350 4800
+P 4600 2800
+F 0 "C25" H 4625 2900 50  0000 L CNN
+F 1 "np" H 4625 2700 50  0000 L CNN
+F 2 "Capacitor_SMD:C_1206_3216Metric" H 4638 2650 50  0001 C CNN
+F 3 "" H 4600 2800 50  0001 C CNN
+	1    4600 2800
 	-1   0    0    1
 $EndComp
@@
 Connection ~ 5500 1450
 Wire Wire Line
-	6750 1150 6650 1150
+	6750 1150 6700 1150
 Text GLabel 6650 1550 0    50   Output ~ 0
 VREF
@@
 L Device:R R21
 U 1 1 5BAED14E
-P 5450 4500
-F 0 "R21" V 5530 4500 50  0000 C CNN
-F 1 "5M11" V 5450 4500 50  0000 C CNN
-F 2 "Resistor_SMD:R_1206_3216Metric" V 5380 4500 50  0001 C CNN
-F 3 "http://www.farnell.com/datasheets/2310790.pdf?_ga=2.154944504.1588585681.1526323724-1626853455.1515011571" H 5450 4500 50  0001 C CNN
-F 4 "2139776" V 5450 4500 50  0001 C CNN "Farnell"
-F 5 "CRCW12065M11FKEA" V 5450 4500 50  0001 C CNN "Manufacturer nr"
-	1    5450 4500
+P 4700 2500
+F 0 "R21" V 4780 2500 50  0000 C CNN
+F 1 "5M11" V 4700 2500 50  0000 C CNN
+F 2 "Resistor_SMD:R_1206_3216Metric" V 4630 2500 50  0001 C CNN
+F 3 "http://www.farnell.com/datasheets/2310790.pdf?_ga=2.154944504.1588585681.1526323724-1626853455.1515011571" H 4700 2500 50  0001 C CNN
+F 4 "2139776" V 4700 2500 50  0001 C CNN "Farnell"
+F 5 "CRCW12065M11FKEA" V 4700 2500 50  0001 C CNN "Manufacturer nr"
+	1    4700 2500
 	0    1    1    0
 $EndComp
@@
 L Device:R R20
 U 1 1 5BAED147
-P 5400 4250
-F 0 "R20" V 5480 4250 50  0000 C CNN
-F 1 "2k00" V 5400 4250 50  0000 C CNN
-F 2 "Resistor_SMD:R_1206_3216Metric" V 5330 4250 50  0001 C CNN
-F 3 "http://www.farnell.com/datasheets/2310790.pdf?_ga=2.246418116.1588585681.1526323724-1626853455.1515011571" H 5400 4250 50  0001 C CNN
-F 4 "1469985" V 5400 4250 50  0001 C CNN "Farnell"
-F 5 "CRCW12062K00FKEA" V 5400 4250 50  0001 C CNN "Manufacturer nr"
-	1    5400 4250
+P 4650 2250
+F 0 "R20" V 4730 2250 50  0000 C CNN
+F 1 "2k00" V 4650 2250 50  0000 C CNN
+F 2 "Resistor_SMD:R_1206_3216Metric" V 4580 2250 50  0001 C CNN
+F 3 "http://www.farnell.com/datasheets/2310790.pdf?_ga=2.246418116.1588585681.1526323724-1626853455.1515011571" H 4650 2250 50  0001 C CNN
+F 4 "1469985" V 4650 2250 50  0001 C CNN "Farnell"
+F 5 "CRCW12062K00FKEA" V 4650 2250 50  0001 C CNN "Manufacturer nr"
+	1    4650 2250
 	1    0    0    -1
 $EndComp
@@
 Wire Wire Line
 	6950 4250 7050 4250
+$Comp
+L TrackAmplifier-rescue:C C40
+U 1 1 5B2B6918
+P 6950 1200
+F 0 "C40" H 6975 1300 50  0000 L CNN
+F 1 "2.2u" H 6975 1100 50  0000 L CNN
+F 2 "Capacitor_SMD:C_1206_3216Metric" H 6988 1050 50  0001 C CNN
+F 3 "" H 6950 1200 50  0001 C CNN
+	1    6950 1200
+	-1   0    0    1
+$EndComp
+Wire Wire Line
+	6950 1050 6700 1050
+Wire Wire Line
+	6700 1050 6700 1150
+Connection ~ 6700 1150
+Wire Wire Line
+	6700 1150 6650 1150
+Wire Wire Line
+	6950 1350 7200 1350
+$Comp
+L Amplifier_Instrumentation:INA326 U7
+U 1 1 5B58EFF0
+P 4950 1750
+F 0 "U7" H 5100 1875 50  0000 L CNN
+F 1 "INA326" H 5100 1625 50  0000 L CNN
+F 2 "Package_SO:MSOP-8_3x3mm_P0.65mm" H 4950 1750 50  0001 L CNN
+F 3 "http://www.ti.com/lit/ds/symlink/ina326.pdf" H 5050 1750 50  0001 C CNN
+F 4 "2764750" H 4950 1750 50  0001 C CNN "Farnell"
+F 5 "INA326EA/2K5" H 4950 1750 50  0001 C CNN "Manufacturer nr"
+	1    4950 1750
+	1    0    0    -1
+$EndComp
+Text Notes 5350 650  0    50   ~ 0
+Output capacitance on REF required between 1 and 10 uF
 $EndSCHEMATC

Commit message: Updating design according to findings on proto (LEFT  config). Still some spces between sub -d screws is NOK.
Parts:
- Q1: value BVSS123LT1G -> NTR5103NT1G; Farnell 2727944 -> 2724423
- U8: value INA180A4 -> INA2180A4; Farnell 2761899 -> 2842970; Manufacturer nr INA180A4IDBVT -> INA2180A4IDBVT
- U9: Farnell grote versie PIC (none) -> 2564169
Changed lines of the file:
@@
 F 4 "2696647" H 7850 2350 50  0001 C CNN "Farnell"
 F 5 "PIC16F18854-I/SO" H 7850 2350 50  0001 C CNN "Manufacturer nr"
+F 6 "2564169" H 7850 2350 50  0001 C CNN "Farnell grote versie PIC"
 	1    7850 2350
 	1    0    0    -1
@@
 P 3300 2300
 F 0 "Q1" H 3500 2375 50  0000 L CNN
-F 1 "BVSS123LT1G" H 3500 2300 50  0000 L CNN
+F 1 "NTR5103NT1G" H 3500 2300 50  0000 L CNN
 F 2 "Package_TO_SOT_SMD:SOT-23" H 3500 2225 50  0001 L CIN
-F 3 "http://www.farnell.com/datasheets/2255231.pdf?_ga=2.44068322.792852979.1526285019-1651149783.1519657816" H 3300 2300 50  0001 L CNN
-F 4 "2727944" H 3300 2300 50  0001 C CNN "Farnell"
+F 3 "http://www.farnell.com/datasheets/2237046.pdf?_ga=2.4452979.1171392300.1539637038-1187106011.1538513614&_gac=1.57490904.1539637038.Cj0KCQjw9ZDeBRD9ARIsAMbAmoZd4avaFcxEjpXB3_KNG_tD__FtzrWWllmA5UwXEEOZiBvxHw6MpjQaAlwNEALw_wcB" H 3300 2300 50  0001 L CNN
+F 4 "2724423" H 3300 2300 50  0001 C CNN "Farnell"
 F 5 "BVSS123LT1G" H 3300 2300 50  0001 C CNN "Manufacturer nr"
 	1    3300 2300
@@
 P 6550 4250
 F 0 "U8" H 6650 4600 50  0000 L CNN
-F 1 "INA180A4" H 6650 4500 50  0000 L CNN
+F 1 "INA2180A4" H 6650 4500 50  0000 L CNN
 F 2 "Package_TO_SOT_SMD:SOT-23-5" H 6600 4000 50  0001 L CNN
 F 3 "http://www.ti.com/lit/ds/symlink/ina138.pdf" H 6550 4255 50  0001 C CNN
-F 4 "2761899" H 6550 4250 50  0001 C CNN "Farnell"
-F 5 "INA180A4IDBVT" H 6550 4250 50  0001 C CNN "Manufacturer nr"
+F 4 "2842970" H 6550 4250 50  0001 C CNN "Farnell"
+F 5 "INA2180A4IDBVT" H 6550 4250 50  0001 C CNN "Manufacturer nr"
 	1    6550 4250
 	1    0    0    -1

Commit message: Revert to working version of commit on 16-10-18
Parts:
- Q1: value NTR5103NT1G -> BVSS123LT1G; Farnell 2724423 -> 2727944
- U8: value INA2180A4 -> INA180A4; Farnell 2842970 -> 2761899; Manufacturer nr INA2180A4IDBVT -> INA180A4IDBVT
- U9: Farnell grote versie PIC 2564169 -> (none)
Changed lines of the file:
@@
 F 4 "2696647" H 7850 2350 50  0001 C CNN "Farnell"
 F 5 "PIC16F18854-I/SO" H 7850 2350 50  0001 C CNN "Manufacturer nr"
-F 6 "2564169" H 7850 2350 50  0001 C CNN "Farnell grote versie PIC"
 	1    7850 2350
 	1    0    0    -1
@@
 P 3300 2300
 F 0 "Q1" H 3500 2375 50  0000 L CNN
-F 1 "NTR5103NT1G" H 3500 2300 50  0000 L CNN
+F 1 "BVSS123LT1G" H 3500 2300 50  0000 L CNN
 F 2 "Package_TO_SOT_SMD:SOT-23" H 3500 2225 50  0001 L CIN
-F 3 "http://www.farnell.com/datasheets/2237046.pdf?_ga=2.4452979.1171392300.1539637038-1187106011.1538513614&_gac=1.57490904.1539637038.Cj0KCQjw9ZDeBRD9ARIsAMbAmoZd4avaFcxEjpXB3_KNG_tD__FtzrWWllmA5UwXEEOZiBvxHw6MpjQaAlwNEALw_wcB" H 3300 2300 50  0001 L CNN
-F 4 "2724423" H 3300 2300 50  0001 C CNN "Farnell"
+F 3 "http://www.farnell.com/datasheets/2255231.pdf?_ga=2.44068322.792852979.1526285019-1651149783.1519657816" H 3300 2300 50  0001 L CNN
+F 4 "2727944" H 3300 2300 50  0001 C CNN "Farnell"
 F 5 "BVSS123LT1G" H 3300 2300 50  0001 C CNN "Manufacturer nr"
 	1    3300 2300
@@
 P 6550 4250
 F 0 "U8" H 6650 4600 50  0000 L CNN
-F 1 "INA2180A4" H 6650 4500 50  0000 L CNN
+F 1 "INA180A4" H 6650 4500 50  0000 L CNN
 F 2 "Package_TO_SOT_SMD:SOT-23-5" H 6600 4000 50  0001 L CNN
 F 3 "http://www.ti.com/lit/ds/symlink/ina138.pdf" H 6550 4255 50  0001 C CNN
-F 4 "2842970" H 6550 4250 50  0001 C CNN "Farnell"
-F 5 "INA2180A4IDBVT" H 6550 4250 50  0001 C CNN "Manufacturer nr"
+F 4 "2761899" H 6550 4250 50  0001 C CNN "Farnell"
+F 5 "INA180A4IDBVT" H 6550 4250 50  0001 C CNN "Manufacturer nr"
 	1    6550 4250
 	1    0    0    -1

Commit message: Updates on schematic
Parts:
- removed D7: 1n4148, Diode_SMD:D_1206_3216Metric, symbol Device:D
- added R? (x2): 470, Resistor_SMD:R_1206_3216Metric, symbol Device:R
- R33: value 402k -> 470
Connections:
- wire segments 417 -> 419
Changed lines of the file:
@@
 Wire Wire Line
 	8550 1850 8350 1850
-Text GLabel 10600 3350 2    50   Input ~ 0
+Text GLabel 10950 3350 2    50   Input ~ 0
 VPP
 Text GLabel 10600 3650 2    50   Output ~ 0
@@
 Wire Wire Line
 	3400 2000 3400 2100
-$Comp
-L Device:D D7
-U 1 1 5B3F6022
-P 10100 3500
-F 0 "D7" H 10100 3600 50  0000 C CNN
-F 1 "1n4148" H 10100 3400 50  0000 C CNN
-F 2 "Diode_SMD:D_1206_3216Metric" H 10100 3500 50  0001 C CNN
-F 3 "http://www.farnell.com/datasheets/2182681.pdf?_ga=2.208013010.1588585681.1526323724-1626853455.1515011571" H 10100 3500 50  0001 C CNN
-F 4 "2677464" H 10100 3500 50  0001 C CNN "Farnell"
-	1    10100 3500
-	-1   0    0    1
-$EndComp
 Text GLabel 10600 3500 2    50   Output ~ 0
 ~MCLR
@@
 Wire Wire Line
 	6800 2550 7350 2550
-Wire Wire Line
-	10600 3350 10450 3350
-Wire Wire Line
-	10450 3350 10450 3500
 Wire Wire Line
 	10450 3500 10600 3500
@@
 	10450 3650 10450 3500
 Connection ~ 10450 3500
-Wire Wire Line
-	10250 3500 10450 3500
-Wire Wire Line
-	9850 3500 9950 3500
 Connection ~ 9850 3500
 Wire Wire Line
@@
 P 9900 950
 F 0 "R33" V 9980 950 50  0000 C CNN
-F 1 "402k" V 9900 950 50  0000 C CNN
+F 1 "470" V 9900 950 50  0000 C CNN
 F 2 "Resistor_SMD:R_1206_3216Metric" V 9830 950 50  0001 C CNN
 F 3 "~" H 9900 950 50  0001 C CNN
@@
 Text Notes 5350 650  0    50   ~ 0
 Output capacitance on REF required between 1 and 10 uF
+$Comp
+L Device:R R?
+U 1 1 5BD7BB41
+P 10150 3500
+F 0 "R?" V 10230 3500 50  0000 C CNN
+F 1 "470" V 10150 3500 50  0000 C CNN
+F 2 "Resistor_SMD:R_1206_3216Metric" V 10080 3500 50  0001 C CNN
+F 3 "~" H 10150 3500 50  0001 C CNN
+	1    10150 3500
+	0    1    1    0
+$EndComp
+Wire Wire Line
+	10000 3500 9850 3500
+Wire Wire Line
+	10300 3500 10350 3500
+$Comp
+L Device:R R?
+U 1 1 5BDD06F3
+P 10600 3350
+F 0 "R?" V 10500 3350 50  0000 C CNN
+F 1 "470" V 10600 3350 50  0000 C CNN
+F 2 "Resistor_SMD:R_1206_3216Metric" V 10530 3350 50  0001 C CNN
+F 3 "~" H 10600 3350 50  0001 C CNN
+	1    10600 3350
+	0    1    1    0
+$EndComp
+Wire Wire Line
+	10750 3350 10950 3350
+Wire Wire Line
+	10450 3350 10350 3350
+Wire Wire Line
+	10350 3350 10350 3500
+Connection ~ 10350 3500
+Wire Wire Line
+	10350 3500 10450 3500
 $EndSCHEMATC

Commit message: updating TrackAmplifier2.sch
Parts:
- removed C21, C25: np, Capacitor_SMD:C_1206_3216Metric, symbol TrackAmplifier-rescue:C
- removed C40: 2.2u, Capacitor_SMD:C_1206_3216Metric, symbol TrackAmplifier-rescue:C
- removed R16: 0.025E, Resistor_SMD:R_Shunt_2512_6332Metric_0.005-0.2, symbol Device:R_Shunt
- removed U7: INA326, Package_SO:MSOP-8_3x3mm_P0.65mm, symbol Amplifier_Instrumentation:INA326
- removed U8: INA180A4, Package_TO_SOT_SMD:SOT-23-5, symbol Amplifier_Current:INA138
- added C21: 470u, Capacitor_THT:CP_Radial_D10.0mm_P5.00mm, symbol Device:CP
- added D11, D12, D7: V8PAL45, Diode_SMD:D_1206_3216Metric, symbol Device:D
- added D13: LED BL ?, LED_SMD:LED_0603_1608Metric, symbol Device:LED
- added D14, D15: 1n4148, Diode_SMD:D_1206_3216Metric, symbol Device:D
- added D?: LED BL OCC, LED_SMD:LED_0603_1608Metric, symbol Device:LED
- added R16: 1k, Resistor_SMD:R_1206_3216Metric, symbol Device:R
- added R41: 50E, Resistor_SMD:R_1206_3216Metric, symbol Device:R
- added R42: 4k75, Resistor_SMD:R_1206_3216Metric, symbol Device:R
- added R43, R?: 301E, Resistor_SMD:R_1206_3216Metric, symbol Device:R
- added U7: MCP6N11, Package_SO:SOIC-8_3.9x4.9mm_P1.27mm, symbol Amplifier_Instrumentation:MCP6N11
- added U8: INA2180, symbol Amplifier_Current:INA2180
- C1, C11, C12, C19, C2, C23, C26, C32, C34, C36, C38, C39, C8: value 2.2u -> 4.7u; Farnell (none) -> 2576764; Manufacturer nr (none) -> C3216X7R1E475M160AC
- C13, C5: value 2.2u -> 4.7u; Farnell 1759451 -> 2576764; Manufacturer nr MC1206F225Z250CT -> C3216X7R1E475M160AC
- C6: Manufacturer nr (none) -> B41858C7477M000
- D1: value LED GR -> LED GR RUN
- D10, D5, D6, D9: Manufacturer nr (none) -> 1N4148W
- D2: value LED YE -> LED YE WAR
- D3: value LED RD -> LED RD ERR
- D4: value LED BL -> LED BL RX
- D8: value LED BL -> LED BL TX
- J1: Farnell 2294292 -> -; Manufacturer nr 182-015-113R531 -> -
- J2: Farnell 3418327 -> -; Manufacturer nr 826629-6 -> -
- Q1: value BVSS123LT1G -> NTR5103NT1G; Farnell 2727944 -> 2724423; Manufacturer nr BVSS123LT1G -> NTR5103NT1G
- R1, R10, R11, R2, R22, R9: value 10E -> 0E
- R12, R19, R34, R37, R5: Farnell (none) -> 1653053; Manufacturer nr (none) -> CRCW120610R0FKEB
- R13: value 402k -> 1k; Farnell 2139646 -> 1653077
- R14: value 4k7 -> 1k; Farnell (none) -> 1653077
- R15: value 39k -> 100k
- R20: value 2k00 -> 9k10
- R21: value 5M11 -> 9k10
- R30: Farnell (none) -> 1653077
- R38: value 10E -> 1k; Farnell (none) -> 1653077; Manufacturer nr (none) -> CRCW12065M11FKEA
- gave numbers to parts that had none: 2
Connections:
- net labels removed: +15V
- wire segments 419 -> 455
- no-connect marks 4 -> 2
Other:
- moved on the sheet: FL2

Commit message: Added Farnell.py to process the BOM in KiCad to Farnell order list.
Parts:
- C10, C7: Farnell 2760738 -> 1759361; Manufacturer nr C1206S104K5RACTU -> MC1206B104K500CT
- C14, C15, C20, C22, C24, C27, C28, C29, C3, C30, C31, C33, C35, C37, C4, C9: Farnell (none) -> 1759361; Manufacturer nr (none) -> MC1206B104K500CT
- D1: value LED GR RUN -> LED GR
- D13: footprint LED_SMD:LED_0603_1608Metric -> -; Farnell 2426212 -> (none); Manufacturer nr KPH-1608QBC-D -> -
- D16: renamed from D?; value LED BL OCC -> LED BL
- D2: value LED YE WAR -> LED YE
- D3: value LED RD ERR -> LED RD
- D4: value LED BL RX -> LED GR; Farnell 2426212 -> 2426215; Manufacturer nr KPH-1608QBC-D -> KPH-1608SGC
- D8: value LED BL TX -> LED GR; Farnell 2426212 -> 2426215; Manufacturer nr KPH-1608QBC-D -> KPH-1608SGC
- FL1, FL2: Farnell 1223076 -> (none)
- J1, J2, MK1: Farnell - -> (none)
- R1, R10, R11, R2, R22, R9: Farnell (none) -> 1100137; Manufacturer nr (none) -> WCR1206-R005JI
- R13: Manufacturer nr CRCW1206402KFKEA -> CRCW12061K00JNEA
- R14, R30: Manufacturer nr (none) -> CRCW12061K00JNEA
- R15: Farnell 2139553 -> 1469975; Manufacturer nr CRCW120639K0FKEA -> CRCW1206100KFKEA
- R16, R38: Manufacturer nr CRCW12065M11FKEA -> CRCW12061K00JNEA
- R17: Farnell 1470015 -> 2695161; Manufacturer nr CRCW12064K99FKEA -> MCWR12X4991FTL
- R18, R23: Farnell (none) -> 2616760; Manufacturer nr (none) -> CRCW1206100RJNEA
- R20: Farnell 1469985 -> 1100217; Manufacturer nr CRCW12062K00FKEA -> WCR1206-9K1FI
- R21: Farnell 2139776 -> 1100217; Manufacturer nr CRCW12065M11FKEA -> WCR1206-9K1FI
- R25, R4, R6, R7: value 4k7 -> 4k75; Farnell (none) -> 1470014; Manufacturer nr (none) -> CRCW12064K75FKEA
- R29, R35: Manufacturer nr CRCW1206162RFKEA -> CRCW1206301RFKEA
- R31: value 100K -> 100k
- R32: Farnell (none) -> 2079007; Manufacturer nr (none) -> ASC1206-10KFT5
- R33, R44, R45: Farnell (none) -> 2078999; Manufacturer nr (none) -> ASC1206-470RFT5
- R36: Farnell 1469970 -> 2079007; Manufacturer nr CRCW120610K0FKEA -> ASC1206-10KFT5
- R40: value 4k7 -> 4k75
- R41: value 50E -> 47E; Farnell 1470015 -> 2078992; Manufacturer nr CRCW12064K99FKEA -> ASC1206-47RFT5
- R42: Farnell 1469985 -> 1470014; Manufacturer nr CRCW12062K00FKEA -> CRCW12064K75FKEA
- U4: Farnell 1468979 -> (none)
- U8: footprint (none) -> Package_SO:VSSOP-8_3.0x3.0mm_P0.65mm
- gave numbers to parts that had none: 1

Commit message: Updated schematic with PIC18F25K40 and R47. Updated shopping csv file.
Parts:
- added R47: NP, Resistor_SMD:R_1206_3216Metric, symbol Device:R
- R8: value 100E -> 1k; Farnell 2616760 -> 1653077; Manufacturer nr CRCW1206100RJNEA -> CRCW12061K00JNEA
- U9: value PIC16F18854-SO -> PIC18F25K40; Farnell 2696647 -> 2564200
Connections:
- wire segments 455 -> 457
Other:
- note added: "Disconnected receiver inputs\nor idle bus will have RO high.\nInvert for continuous uController reset\nIn order to flash standalone connect\nthe R47 pads"
- note removed: "Disconnected receiver inputs\nor idle bus will have RO high.\nInvert for continuous uController reset"
Changed lines of the file:
@@
 P 7850 2350
 F 0 "U9" H 7500 3100 50  0000 C CNN
-F 1 "PIC16F18854-SO" H 8250 3100 50  0000 C CNN
+F 1 "PIC18F25K40" H 8250 3100 50  0000 C CNN
 F 2 "Package_SO:SOIC-28W_7.5x17.9mm_P1.27mm" H 7850 1250 50  0001 C CNN
-F 3 "http://ww1.microchip.com/downloads/en/DeviceDoc/PIC16(L)F18854%20Data%20Sheet_DS40001826C.pdf" H 8150 1750 50  0001 C CNN
-F 4 "2696647" H 7850 2350 50  0001 C CNN "Farnell"
+F 3 "http://ww1.microchip.com/downloads/en/DeviceDoc/PIC18(L)F24_25K40%2028-Pin%20Low-Power%20High-Performance%20MCU%20with%20XLP%20Technology%2040001843D.pdf" H 8150 1750 50  0001 C CNN
+F 4 "2564200" H 7850 2350 50  0001 C CNN "Farnell"
 F 5 "PIC16F18854-I/SO" H 7850 2350 50  0001 C CNN "Manufacturer nr"
 	1    7850 2350
@@
 P 2450 2300
 F 0 "R8" V 2530 2300 50  0000 C CNN
-F 1 "100E" V 2450 2300 50  0000 C CNN
+F 1 "1k" V 2450 2300 50  0000 C CNN
 F 2 "Resistor_SMD:R_1206_3216Metric" V 2380 2300 50  0001 C CNN
-F 3 "http://www.farnell.com/datasheets/2310790.pdf?_ga=2.153896696.1588585681.1526323724-1626853455.1515011571" H 2450 2300 50  0001 C CNN
-F 4 "2616760" V 2450 2300 50  0001 C CNN "Farnell"
-F 5 "CRCW1206100RJNEA" V 2450 2300 50  0001 C CNN "Manufacturer nr"
+F 3 "http://www.farnell.com/datasheets/2310790.pdf?_ga=2.210134357.1588585681.1526323724-1626853455.1515011571" H 2450 2300 50  0001 C CNN
+F 4 "1653077" V 2450 2300 50  0001 C CNN "Farnell"
+F 5 "CRCW12061K00JNEA" V 2450 2300 50  0001 C CNN "Manufacturer nr"
 	1    2450 2300
 	0    -1   -1   0
@@
 Text Notes 10050 4050 0    50   ~ 0
 ~MCLR~ Vil = 0.2V Vih = 0.7V\nLVP is possible, HVP only\nwhen "RESET" transceiver \ninput A < B
-Text Notes 2150 1900 0    50   ~ 0
-Disconnected receiver inputs\nor idle bus will have RO high.\nInvert for continuous uController reset
+Text Notes 1100 1850 0    50   ~ 0
+Disconnected receiver inputs\nor idle bus will have RO high.\nInvert for continuous uController reset\nIn order to flash standalone connect\nthe R47 pads
 $Comp
 L power:GNDD #PWR046
@@
 	7400 5100 7000 5100
 Connection ~ 7000 5100
+$Comp
+L Device:R R47
+U 1 1 5C04E09A
+P 2650 2050
+F 0 "R47" V 2730 2050 50  0000 C CNN
+F 1 "NP" V 2650 2050 50  0000 C CNN
+F 2 "Resistor_SMD:R_1206_3216Metric" V 2580 2050 50  0001 C CNN
+F 3 "http://www.farnell.com/datasheets/2331353.pdf?_ga=2.31327414.804204398.1540810031-466615820.1533907205&_gac=1.187361882.1540810769.CjwKCAjw39reBRBJEiwAO1m0OeFHyFqLAwRfo1TyfiEw1u5wgH8YT365nEvQxYyzS_SVx6sHehne4BoC4gYQAvD_BwE" H 2650 2050 50  0001 C CNN
+F 4 "1100137" H 1900 0   50  0001 C CNN "Farnell"
+F 5 "WCR1206-R005JI" H 1900 0   50  0001 C CNN "Manufacturer nr"
+	1    2650 2050
+	-1   0    0    1
+$EndComp
+Wire Wire Line
+	2650 2200 2650 2300
+$Comp
+L power:+5V #PWR07
+U 1 1 5C083150
+P 2650 1850
+F 0 "#PWR07" H 2650 1700 50  0001 C CNN
+F 1 "+5V" H 2650 1990 50  0000 C CNN
+F 2 "" H 2650 1850 50  0001 C CNN
+F 3 "" H 2650 1850 50  0001 C CNN
+	1    2650 1850
+	1    0    0    -1
+$EndComp
+Wire Wire Line
+	2650 1850 2650 1900
 $EndSCHEMATC

Commit message: Updated schematic, cheaper components.
Parts:
- added R48, R49: 1k, Resistor_SMD:R_1206_3216Metric, symbol Device:R
- C1, C11, C12, C13, C19, C2, C23, C26, C32, C34, C36, C38, C39, C5, C8: Farnell 2576764 -> 2320886; Manufacturer nr C3216X7R1E475M160AC -> MC1206B475K250CT
- C10, C14, C15, C20, C22, C24, C27, C28, C29, C3, C30, C31, C33, C35, C37, C4, C7, C9: Farnell 1759361 -> 1414715; Manufacturer nr MC1206B104K500CT -> C1206C104K5RACTU
- C21: footprint Capacitor_THT:CP_Radial_D10.0mm_P5.00mm -> Capacitor_SMD:CP_Elec_6.3x3; Farnell 9451315 -> (none)
- D11, D12, D7: value V8PAL45 -> VS-6ESH06-M3; footprint Diode_SMD:D_1206_3216Metric -> Package_TO_SOT_SMD:TO-277A; Farnell 2425092 -> 2471194; Manufacturer nr V8PAL45-M3/I -> VS-6ESH06-M3/86A
- R12, R19, R3, R34, R37, R5: Farnell 1653053 -> 1100138; Manufacturer nr CRCW120610R0FKEB -> WCR1206-10RFI
- R13, R14, R16, R30, R38, R8: Farnell 1653077 -> 1100192; Manufacturer nr CRCW12061K00JNEA -> WCR1206-1K0FI
- R15, R31: value 100k -> 110k; Farnell 1469975 -> 1100244; Manufacturer nr CRCW1206100KFKEA -> WCR1206-100KFI
- R17: value 4k99 -> 5k1; Manufacturer nr MCWR12X4991FTL -> WCR1206-5K1FI
- R18, R23: Farnell 2616760 -> 1100164; Manufacturer nr CRCW1206100RJNEA -> WCR1206-100RFI
- R24: Farnell 1653122 -> 1100204; Manufacturer nr CRCW12063K30FKEA -> WCR1206-3K3FI
- R25, R4, R40, R42, R6, R7: value 4k75 -> 4k7; Farnell 1470014 -> 1100209; Manufacturer nr CRCW12064K75FKEA -> WCR1206-4K7FI
- R26, R27, R29, R35, R43, R46: value 301E -> 300E; Farnell 2139391 -> 1100176; Manufacturer nr CRCW1206301RFKEA -> WCR1206-300RFI
- R28: value 330E -> 300E; Farnell 1470008 -> 1100176; Manufacturer nr CRCW1206330RFKEA -> WCR1206-300RFI
- R32, R36: Farnell 2079007 -> 1100218; Manufacturer nr ASC1206-10KFT5 -> WCR1206-10KFI
- R33, R44, R45: Farnell 2078999 -> 1100183; Manufacturer nr ASC1206-470RFT5 -> WCR1206-470RFI
- R39: value 1k -> 910R; Farnell 1653077 -> 1100190; Manufacturer nr CRCW12061K00JNEA -> WCR1206-910RFI
- R41: Farnell 2078992 -> 1100156; Manufacturer nr ASC1206-47RFT5 -> WCR1206-47RFI
- R47: Farnell 1100137 -> (none)
- U1, U2, U5, U6: Farnell 1467755 -> (none)
Connections:
- wire segments 457 -> 459
Other:
- note added: "Farnell: 1467755"
- moved on the sheet: FL2
