File: KiCad/TrackAmplifier2/TrackAmplifier.sch (KiCad schematic (older format))
At the start: 121 parts, among them J1 DB15_Male_MountingHoles, J2 Conn_01x06, Q1 NTR5103NT1G, U1 ST485EBDR, U10 MCP1525, U11 MCP9701A-E/TO, U2 ST485EBDR, U3 L78M05CDT-1-TO-251-3, U4 LMD18200, U5 ST485EBDR, U6 ST485EBDR, U7 MCP6N11, U8 INA2180, U9 PIC18F25K40

Commit message: updated schematic and layout, not finished yet. To do: - Update components with real used values
Parts:
- removed R48, R49: 1k, Resistor_SMD:R_1206_3216Metric, symbol Device:R
- D11, D12, D7: symbol Device:D -> Device:D_Schottky_AAK
- D13: footprint - -> LED_SMD:LED_0603_1608Metric
- R47: footprint Resistor_SMD:R_1206_3216Metric -> Resistor_SMD:R_0603_1608Metric; Farnell (none) -> -
- U3: symbol Regulator_Linear:LM78M05_TO252 -> Regulator_Linear:LM78M05_TO251-3
Connections:
- wire segments 459 -> 460

Commit message: Updated schematic according to proto board.
Parts:
- C21: footprint Capacitor_SMD:CP_Elec_6.3x3 -> Capacitor_SMD:CP_Elec_8x10.5
- D1: value LED GR -> LED GR RUN; footprint LED_SMD:LED_0603_1608Metric -> Diode_SMD:LED_0.8x0.8
- D13: footprint LED_SMD:LED_0603_1608Metric -> Diode_SMD:LED_0.8x0.8
- D16: value LED BL -> LED BL OCC; footprint LED_SMD:LED_0603_1608Metric -> Diode_SMD:LED_0.8x0.8
- D2: value LED YE -> LED YE WAR; footprint LED_SMD:LED_0603_1608Metric -> Diode_SMD:LED_0.8x0.8
- D3: value LED RD -> LED RD ERR; footprint LED_SMD:LED_0603_1608Metric -> Diode_SMD:LED_0.8x0.8
- D4: value LED GR -> LED GR RX; footprint LED_SMD:LED_0603_1608Metric -> Diode_SMD:LED_0.8x0.8
- D8: value LED GR -> LED GR TX; footprint LED_SMD:LED_0603_1608Metric -> Diode_SMD:LED_0.8x0.8
- R13: value 1k -> 39k; Farnell 1100192 -> 1100234; Manufacturer nr WCR1206-1K0FI -> WCR1206-39KFI
- R15: value 110k -> 39k; Farnell 1100244 -> 1100234; Manufacturer nr WCR1206-100KFI -> WCR1206-39KFI
- R18: value 100E -> 4k99; Farnell 1100164 -> 2695161; Manufacturer nr WCR1206-100RFI -> MCWR12X4991FTL
- U3: symbol Regulator_Linear:LM78M05_TO251-3 -> TrackAmplifier-rescue:LM78M05_TO251-3-Regulator_Linear
- U7: symbol Amplifier_Instrumentation:MCP6N11 -> TrackAmplifier-rescue:MCP6N11-Amplifier_Instrumentation
- U8: symbol Amplifier_Current:INA2180 -> TrackAmplifier-rescue:INA2180-Amplifier_Current
Other:
- note added: "OR: 4x MAX3468"
- note removed: "Resistor on backplane \nwill determine ID voltage\n\nIf with potmeter:\nFarnell: 1141389"
Changed lines of the file:
@@
 $EndComp
 $Comp
-L Regulator_Linear:LM78M05_TO251-3 U3
+L TrackAmplifier-rescue:LM78M05_TO251-3-Regulator_Linear U3
 U 1 1 5AE1A916
 P 2800 800
@@
 $EndComp
 Connection ~ 9900 1150
-Text Notes 10200 1350 0    50   ~ 0
-Resistor on backplane \nwill determine ID voltage\n\nIf with potmeter:\nFarnell: 1141389
 $Comp
 L Device:R R30
@@
 P 5250 2100
 F 0 "R13" V 5330 2100 50  0000 C CNN
-F 1 "1k" V 5250 2100 50  0000 C CNN
+F 1 "39k" V 5250 2100 50  0000 C CNN
 F 2 "Resistor_SMD:R_1206_3216Metric" V 5180 2100 50  0001 C CNN
 F 3 "http://www.farnell.com/datasheets/2158849.pdf?_ga=2.191239274.13702668.1544197496-523844734.1542029203&_gac=1.245695152.1543322461.EAIaIQobChMIof7Tlcz03gIVkuJ3Ch1UVwqwEAAYASAAEgK8PvD_BwE" H 5250 2100 50  0001 C CNN
-F 4 "1100192" V 5250 2100 50  0001 C CNN "Farnell"
-F 5 "WCR1206-1K0FI" V 5250 2100 50  0001 C CNN "Manufacturer nr"
+F 4 "1100234" V 5250 2100 50  0001 C CNN "Farnell"
+F 5 "WCR1206-39KFI" V 5250 2100 50  0001 C CNN "Manufacturer nr"
 	1    5250 2100
 	0    1    1    0
@@
 P 5250 2300
 F 0 "R15" V 5330 2300 50  0000 C CNN
-F 1 "110k" V 5250 2300 50  0000 C CNN
+F 1 "39k" V 5250 2300 50  0000 C CNN
 F 2 "Resistor_SMD:R_1206_3216Metric" V 5180 2300 50  0001 C CNN
 F 3 "http://www.farnell.com/datasheets/2331353.pdf?_ga=2.264231116.13702668.1544197496-523844734.1542029203&_gac=1.217211554.1543322461.EAIaIQobChMIof7Tlcz03gIVkuJ3Ch1UVwqwEAAYASAAEgK8PvD_BwE" H 5250 2300 50  0001 C CNN
-F 4 "1100244" V 5250 2300 50  0001 C CNN "Farnell"
-F 5 "WCR1206-100KFI" V 5250 2300 50  0001 C CNN "Manufacturer nr"
+F 4 "1100234" V 5250 2300 50  0001 C CNN "Farnell"
+F 5 "WCR1206-39KFI" V 5250 2300 50  0001 C CNN "Manufacturer nr"
 	1    5250 2300
 	0    1    1    0
@@
 P 5650 1750
 F 0 "R18" V 5730 1750 50  0000 C CNN
-F 1 "100E" V 5650 1750 50  0000 C CNN
+F 1 "4k99" V 5650 1750 50  0000 C CNN
 F 2 "Resistor_SMD:R_1206_3216Metric" V 5580 1750 50  0001 C CNN
 F 3 "http://www.farnell.com/datasheets/2158849.pdf?_ga=2.36114656.13702668.1544197496-523844734.1542029203&_gac=1.195831192.1543322461.EAIaIQobChMIof7Tlcz03gIVkuJ3Ch1UVwqwEAAYASAAEgK8PvD_BwE" H 5650 1750 50  0001 C CNN
-F 4 "1100164" H 0   0   50  0001 C CNN "Farnell"
-F 5 "WCR1206-100RFI" H 0   0   50  0001 C CNN "Manufacturer nr"
+F 4 "2695161" H 0   0   50  0001 C CNN "Farnell"
+F 5 "MCWR12X4991FTL" H 0   0   50  0001 C CNN "Manufacturer nr"
 	1    5650 1750
 	0    1    1    0
@@
 P 9150 1950
 F 0 "D1" H 8900 1900 50  0000 C CNN
-F 1 "LED GR" H 8550 1950 50  0000 C CNN
-F 2 "LED_SMD:LED_0603_1608Metric" H 9150 1950 50  0001 C CNN
+F 1 "LED GR RUN" H 8500 1950 50  0000 C CNN
+F 2 "Diode_SMD:LED_0.8x0.8" H 9150 1950 50  0001 C CNN
 F 3 "http://www.farnell.com/datasheets/2045940.pdf?_ga=2.245392706.792852979.1526285019-1651149783.1519657816" H 9150 1950 50  0001 C CNN
 F 4 "2426215" H 9150 1950 50  0001 C CNN "Farnell"
@@
 P 9150 2050
 F 0 "D2" H 8900 2000 50  0000 C CNN
-F 1 "LED YE" H 8550 2050 50  0000 C CNN
-F 2 "LED_SMD:LED_0603_1608Metric" H 9150 2050 50  0001 C CNN
+F 1 "LED YE WAR" H 8500 2050 50  0000 C CNN
+F 2 "Diode_SMD:LED_0.8x0.8" H 9150 2050 50  0001 C CNN
 F 3 "http://www.farnell.com/datasheets/2046217.pdf?_ga=2.214478033.792852979.1526285019-1651149783.1519657816" H 9150 2050 50  0001 C CNN
 F 4 "2426218" H 9150 2050 50  0001 C CNN "Farnell"
@@
 P 9150 2150
 F 0 "D3" H 8900 2100 50  0000 C CNN
-F 1 "LED RD" H 8550 2150 50  0000 C CNN
-F 2 "LED_SMD:LED_0603_1608Metric" H 9150 2150 50  0001 C CNN
+F 1 "LED RD ERR" H 8500 2150 50  0000 C CNN
+F 2 "Diode_SMD:LED_0.8x0.8" H 9150 2150 50  0001 C CNN
 F 3 "http://www.farnell.com/datasheets/2046367.pdf?_ga=2.218710495.792852979.1526285019-1651149783.1519657816" H 9150 2150 50  0001 C CNN
 F 4 "2426211" H 9150 2150 50  0001 C CNN "Farnell"
@@
 P 9150 2250
 F 0 "D4" H 8900 2200 50  0000 C CNN
-F 1 "LED GR" H 8550 2250 50  0000 C CNN
-F 2 "LED_SMD:LED_0603_1608Metric" H 9150 2250 50  0001 C CNN
+F 1 "LED GR RX " H 8500 2250 50  0000 C CNN
+F 2 "Diode_SMD:LED_0.8x0.8" H 9150 2250 50  0001 C CNN
 F 3 "http://www.farnell.com/datasheets/2045940.pdf?_ga=2.245392706.792852979.1526285019-1651149783.1519657816" H 9150 2250 50  0001 C CNN
 F 4 "2426215" H 9150 2250 50  0001 C CNN "Farnell"
@@
 P 9150 2350
 F 0 "D8" H 8900 2300 50  0000 C CNN
-F 1 "LED GR" H 8550 2350 50  0000 C CNN
-F 2 "LED_SMD:LED_0603_1608Metric" H 9150 2350 50  0001 C CNN
+F 1 "LED GR TX " H 8500 2350 50  0000 C CNN
+F 2 "Diode_SMD:LED_0.8x0.8" H 9150 2350 50  0001 C CNN
 F 3 "http://www.farnell.com/datasheets/2045940.pdf?_ga=2.245392706.792852979.1526285019-1651149783.1519657816" H 9150 2350 50  0001 C CNN
 F 4 "2426215" H 9150 2350 50  0001 C CNN "Farnell"
@@
 	10650 2250 10650 2400
 $Comp
-L Amplifier_Current:INA2180 U8
+L TrackAmplifier-rescue:INA2180-Amplifier_Current U8
 U 1 1 5BD5C8E8
 P 6150 3650
@@
 $EndComp
 $Comp
-L Amplifier_Current:INA2180 U8
+L TrackAmplifier-rescue:INA2180-Amplifier_Current U8
 U 2 1 5BD5C9FE
 P 6150 4500
@@
 $EndComp
 $Comp
-L Amplifier_Current:INA2180 U8
+L TrackAmplifier-rescue:INA2180-Amplifier_Current U8
 U 3 1 5BD5CB16
 P 7400 5450
@@
 	4500 2200 4500 1600
 $Comp
-L Amplifier_Instrumentation:MCP6N11 U7
+L TrackAmplifier-rescue:MCP6N11-Amplifier_Instrumentation U7
 U 1 1 5C93942B
 P 4950 1750
@@
 F 0 "D13" H 6400 2800 50  0000 C CNN
 F 1 "LED BL ?" H 6350 3000 50  0000 C CNN
-F 2 "LED_SMD:LED_0603_1608Metric" H 6400 2900 50  0001 C CNN
+F 2 "Diode_SMD:LED_0.8x0.8" H 6400 2900 50  0001 C CNN
 F 3 "-" H 6400 2900 50  0001 C CNN
 F 4 "-" H 6400 2900 50  0001 C CNN "Manufacturer nr"
@@
 F 0 "C21" H 1750 950 50  0000 L CNN
 F 1 "470u" H 1650 1150 50  0000 L CNN
-F 2 "Capacitor_SMD:CP_Elec_6.3x3" H 1988 900 50  0001 C CNN
+F 2 "Capacitor_SMD:CP_Elec_8x10.5" H 1988 900 50  0001 C CNN
 F 3 "" H 1950 1050 50  0001 C CNN
 F 4 "MCGPR35V477M10X21" H 1950 1050 50  0001 C CNN "Manufacturer nr"
@@
 P 6100 2900
 F 0 "D16" H 6100 2800 50  0000 C CNN
-F 1 "LED BL" H 6050 3000 50  0000 C CNN
-F 2 "LED_SMD:LED_0603_1608Metric" H 6100 2900 50  0001 C CNN
+F 1 "LED BL OCC" H 6050 3000 50  0000 C CNN
+F 2 "Diode_SMD:LED_0.8x0.8" H 6100 2900 50  0001 C CNN
 F 3 "http://www.farnell.com/datasheets/2046366.pdf?_ga=2.60295403.792852979.1526285019-1651149783.1519657816" H 6100 2900 50  0001 C CNN
 F 4 "2426212" H 6100 2900 50  0001 C CNN "Farnell"
@@
 Wire Wire Line
 	5200 7200 5300 7200
+Text Notes 3800 3000 0    50   ~ 0
+OR: 4x MAX3468
 $EndSCHEMATC

Commit message: updated schematic, grouped together resistors.
Parts:
- R16, R38: value 1k -> 3k9; Farnell 1100192 -> 1100206; Manufacturer nr WCR1206-1K0FI -> WCR1206-3K9FI
- R17: value 5k1 -> 4k99; Manufacturer nr WCR1206-5K1FI -> MCWR12X4991FTL
- R20, R21: value 9k10 -> 20k; Farnell 1100217 -> 1100226; Manufacturer nr WCR1206-9K1FI -> WCR1206-20KFI
- R25, R4, R40, R42, R6, R7: value 4k7 -> 4k99; Farnell 1100209 -> 2695161; Manufacturer nr WCR1206-4K7FI -> MCWR12X4991FTL
- R31: Farnell 1100244 -> 1100246; Manufacturer nr WCR1206-100KFI -> WCR1206-110KFI
- R39: value 910R -> 1k; Farnell 1100190 -> 1100192; Manufacturer nr WCR1206-910RFI -> WCR1206-1K0FI
Changed lines of the file:
@@
 P 1700 7200
 F 0 "R6" V 1780 7200 50  0000 C CNN
-F 1 "4k7" V 1700 7200 50  0000 C CNN
+F 1 "4k99" V 1700 7200 50  0000 C CNN
 F 2 "Resistor_SMD:R_1206_3216Metric" V 1630 7200 50  0001 C CNN
 F 3 "http://www.farnell.com/datasheets/2158849.pdf?_ga=2.191241066.13702668.1544197496-523844734.1542029203&_gac=1.7619462.1543322461.EAIaIQobChMIof7Tlcz03gIVkuJ3Ch1UVwqwEAAYASAAEgK8PvD_BwE" H 1700 7200 50  0001 C CNN
-F 4 "1100209" H 0   0   50  0001 C CNN "Farnell"
-F 5 "WCR1206-4K7FI" H 0   0   50  0001 C CNN "Manufacturer nr"
+F 4 "2695161" H 0   0   50  0001 C CNN "Farnell"
+F 5 "MCWR12X4991FTL" H 0   0   50  0001 C CNN "Manufacturer nr"
 	1    1700 7200
 	-1   0    0    1
@@
 P 1250 6700
 F 0 "R4" V 1330 6700 50  0000 C CNN
-F 1 "4k7" V 1250 6700 50  0000 C CNN
+F 1 "4k99" V 1250 6700 50  0000 C CNN
 F 2 "Resistor_SMD:R_1206_3216Metric" V 1180 6700 50  0001 C CNN
 F 3 "http://www.farnell.com/datasheets/2158849.pdf?_ga=2.191241066.13702668.1544197496-523844734.1542029203&_gac=1.7619462.1543322461.EAIaIQobChMIof7Tlcz03gIVkuJ3Ch1UVwqwEAAYASAAEgK8PvD_BwE" H 1250 6700 50  0001 C CNN
-F 4 "1100209" H 0   0   50  0001 C CNN "Farnell"
-F 5 "WCR1206-4K7FI" H 0   0   50  0001 C CNN "Manufacturer nr"
+F 4 "2695161" H 0   0   50  0001 C CNN "Farnell"
+F 5 "MCWR12X4991FTL" H 0   0   50  0001 C CNN "Manufacturer nr"
 	1    1250 6700
 	-1   0    0    1
@@
 P 1900 7200
 F 0 "R7" V 1980 7200 50  0000 C CNN
-F 1 "4k7" V 1900 7200 50  0000 C CNN
+F 1 "4k99" V 1900 7200 50  0000 C CNN
 F 2 "Resistor_SMD:R_1206_3216Metric" V 1830 7200 50  0001 C CNN
 F 3 "http://www.farnell.com/datasheets/2158849.pdf?_ga=2.191241066.13702668.1544197496-523844734.1542029203&_gac=1.7619462.1543322461.EAIaIQobChMIof7Tlcz03gIVkuJ3Ch1UVwqwEAAYASAAEgK8PvD_BwE" H 1900 7200 50  0001 C CNN
-F 4 "1100209" H 0   0   50  0001 C CNN "Farnell"
-F 5 "WCR1206-4K7FI" H 0   0   50  0001 C CNN "Manufacturer nr"
+F 4 "2695161" H 0   0   50  0001 C CNN "Farnell"
+F 5 "MCWR12X4991FTL" H 0   0   50  0001 C CNN "Manufacturer nr"
 	1    1900 7200
 	-1   0    0    1
@@
 P 5500 6850
 F 0 "FL1" H 5500 7025 50  0000 C CNN
-F 1 "EMI_Filter_CMode" H 5600 7150 50  0000 C CNN
+F 1 "EMI_Filter_CMode" H 5550 7100 50  0000 C CNN
 F 2 "Inductor_THT:Choke_EPCOS_B82722-A2302-N1-22.3x22.7mm" V 5500 6890 50  0001 C CNN
 F 3 "http://www.farnell.com/datasheets/1860373.pdf?_ga=2.174943842.1588585681.1526323724-1626853455.1515011571" V 5500 6890 50  0001 C CNN
@@
 P 8550 5400
 F 0 "R25" V 8630 5400 50  0000 C CNN
-F 1 "4k7" V 8550 5400 50  0000 C CNN
+F 1 "4k99" V 8550 5400 50  0000 C CNN
 F 2 "Resistor_SMD:R_1206_3216Metric" V 8480 5400 50  0001 C CNN
 F 3 "http://www.farnell.com/datasheets/2158849.pdf?_ga=2.191241066.13702668.1544197496-523844734.1542029203&_gac=1.7619462.1543322461.EAIaIQobChMIof7Tlcz03gIVkuJ3Ch1UVwqwEAAYASAAEgK8PvD_BwE" H 8550 5400 50  0001 C CNN
-F 4 "1100209" H 0   0   50  0001 C CNN "Farnell"
-F 5 "WCR1206-4K7FI" H 0   0   50  0001 C CNN "Manufacturer nr"
+F 4 "2695161" H 0   0   50  0001 C CNN "Farnell"
+F 5 "MCWR12X4991FTL" H 0   0   50  0001 C CNN "Manufacturer nr"
 	1    8550 5400
 	0    -1   -1   0
@@
 F 2 "Resistor_SMD:R_1206_3216Metric" V 9880 2600 50  0001 C CNN
 F 3 "http://www.farnell.com/datasheets/2331353.pdf?_ga=2.264231116.13702668.1544197496-523844734.1542029203&_gac=1.217211554.1543322461.EAIaIQobChMIof7Tlcz03gIVkuJ3Ch1UVwqwEAAYASAAEgK8PvD_BwE" H 9950 2600 50  0001 C CNN
-F 4 "1100244" V 9950 2600 50  0001 C CNN "Farnell"
-F 5 "WCR1206-100KFI" V 9950 2600 50  0001 C CNN "Manufacturer nr"
+F 4 "1100246" V 9950 2600 50  0001 C CNN "Farnell"
+F 5 "WCR1206-110KFI" V 9950 2600 50  0001 C CNN "Manufacturer nr"
 	1    9950 2600
 	1    0    0    -1
@@
 P 5000 5700
 F 0 "R17" V 5080 5700 50  0000 C CNN
-F 1 "5k1" V 5000 5700 50  0000 C CNN
+F 1 "4k99" V 5000 5700 50  0000 C CNN
 F 2 "Resistor_SMD:R_1206_3216Metric" V 4930 5700 50  0001 C CNN
 F 3 "http://www.farnell.com/datasheets/2331353.pdf?_ga=2.3463152.13702668.1544197496-523844734.1542029203&_gac=1.11733504.1543322461.EAIaIQobChMIof7Tlcz03gIVkuJ3Ch1UVwqwEAAYASAAEgK8PvD_BwE" H 5000 5700 50  0001 C CNN
 F 4 "" V 5000 5700 50  0001 C CNN "1100211"
-F 5 "WCR1206-5K1FI" V 5000 5700 50  0001 C CNN "Manufacturer nr"
+F 5 "MCWR12X4991FTL" V 5000 5700 50  0001 C CNN "Manufacturer nr"
 F 6 "2695161" H 0   0   50  0001 C CNN "Farnell"
 	1    5000 5700
@@
 P 5250 5900
 F 0 "R39" V 5330 5900 50  0000 C CNN
-F 1 "910R" V 5250 5900 50  0000 C CNN
+F 1 "1k" V 5250 5900 50  0000 C CNN
 F 2 "Resistor_SMD:R_1206_3216Metric" V 5180 5900 50  0001 C CNN
 F 3 "http://www.farnell.com/datasheets/2331353.pdf?_ga=2.25152762.13702668.1544197496-523844734.1542029203&_gac=1.12378624.1543322461.EAIaIQobChMIof7Tlcz03gIVkuJ3Ch1UVwqwEAAYASAAEgK8PvD_BwE" H 5250 5900 50  0001 C CNN
-F 4 "1100190" V 5250 5900 50  0001 C CNN "Farnell"
-F 5 "WCR1206-910RFI" V 5250 5900 50  0001 C CNN "Manufacturer nr"
+F 4 "1100192" V 5250 5900 50  0001 C CNN "Farnell"
+F 5 "WCR1206-1K0FI" V 5250 5900 50  0001 C CNN "Manufacturer nr"
 	1    5250 5900
 	-1   0    0    1
@@
 P 2350 7450
 F 0 "R40" V 2430 7450 50  0000 C CNN
-F 1 "4k7" V 2350 7450 50  0000 C CNN
+F 1 "4k99" V 2350 7450 50  0000 C CNN
 F 2 "Resistor_SMD:R_1206_3216Metric" V 2280 7450 50  0001 C CNN
 F 3 "http://www.farnell.com/datasheets/2158849.pdf?_ga=2.191241066.13702668.1544197496-523844734.1542029203&_gac=1.7619462.1543322461.EAIaIQobChMIof7Tlcz03gIVkuJ3Ch1UVwqwEAAYASAAEgK8PvD_BwE" H 2350 7450 50  0001 C CNN
-F 4 "1100209" V 2350 7450 50  0001 C CNN "Farnell"
-F 5 "WCR1206-4K7FI" V 2350 7450 50  0001 C CNN "Manufacturer nr"
+F 4 "2695161" V 2350 7450 50  0001 C CNN "Farnell"
+F 5 "MCWR12X4991FTL" V 2350 7450 50  0001 C CNN "Manufacturer nr"
 	1    2350 7450
 	0    -1   -1   0
@@
 P 4300 1900
 F 0 "R21" V 4380 1900 50  0000 C CNN
-F 1 "9k10" V 4300 1900 50  0000 C CNN
+F 1 "20k" V 4300 1900 50  0000 C CNN
 F 2 "Resistor_SMD:R_1206_3216Metric" V 4230 1900 50  0001 C CNN
 F 3 "http://www.farnell.com/datasheets/2331353.pdf?_ga=2.57067299.804204398.1540810031-466615820.1533907205&_gac=1.79366502.1540810769.CjwKCAjw39reBRBJEiwAO1m0OeFHyFqLAwRfo1TyfiEw1u5wgH8YT365nEvQxYyzS_SVx6sHehne4BoC4gYQAvD_BwE" H 4300 1900 50  0001 C CNN
-F 4 "1100217" V 4300 1900 50  0001 C CNN "Farnell"
-F 5 "WCR1206-9K1FI" V 4300 1900 50  0001 C CNN "Manufacturer nr"
+F 4 "1100226" V 4300 1900 50  0001 C CNN "Farnell"
+F 5 "WCR1206-20KFI" V 4300 1900 50  0001 C CNN "Manufacturer nr"
 	1    4300 1900
 	0    -1   -1   0
@@
 P 4300 1600
 F 0 "R20" V 4380 1600 50  0000 C CNN
-F 1 "9k10" V 4300 1600 50  0000 C CNN
+F 1 "20k" V 4300 1600 50  0000 C CNN
 F 2 "Resistor_SMD:R_1206_3216Metric" V 4230 1600 50  0001 C CNN
 F 3 "http://www.farnell.com/datasheets/2331353.pdf?_ga=2.57067299.804204398.1540810031-466615820.1533907205&_gac=1.79366502.1540810769.CjwKCAjw39reBRBJEiwAO1m0OeFHyFqLAwRfo1TyfiEw1u5wgH8YT365nEvQxYyzS_SVx6sHehne4BoC4gYQAvD_BwE" H 4300 1600 50  0001 C CNN
-F 4 "1100217" V 4300 1600 50  0001 C CNN "Farnell"
-F 5 "WCR1206-9K1FI" V 4300 1600 50  0001 C CNN "Manufacturer nr"
+F 4 "1100226" V 4300 1600 50  0001 C CNN "Farnell"
+F 5 "WCR1206-20KFI" V 4300 1600 50  0001 C CNN "Manufacturer nr"
 	1    4300 1600
 	0    1    1    0
@@
 P 4500 2350
 F 0 "R16" V 4400 2350 50  0000 C CNN
-F 1 "1k" V 4500 2350 50  0000 C CNN
+F 1 "3k9" V 4500 2350 50  0000 C CNN
 F 2 "Resistor_SMD:R_1206_3216Metric" V 4430 2350 50  0001 C CNN
 F 3 "http://www.farnell.com/datasheets/2158849.pdf?_ga=2.191239274.13702668.1544197496-523844734.1542029203&_gac=1.245695152.1543322461.EAIaIQobChMIof7Tlcz03gIVkuJ3Ch1UVwqwEAAYASAAEgK8PvD_BwE" H 4500 2350 50  0001 C CNN
-F 4 "1100192" V 4500 2350 50  0001 C CNN "Farnell"
-F 5 "WCR1206-1K0FI" V 4500 2350 50  0001 C CNN "Manufacturer nr"
+F 4 "1100206" V 4500 2350 50  0001 C CNN "Farnell"
+F 5 "WCR1206-3K9FI" V 4500 2350 50  0001 C CNN "Manufacturer nr"
 	1    4500 2350
 	1    0    0    -1
@@
 P 4600 2350
 F 0 "R38" V 4700 2350 50  0000 C CNN
-F 1 "1k" V 4600 2350 50  0000 C CNN
+F 1 "3k9" V 4600 2350 50  0000 C CNN
 F 2 "Resistor_SMD:R_1206_3216Metric" V 4530 2350 50  0001 C CNN
 F 3 "http://www.farnell.com/datasheets/2158849.pdf?_ga=2.191239274.13702668.1544197496-523844734.1542029203&_gac=1.245695152.1543322461.EAIaIQobChMIof7Tlcz03gIVkuJ3Ch1UVwqwEAAYASAAEgK8PvD_BwE" H 4600 2350 50  0001 C CNN
-F 4 "1100192" V 4600 2350 50  0001 C CNN "Farnell"
-F 5 "WCR1206-1K0FI" V 4600 2350 50  0001 C CNN "Manufacturer nr"
+F 4 "1100206" V 4600 2350 50  0001 C CNN "Farnell"
+F 5 "WCR1206-3K9FI" V 4600 2350 50  0001 C CNN "Manufacturer nr"
 	1    4600 2350
 	1    0    0    -1
@@
 P 4950 1150
 F 0 "R42" V 5030 1150 50  0000 C CNN
-F 1 "4k7" V 4950 1150 50  0000 C CNN
+F 1 "4k99" V 4950 1150 50  0000 C CNN
 F 2 "Resistor_SMD:R_1206_3216Metric" V 4880 1150 50  0001 C CNN
 F 3 "http://www.farnell.com/datasheets/2158849.pdf?_ga=2.191241066.13702668.1544197496-523844734.1542029203&_gac=1.7619462.1543322461.EAIaIQobChMIof7Tlcz03gIVkuJ3Ch1UVwqwEAAYASAAEgK8PvD_BwE" H 4950 1150 50  0001 C CNN
-F 4 "1100209" V 4950 1150 50  0001 C CNN "Farnell"
-F 5 "WCR1206-4K7FI" V 4950 1150 50  0001 C CNN "Manufacturer nr"
+F 4 "2695161" V 4950 1150 50  0001 C CNN "Farnell"
+F 5 "MCWR12X4991FTL" V 4950 1150 50  0001 C CNN "Manufacturer nr"
 	1    4950 1150
 	1    0    0    -1
@@
 Wire Wire Line
 	9550 5150 9550 5950
-Text Notes 1250 3100 0    50   ~ 0
+Text Notes 2000 3100 0    50   ~ 0
 Farnell: 1467755
 Wire Wire Line
@@
 Wire Wire Line
 	5200 7200 5300 7200
-Text Notes 3800 3000 0    50   ~ 0
+Text Notes 2000 3200 0    50   ~ 0
 OR: 4x MAX3468
 $EndSCHEMATC

Commit message: Updating BackplanePCB_slave.sch
Parts:
- C21: value 470u -> 220u
Changed lines of the file:
@@
 P 1950 1050
 F 0 "C21" H 1750 950 50  0000 L CNN
-F 1 "470u" H 1650 1150 50  0000 L CNN
+F 1 "220u" H 1650 1150 50  0000 L CNN
 F 2 "Capacitor_SMD:CP_Elec_8x10.5" H 1988 900 50  0001 C CNN
 F 3 "" H 1950 1050 50  0001 C CNN

Commit message: Updated BackplanePCB_slave.sch and layout. Updated all components to be ordered.
Parts:
- U9: Manufacturer nr PIC16F18854-I/SO -> PIC18F25K40-I/SO
Connections:
- wire segments 460 -> 458
Changed lines of the file:
@@
 $EndComp
 Wire Wire Line
-	2200 750  2200 900
+	2200 800  2200 900
 Wire Wire Line
-	2200 750  2450 750
+	2200 800  2450 800
 Wire Wire Line
 	2450 900  2450 800
@@
 F 3 "http://ww1.microchip.com/downloads/en/DeviceDoc/PIC18(L)F24_25K40%2028-Pin%20Low-Power%20High-Performance%20MCU%20with%20XLP%20Technology%2040001843D.pdf" H 8150 1750 50  0001 C CNN
 F 4 "2564200" H 7850 2350 50  0001 C CNN "Farnell"
-F 5 "PIC16F18854-I/SO" H 7850 2350 50  0001 C CNN "Manufacturer nr"
+F 5 "PIC18F25K40-I/SO" H 7850 2350 50  0001 C CNN "Manufacturer nr"
 	1    7850 2350
 	1    0    0    -1
@@
 L Device:D_Schottky_AAK D7
 U 1 1 5CF61E9D
-P 1750 750
-F 0 "D7" H 1750 550 50  0000 C CNN
-F 1 "VS-6ESH06-M3" H 1750 650 50  0000 C CNN
-F 2 "Package_TO_SOT_SMD:TO-277A" H 1750 750 50  0001 C CNN
-F 3 "http://www.farnell.com/datasheets/2182681.pdf?_ga=2.208013010.1588585681.1526323724-1626853455.1515011571" H 1750 750 50  0001 C CNN
-F 4 "2471194" H 1750 750 50  0001 C CNN "Farnell"
-F 5 "VS-6ESH06-M3/86A" H 0   -50 50  0001 C CNN "Manufacturer nr"
-	1    1750 750
+P 1750 800
+F 0 "D7" H 1750 600 50  0000 C CNN
+F 1 "VS-6ESH06-M3" H 1750 700 50  0000 C CNN
+F 2 "Package_TO_SOT_SMD:TO-277A" H 1750 800 50  0001 C CNN
+F 3 "http://www.farnell.com/datasheets/2182681.pdf?_ga=2.208013010.1588585681.1526323724-1626853455.1515011571" H 1750 800 50  0001 C CNN
+F 4 "2471194" H 1750 800 50  0001 C CNN "Farnell"
+F 5 "VS-6ESH06-M3/86A" H 0   0   50  0001 C CNN "Manufacturer nr"
+	1    1750 800
 	-1   0    0    1
 $EndComp
@@
 $EndComp
 Wire Wire Line
-	2200 750  1950 750
+	2200 800  1950 800
 Wire Wire Line
-	1950 750  1950 900
-Connection ~ 2200 750
+	1950 800  1950 900
+Connection ~ 2200 800
 Wire Wire Line
 	1950 1200 1950 1300
@@
 Wire Wire Line
 	1950 1300 2200 1300
-Connection ~ 1950 750
+Connection ~ 1950 800
 Wire Wire Line
-	1900 750  1950 750
+	1900 800  1950 800
 Wire Wire Line
 	850  800  900  800
@@
 Connection ~ 2450 800
 Wire Wire Line
-	2450 800  2450 750
-Wire Wire Line
-	1550 750  1550 800
-Wire Wire Line
-	1550 850  1550 800
-Connection ~ 1550 800
-Wire Wire Line
 	9800 3900 10000 3900
 Wire Wire Line
@@
 Text Notes 2000 3200 0    50   ~ 0
 OR: 4x MAX3468
+Connection ~ 1550 800
+Wire Wire Line
+	1550 800  1550 900
 $EndSCHEMATC
