File: KiCad/TrackAmplifier2/TrackAmplifier.sch (KiCad schematic (older format))
At the start: 119 parts, among them J1 DB15_Male_MountingHoles, J2 Conn_01x06, Q1 NTR5103NT1G, U1 ST485EBDR, U10 MCP1525, U11 MCP9701A-E/TO, U2 ST485EBDR, U3 L78M05CDT-1-TO-251-3, U4 LMD18200, U5 ST485EBDR, U6 ST485EBDR, U7 MCP6N11, U8 INA2180, U9 PIC18F25K40

Commit message: Updated all schematics and layouts. Updated all component lists and csv files. Created ShopCartAll.csv from farnell big order for these 4 boards. Created new gerber files in the board-named directories to be send to PCB farmer.
Parts:
- C10, C14, C15, C20, C22, C24, C27, C28, C29, C3, C30, C31, C33, C35, C37, C4, C7, C9: Farnell 1414715 -> 2896646; Manufacturer nr C1206C104K5RACTU -> VJ1206Y104KXXPW1BC
- R14: value 1k -> 4k99; Farnell 1100192 -> 2695161; Manufacturer nr WCR1206-1K0FI -> MCWR12X4991FTL
- R47: Farnell - -> (none)
