File: KiCad/TrackAmplifier2/TrackAmplifier.kicad_pcb (KiCad board)
At the start: 2 copper layers, 105 x 70 mm, 122 parts, among them J1 DB15_Male_MountingHoles, J2 Conn_01x06, Q1 NTR5103NT1G, U1 ST485EBDR, U10 MCP1525, U11 MCP9701A-E/TO, U2 ST485EBDR, U3 L78M05CDT-1-TO-251-3, U4 LMD18200, U5 ST485EBDR, U6 ST485EBDR, U7 MCP6N11, U8 INA2180, U9 PIC18F25K40

Commit message: Final checks and updates, PCB's ordered.
Changed lines of the file:
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@@
     (descr "TO-220-11, Horizontal, RM 1.7mm, staggered type-1, see http://www.ti.com/lit/ds/symlink/lmd18200.pdf")
     (tags "TO-220-11 Horizontal RM 1.7mm staggered type-1")
-    (fp_text reference U4 (at 20.255 -2.697 180) (layer F.SilkS)
+    (fp_text reference U4 (at 22.414 -4.602 180) (layer F.SilkS)
       (effects (font (size 1 1) (thickness 0.15)))
     )
@@
     (descr "TO-92 leads molded, narrow, drill 0.75mm (see NXP sot054_po.pdf)")
     (tags "to-92 sc-43 sc-43a sot54 PA33 transistor")
-    (fp_text reference U11 (at 6.35 -0.381 180) (layer F.SilkS)
+    (fp_text reference U11 (at 4.445 -2.54 180) (layer F.SilkS)
       (effects (font (size 1 1) (thickness 0.15)))
     )
@@
     (tags "VSSOP-8 3.0 x 3.0")
     (attr smd)
-    (fp_text reference U8 (at 0 0) (layer F.SilkS)
+    (fp_text reference U8 (at -4.318 0 270) (layer F.SilkS)
       (effects (font (size 1 1) (thickness 0.15)))
     )
@@
   (gr_line (start 133.589102 56.72666) (end 133.462102 56.59966) (layer B.SilkS) (width 0.2))
   (gr_line (start 131.430102 56.72666) (end 133.589102 56.72666) (layer B.SilkS) (width 0.2))
-  (gr_text ICSP (at 132.319102 57.74266 180) (layer B.SilkS)
+  (gr_text ICSP (at 132.319102 57.74266) (layer B.SilkS)
     (effects (font (size 1 1) (thickness 0.15)) (justify mirror))
   )
@@
     (effects (font (size 1 1) (thickness 0.15)))
   )
-  (gr_text 10 (at 130.518 83.3224) (layer F.SilkS)
+  (gr_text 10 (at 126.962 80.63) (layer F.SilkS)
     (effects (font (size 1 1) (thickness 0.15)))
   )
-  (gr_text 2 (at 144.1324 83.3224) (layer F.SilkS)
+  (gr_text 2 (at 147.028 80.63) (layer F.SilkS)
     (effects (font (size 1 1) (thickness 0.15)))
   )
