File: KiCad/BackplanePCB_solder2/BackplanePCB_solder.kicad_pcb (KiCad board)
At the start: 2 copper layers, 470 x 59 mm, 87 parts, among them J1 Conn_02x05_Odd_Even, J10 Conn_01x03, J11 Conn_01x03, J12 Conn_01x03, J13 Conn_01x03, J14 Conn_01x03, J15 Conn_01x03, J16 DB15_Female_MountingHoles, J17 DB15_Female_MountingHoles, J18 Conn_01x03, J19 DB15_Female_MountingHoles, J2 Conn_02x05_Odd_Even, J20 DB15_Female_MountingHoles, J21 DB15_Female_MountingHoles, J22 DB15_Female_MountingHoles, J23 DB15_Female_MountingHoles, J24 DB15_Female_MountingHoles, J25 Conn_01x06, J3 PowerBug+15V, J4 PowerBug_GND, J5 Conn_01x03, J6 Conn_01x03, J7 Conn_01x03, J8 DB15_Female_MountingHoles, J9 DB15_Female_MountingHoles, Q1 Q_NMOS_GSD, U1 ST485EBDR, U2 ST485EBDR, U3 ST485EBDR, U4 KA78M05_TO252, U5 ST485EBDR, U6 PIC16F18854-SO

Commit message: updated BackplanePCB_solder2 PCB for prototyping and production.
Routing:
- net GND: track 340.8 -> 339.0 mm
- net ID_3: track 52.8 -> 51.2 mm
- net Net-(C18-Pad1): track 17.6 -> 16.9 mm
Other:
- rule trace_min: 0.1 -> 0.2
- rule via_min_drill: 0.3 -> 0.4
- rule via_min_size: 0.6 -> 0.8
