File: KiCad/BackplanePCB_solder2/BackplanePCB_slave.sch (KiCad schematic (older format))
At the start: 55 parts, among them J25 Conn_01x06, Q1 Q_NMOS_GSD, U1 ST485EBDR, U2 ST485EBDR, U3 ST485EBDR, U4 KA78M05_TO252, U5 ST485EBDR, U6 PIC16F18854-SO

Commit message: Updating design according to findings on proto (LEFT  config). Still some spces between sub -d screws is NOK.
Parts:
- U4: symbol Regulator_Linear:L78M05CDT-1_TO251-3 -> BackplanePCB_solder-rescue:L78M05CDT-1_TO251-3-Regulator_Linear
- U6: symbol MCU_Microchip_PIC16:PIC16F18854-SO -> BackplanePCB_solder-rescue:PIC16F18854-SO-MCU_Microchip_PIC16
Changed lines of the file:
@@
 $EndComp
 $Comp
-L Regulator_Linear:L78M05CDT-1_TO251-3 U4
+L BackplanePCB_solder-rescue:L78M05CDT-1_TO251-3-Regulator_Linear U4
 U 1 1 5BD693B7
 P 2900 900
@@
 Connection ~ 4150 1450
 $Comp
-L MCU_Microchip_PIC16:PIC16F18854-SO U6
+L BackplanePCB_solder-rescue:PIC16F18854-SO-MCU_Microchip_PIC16 U6
 U 1 1 5BD6BD7D
 P 8200 2650
@@
 	10000 2650 10000 2750
 Text GLabel 7250 2050 0    50   Output ~ 0
+ID_10
+Text GLabel 7250 2150 0    50   Output ~ 0
+ID_9
+Text GLabel 7250 2250 0    50   Output ~ 0
+ID_8
+Text GLabel 7250 2350 0    50   Output ~ 0
+ID_7
+Text GLabel 7250 2450 0    50   Output ~ 0
+ID_6
+Text GLabel 9000 3250 2    50   Output ~ 0
+ID_5
+Text GLabel 9000 3150 2    50   Output ~ 0
+ID_4
+Text GLabel 9000 3050 2    50   Output ~ 0
+ID_3
+Text GLabel 9000 2950 2    50   Output ~ 0
+ID_2
+Text GLabel 9000 2850 2    50   Output ~ 0
 ID_1
-Text GLabel 7250 2150 0    50   Output ~ 0
-ID_2
-Text GLabel 7250 2250 0    50   Output ~ 0
-ID_3
-Text GLabel 7250 2350 0    50   Output ~ 0
-ID_4
-Text GLabel 7250 2450 0    50   Output ~ 0
-ID_5
-Text GLabel 9000 3250 2    50   Output ~ 0
-ID_6
-Text GLabel 9000 3150 2    50   Output ~ 0
-ID_7
-Text GLabel 9000 3050 2    50   Output ~ 0
-ID_8
-Text GLabel 9000 2950 2    50   Output ~ 0
-ID_9
-Text GLabel 9000 2850 2    50   Output ~ 0
-ID_10
 Wire Wire Line
 	7250 2050 7700 2050

Commit message: Revert to working version of commit on 16-10-18
Parts:
- U4: symbol BackplanePCB_solder-rescue:L78M05CDT-1_TO251-3-Regulator_Linear -> Regulator_Linear:L78M05CDT-1_TO251-3
- U6: symbol BackplanePCB_solder-rescue:PIC16F18854-SO-MCU_Microchip_PIC16 -> MCU_Microchip_PIC16:PIC16F18854-SO
Changed lines of the file:
@@
 $EndComp
 $Comp
-L BackplanePCB_solder-rescue:L78M05CDT-1_TO251-3-Regulator_Linear U4
+L Regulator_Linear:L78M05CDT-1_TO251-3 U4
 U 1 1 5BD693B7
 P 2900 900
@@
 Connection ~ 4150 1450
 $Comp
-L BackplanePCB_solder-rescue:PIC16F18854-SO-MCU_Microchip_PIC16 U6
+L MCU_Microchip_PIC16:PIC16F18854-SO U6
 U 1 1 5BD6BD7D
 P 8200 2650
@@
 	10000 2650 10000 2750
 Text GLabel 7250 2050 0    50   Output ~ 0
+ID_1
+Text GLabel 7250 2150 0    50   Output ~ 0
+ID_2
+Text GLabel 7250 2250 0    50   Output ~ 0
+ID_3
+Text GLabel 7250 2350 0    50   Output ~ 0
+ID_4
+Text GLabel 7250 2450 0    50   Output ~ 0
+ID_5
+Text GLabel 9000 3250 2    50   Output ~ 0
+ID_6
+Text GLabel 9000 3150 2    50   Output ~ 0
+ID_7
+Text GLabel 9000 3050 2    50   Output ~ 0
+ID_8
+Text GLabel 9000 2950 2    50   Output ~ 0
+ID_9
+Text GLabel 9000 2850 2    50   Output ~ 0
 ID_10
-Text GLabel 7250 2150 0    50   Output ~ 0
-ID_9
-Text GLabel 7250 2250 0    50   Output ~ 0
-ID_8
-Text GLabel 7250 2350 0    50   Output ~ 0
-ID_7
-Text GLabel 7250 2450 0    50   Output ~ 0
-ID_6
-Text GLabel 9000 3250 2    50   Output ~ 0
-ID_5
-Text GLabel 9000 3150 2    50   Output ~ 0
-ID_4
-Text GLabel 9000 3050 2    50   Output ~ 0
-ID_3
-Text GLabel 9000 2950 2    50   Output ~ 0
-ID_2
-Text GLabel 9000 2850 2    50   Output ~ 0
-ID_1
 Wire Wire Line
 	7250 2050 7700 2050
