File: KiCad/BackplanePCB_solder2/BackplanePCB_slave.sch (KiCad schematic (older format))
At the start: 55 parts, among them J25 Conn_01x06, Q1 Q_NMOS_GSD, U1 ST485EBDR, U2 ST485EBDR, U3 ST485EBDR, U4 KA78M05_TO252, U5 ST485EBDR, U6 PIC16F18854-SO

Commit message: backplane schematic updates
Parts:
- removed R11, R21, R4, R5, R6: R, Resistor_SMD:R_1206_3216Metric, symbol Device:R
- U4: symbol Regulator_Linear:L78M05CDT-1_TO251-3 -> BackplanePCB_solder-rescue:L78M05CDT-1_TO251-3-Regulator_Linear
Connections:
- wire segments 235 -> 230
Other:
- note added: "BIT1"
- note added: "BIT2"
- note added: "BIT4"
Changed lines of the file:
@@
 $EndComp
 $Comp
-L Regulator_Linear:L78M05CDT-1_TO251-3 U4
+L BackplanePCB_solder-rescue:L78M05CDT-1_TO251-3-Regulator_Linear U4
 U 1 1 5BD693B7
 P 2900 900
@@
 $EndComp
 $Comp
-L Device:R R6
-U 1 1 5BD6BEE7
-P 900 2250
-F 0 "R6" V 980 2250 50  0000 C CNN
-F 1 "R" V 900 2250 50  0000 C CNN
-F 2 "Resistor_SMD:R_1206_3216Metric" V 830 2250 50  0001 C CNN
-F 3 "~" H 900 2250 50  0001 C CNN
-	1    900  2250
-	-1   0    0    1
-$EndComp
-$Comp
 L Device:C C5
 U 1 1 5BD6BF1D
@@
 	900  2550 900  2450
 Wire Wire Line
-	900  2100 900  2050
-Wire Wire Line
 	900  2450 1150 2450
 Wire Wire Line
 	1150 2450 1150 2550
 Connection ~ 900  2450
-Wire Wire Line
-	900  2450 900  2400
 Wire Wire Line
 	900  2900 1150 2900
@@
 $EndComp
 $Comp
-L Device:R R4
-U 1 1 5BE7D8F3
-P 850 3750
-F 0 "R4" V 930 3750 50  0000 C CNN
-F 1 "R" V 850 3750 50  0000 C CNN
-F 2 "Resistor_SMD:R_1206_3216Metric" V 780 3750 50  0001 C CNN
-F 3 "~" H 850 3750 50  0001 C CNN
-	1    850  3750
-	-1   0    0    1
-$EndComp
-$Comp
 L Device:C C3
 U 1 1 5BE7D8FA
@@
 	850  4050 850  3950
 Wire Wire Line
-	850  3600 850  3550
-Wire Wire Line
 	850  3950 1100 3950
 Wire Wire Line
 	1100 3950 1100 4050
 Connection ~ 850  3950
-Wire Wire Line
-	850  3950 850  3900
 Wire Wire Line
 	850  4400 1100 4400
@@
 $EndComp
 $Comp
-L Device:R R5
-U 1 1 5BE7F7E9
-P 850 5250
-F 0 "R5" V 930 5250 50  0000 C CNN
-F 1 "R" V 850 5250 50  0000 C CNN
-F 2 "Resistor_SMD:R_1206_3216Metric" V 780 5250 50  0001 C CNN
-F 3 "~" H 850 5250 50  0001 C CNN
-	1    850  5250
-	-1   0    0    1
-$EndComp
-$Comp
 L Device:C C4
 U 1 1 5BE7F7F0
@@
 	850  5550 850  5450
 Wire Wire Line
-	850  5100 850  5050
-Wire Wire Line
 	850  5450 1100 5450
 Wire Wire Line
 	1100 5450 1100 5550
 Connection ~ 850  5450
-Wire Wire Line
-	850  5450 850  5400
 Wire Wire Line
 	850  5900 1100 5900
@@
 $EndComp
 $Comp
-L Device:R R11
-U 1 1 5BE82D60
-P 3500 3750
-F 0 "R11" V 3580 3750 50  0000 C CNN
-F 1 "R" V 3500 3750 50  0000 C CNN
-F 2 "Resistor_SMD:R_1206_3216Metric" V 3430 3750 50  0001 C CNN
-F 3 "~" H 3500 3750 50  0001 C CNN
-	1    3500 3750
-	-1   0    0    1
-$EndComp
-$Comp
 L Device:C C11
 U 1 1 5BE82D67
@@
 	3500 4050 3500 3950
 Wire Wire Line
-	3500 3600 3500 3550
-Wire Wire Line
 	3500 3950 3750 3950
 Wire Wire Line
 	3750 3950 3750 4050
 Connection ~ 3500 3950
-Wire Wire Line
-	3500 3950 3500 3900
 Wire Wire Line
 	3500 4400 3750 4400
@@
 $EndComp
 $Comp
-L Device:R R21
-U 1 1 5BEEFBE1
-P 7450 1150
-F 0 "R21" V 7530 1150 50  0000 C CNN
-F 1 "R" V 7450 1150 50  0000 C CNN
-F 2 "Resistor_SMD:R_1206_3216Metric" V 7380 1150 50  0001 C CNN
-F 3 "~" H 7450 1150 50  0001 C CNN
-	1    7450 1150
-	0    -1   -1   0
-$EndComp
-$Comp
 L Device:C C18
 U 1 1 5BEEFD1F
@@
 Wire Wire Line
 	7150 1050 7150 1150
-Wire Wire Line
-	7150 1150 7300 1150
-Wire Wire Line
-	7600 1150 7750 1150
 Wire Wire Line
 	7750 1150 7750 1200
@@
 Wire Wire Line
 	2900 1450 2900 1600
+Wire Wire Line
+	900  2050 900  2450
+Wire Wire Line
+	850  3550 850  3950
+Wire Wire Line
+	850  5050 850  5450
+Wire Wire Line
+	3500 3550 3500 3950
+Wire Wire Line
+	7150 1150 7750 1150
+Text Notes 6100 3300 1    50   ~ 0
+BIT1
+Text Notes 6300 3300 1    50   ~ 0
+BIT2
+Text Notes 6500 3300 1    50   ~ 0
+BIT4
 $EndSCHEMATC

Commit message: Updating BackplanePCB_slave.sch
Parts:
- removed C9: C, Capacitor_SMD:C_1206_3216Metric, symbol Device:C
- removed D1: D_Zener, Diode_SMD:D_1206_3216Metric, symbol Device:D_Zener
- added C24: 4.7u, Capacitor_SMD:C_1206_3216Metric, symbol Device:C
- added C9: 220u, Capacitor_SMD:CP_Elec_8x10.5, symbol Device:CP
- added D1: D_Schottky_AAK, Package_TO_SOT_SMD:TO-277A, symbol Device:D_Schottky_AAK
- added R29: 0E, Resistor_SMD:R_1206_3216Metric, symbol Device:R
- C10, C18: value C -> 4.7u; Farnell (none) -> 2320886; Manufacturer nr (none) -> MC1206B475K250CT
- C12, C15, C19: value C -> 100n; Farnell (none) -> 1414715; Manufacturer nr (none) -> C1206C104K5RACTU
- C16: value CP -> 220u; Farnell (none) -> 2346568; Manufacturer nr (none) -> 16PX220MEFC6.3X11
- D2: value LED -> LED GR RUN; footprint Diode_SMD:D_1206_3216Metric -> Diode_SMD:LED_0.8x0.8; Farnell (none) -> 2426215; Manufacturer nr (none) -> KPH-1608SGC
- D3, D6, D7: value LED GR -> LED GR RUN; footprint Diode_SMD:D_1206_3216Metric -> Diode_SMD:LED_0.8x0.8; Farnell (none) -> 2426215; Manufacturer nr (none) -> KPH-1608SGC
- R12, R22, R23, R24, R25, R26: value R -> 300E; Farnell (none) -> 1100176; Manufacturer nr (none) -> WCR1206-300RFI
- U4: value KA78M05_TO252 -> L78M05CDT-1-TO-251-3; Farnell (none) -> 1077155; Manufacturer nr (none) -> L78M05CDT-1
Connections:
- wire segments 230 -> 236

Commit message: Updated BackplanePCB_slave.sch and layout. Updated all components to be ordered.
Parts:
- added R30: NP, Resistor_SMD:R_0603_1608Metric, symbol Device:R
- added R31, R32, R33, R34: 0E, Resistor_SMD:R_1206_3216Metric, symbol Device:R
- C11, C3, C4, C5: value C -> 4.7u; Farnell (none) -> 2320886; Manufacturer nr (none) -> MC1206B475K250CT
- C13, C14, C17, C6, C7, C8: value C -> 100n; Farnell (none) -> 1414715; Manufacturer nr (none) -> C1206C104K5RACTU
- D4: value LED YE -> LED YE WAR; footprint Diode_SMD:D_1206_3216Metric -> Diode_SMD:LED_0.8x0.8; Farnell (none) -> 2426218; Manufacturer nr (none) -> KPH-1608YC
- D5: value LED RD -> LED RD ERR; footprint Diode_SMD:D_1206_3216Metric -> Diode_SMD:LED_0.8x0.8; Farnell (none) -> 2426211; Manufacturer nr (none) -> KPH-1608EC
- D6: value LED GR RUN -> LED GR RX
- D7: value LED GR RUN -> LED GR TX
- Q1: value Q_NMOS_GSD -> NTR5103NT1G; Farnell (none) -> 2724423; Manufacturer nr (none) -> NTR5103NT1G
- R10, R17: value R -> 10k; Farnell (none) -> 1100218; Manufacturer nr (none) -> WCR1206-10KFI
- R13, R9: value R -> 1k; Farnell (none) -> 1100192; Manufacturer nr (none) -> WCR1206-1K0FI
- R14, R15, R16: value R -> NP; Farnell (none) -> -; Manufacturer nr (none) -> -
- R18: value R -> 110k; Farnell (none) -> 1100246; Manufacturer nr (none) -> WCR1206-110KFI
- R19, R20: value R -> 470; Farnell (none) -> 1100183; Manufacturer nr (none) -> WCR1206-470RFI
- R7, R8: value R -> 10E; Farnell (none) -> 1100138; Manufacturer nr (none) -> WCR1206-10RFI
- U1, U2, U3, U5: Farnell (none) -> -; Manufacturer nr (none) -> ST485EBDR
- U6: value PIC16F18854-SO -> PIC18F25K40; symbol MCU_Microchip_PIC16:PIC16F18854-SO -> BackplanePCB_solder-rescue:PIC16F18854-SO-MCU_Microchip_PIC16; Farnell (none) -> 2564200; Manufacturer nr (none) -> PIC18F25K40-I/SO
Connections:
- wire segments 236 -> 242

Commit message: Updated all schematics and layouts. Updated all component lists and csv files. Created ShopCartAll.csv from farnell big order for these 4 boards. Created new gerber files in the board-named directories to be send to PCB farmer.
Parts:
- C12, C13, C14, C15, C17, C19, C6, C7, C8: Farnell 1414715 -> 2896646; Manufacturer nr C1206C104K5RACTU -> VJ1206Y104KXXPW1BC
- R13: value 1k -> 4k99; Farnell 1100192 -> 2695161; Manufacturer nr WCR1206-1K0FI -> MCWR12X4991FTL
- R14, R15, R16, R30, U1, U2, U3, U5: Farnell - -> (none)
Changed lines of the file:
@@
 F 2 "Package_SO:SOIC-8_3.9x4.9mm_P1.27mm" H 2300 1750 50  0001 C CNN
 F 3 "http://www.st.com/resource/en/datasheet/st485eb.pdf" H 2300 2700 50  0001 C CNN
-F 4 "-" H 2300 2650 50  0001 C CNN "Farnell"
+F 4 "" H 2300 2650 50  0001 C CNN "Farnell"
 F 5 "ST485EBDR" H 2300 2650 50  0001 C CNN "Manufacturer nr"
 	1    2300 2650
@@
 P 5550 4600
 F 0 "R13" V 5630 4600 50  0000 C CNN
-F 1 "1k" V 5550 4600 50  0000 C CNN
+F 1 "4k99" V 5550 4600 50  0000 C CNN
 F 2 "Resistor_SMD:R_1206_3216Metric" V 5480 4600 50  0001 C CNN
-F 3 "http://www.farnell.com/datasheets/2158849.pdf?_ga=2.191239274.13702668.1544197496-523844734.1542029203&_gac=1.245695152.1543322461.EAIaIQobChMIof7Tlcz03gIVkuJ3Ch1UVwqwEAAYASAAEgK8PvD_BwE" H 5550 4600 50  0001 C CNN
-F 4 "1100192" V 5550 4600 50  0001 C CNN "Farnell"
-F 5 "WCR1206-1K0FI" V 5550 4600 50  0001 C CNN "Manufacturer nr"
+F 3 "http://www.farnell.com/datasheets/2158849.pdf?_ga=2.191241066.13702668.1544197496-523844734.1542029203&_gac=1.7619462.1543322461.EAIaIQobChMIof7Tlcz03gIVkuJ3Ch1UVwqwEAAYASAAEgK8PvD_BwE" H 5550 4600 50  0001 C CNN
+F 4 "2695161" V 5550 4600 50  0001 C CNN "Farnell"
+F 5 "MCWR12X4991FTL" V 5550 4600 50  0001 C CNN "Manufacturer nr"
 	1    5550 4600
 	-1   0    0    1
@@
 F 2 "Resistor_SMD:R_0603_1608Metric" V 6480 3000 50  0001 C CNN
 F 3 "~" H 6550 3000 50  0001 C CNN
-F 4 "-" V 6550 3000 50  0001 C CNN "Farnell"
+F 4 "" V 6550 3000 50  0001 C CNN "Farnell"
 F 5 "-" V 6550 3000 50  0001 C CNN "Manufacturer nr"
 	1    6550 3000
@@
 F 2 "Resistor_SMD:R_0603_1608Metric" V 6280 3000 50  0001 C CNN
 F 3 "~" H 6350 3000 50  0001 C CNN
-F 4 "-" V 6350 3000 50  0001 C CNN "Farnell"
+F 4 "" V 6350 3000 50  0001 C CNN "Farnell"
 F 5 "-" V 6350 3000 50  0001 C CNN "Manufacturer nr"
 	1    6350 3000
@@
 F 2 "Resistor_SMD:R_0603_1608Metric" V 6080 3000 50  0001 C CNN
 F 3 "~" H 6150 3000 50  0001 C CNN
-F 4 "-" V 6150 3000 50  0001 C CNN "Farnell"
+F 4 "" V 6150 3000 50  0001 C CNN "Farnell"
 F 5 "-" V 6150 3000 50  0001 C CNN "Manufacturer nr"
 	1    6150 3000
@@
 F 2 "Capacitor_SMD:C_1206_3216Metric" H 2588 1050 50  0001 C CNN
 F 3 "http://www.farnell.com/datasheets/1901289.pdf?_ga=2.262491141.804204398.1540810031-466615820.1533907205&_gac=1.154756810.1540810031.CjwKCAjw39reBRBJEiwAO1m0OUdqKKSX6YgNsFqfn4kAD7vSQS5JfvsNobbwGFQV72towt0oHUutJhoC7b8QAvD_BwE" H 2550 1200 50  0001 C CNN
-F 4 "1414715" H 2550 1200 50  0001 C CNN "Farnell"
-F 5 "C1206C104K5RACTU" H 2550 1200 50  0001 C CNN "Manufacturer nr"
+F 4 "2896646" H 2550 1200 50  0001 C CNN "Farnell"
+F 5 "VJ1206Y104KXXPW1BC" H 2550 1200 50  0001 C CNN "Manufacturer nr"
 	1    2550 1200
 	1    0    0    -1
@@
 F 2 "Capacitor_SMD:C_1206_3216Metric" H 3338 1050 50  0001 C CNN
 F 3 "http://www.farnell.com/datasheets/1901289.pdf?_ga=2.262491141.804204398.1540810031-466615820.1533907205&_gac=1.154756810.1540810031.CjwKCAjw39reBRBJEiwAO1m0OUdqKKSX6YgNsFqfn4kAD7vSQS5JfvsNobbwGFQV72towt0oHUutJhoC7b8QAvD_BwE" H 3300 1200 50  0001 C CNN
-F 4 "1414715" H 3300 1200 50  0001 C CNN "Farnell"
-F 5 "C1206C104K5RACTU" H 3300 1200 50  0001 C CNN "Manufacturer nr"
+F 4 "2896646" H 3300 1200 50  0001 C CNN "Farnell"
+F 5 "VJ1206Y104KXXPW1BC" H 3300 1200 50  0001 C CNN "Manufacturer nr"
 	1    3300 1200
 	1    0    0    -1
@@
 F 2 "Capacitor_SMD:C_1206_3216Metric" H 8038 1200 50  0001 C CNN
 F 3 "http://www.farnell.com/datasheets/1901289.pdf?_ga=2.262491141.804204398.1540810031-466615820.1533907205&_gac=1.154756810.1540810031.CjwKCAjw39reBRBJEiwAO1m0OUdqKKSX6YgNsFqfn4kAD7vSQS5JfvsNobbwGFQV72towt0oHUutJhoC7b8QAvD_BwE" H 8000 1350 50  0001 C CNN
-F 4 "1414715" H 8000 1350 50  0001 C CNN "Farnell"
-F 5 "C1206C104K5RACTU" H 8000 1350 50  0001 C CNN "Manufacturer nr"
+F 4 "2896646" H 8000 1350 50  0001 C CNN "Farnell"
+F 5 "VJ1206Y104KXXPW1BC" H 8000 1350 50  0001 C CNN "Manufacturer nr"
 	1    8000 1350
 	1    0    0    -1
@@
 F 2 "Capacitor_SMD:C_1206_3216Metric" H 6288 4700 50  0001 C CNN
 F 3 "http://www.farnell.com/datasheets/1901289.pdf?_ga=2.262491141.804204398.1540810031-466615820.1533907205&_gac=1.154756810.1540810031.CjwKCAjw39reBRBJEiwAO1m0OUdqKKSX6YgNsFqfn4kAD7vSQS5JfvsNobbwGFQV72towt0oHUutJhoC7b8QAvD_BwE" H 6250 4850 50  0001 C CNN
-F 4 "1414715" H 6250 4850 50  0001 C CNN "Farnell"
-F 5 "C1206C104K5RACTU" H 6250 4850 50  0001 C CNN "Manufacturer nr"
+F 4 "2896646" H 6250 4850 50  0001 C CNN "Farnell"
+F 5 "VJ1206Y104KXXPW1BC" H 6250 4850 50  0001 C CNN "Manufacturer nr"
 	1    6250 4850
 	1    0    0    -1
@@
 F 2 "Resistor_SMD:R_0603_1608Metric" V 3280 2300 50  0001 C CNN
 F 3 "http://www.farnell.com/datasheets/2331353.pdf?_ga=2.31327414.804204398.1540810031-466615820.1533907205&_gac=1.187361882.1540810769.CjwKCAjw39reBRBJEiwAO1m0OeFHyFqLAwRfo1TyfiEw1u5wgH8YT365nEvQxYyzS_SVx6sHehne4BoC4gYQAvD_BwE" H 3350 2300 50  0001 C CNN
-F 4 "-" V 3350 2300 50  0001 C CNN "Farnell"
+F 4 "" V 3350 2300 50  0001 C CNN "Farnell"
 F 5 "-" V 3350 2300 50  0001 C CNN "Manufacturer nr"
 	1    3350 2300
@@
 F 2 "Capacitor_SMD:C_1206_3216Metric" H 3688 2600 50  0001 C CNN
 F 3 "http://www.farnell.com/datasheets/1901289.pdf?_ga=2.262491141.804204398.1540810031-466615820.1533907205&_gac=1.154756810.1540810031.CjwKCAjw39reBRBJEiwAO1m0OUdqKKSX6YgNsFqfn4kAD7vSQS5JfvsNobbwGFQV72towt0oHUutJhoC7b8QAvD_BwE" H 3650 2750 50  0001 C CNN
-F 4 "1414715" H 3650 2750 50  0001 C CNN "Farnell"
-F 5 "C1206C104K5RACTU" H 3650 2750 50  0001 C CNN "Manufacturer nr"
+F 4 "2896646" H 3650 2750 50  0001 C CNN "Farnell"
+F 5 "VJ1206Y104KXXPW1BC" H 3650 2750 50  0001 C CNN "Manufacturer nr"
 	1    3650 2750
 	1    0    0    -1
@@
 F 2 "Capacitor_SMD:C_1206_3216Metric" H 1188 2550 50  0001 C CNN
 F 3 "http://www.farnell.com/datasheets/1901289.pdf?_ga=2.262491141.804204398.1540810031-466615820.1533907205&_gac=1.154756810.1540810031.CjwKCAjw39reBRBJEiwAO1m0OUdqKKSX6YgNsFqfn4kAD7vSQS5JfvsNobbwGFQV72towt0oHUutJhoC7b8QAvD_BwE" H 1150 2700 50  0001 C CNN
-F 4 "1414715" H 1150 2700 50  0001 C CNN "Farnell"
-F 5 "C1206C104K5RACTU" H 1150 2700 50  0001 C CNN "Manufacturer nr"
+F 4 "2896646" H 1150 2700 50  0001 C CNN "Farnell"
+F 5 "VJ1206Y104KXXPW1BC" H 1150 2700 50  0001 C CNN "Manufacturer nr"
 	1    1150 2700
 	1    0    0    -1
@@
 F 2 "Package_SO:SOIC-8_3.9x4.9mm_P1.27mm" H 2250 3250 50  0001 C CNN
 F 3 "http://www.st.com/resource/en/datasheet/st485eb.pdf" H 2250 4200 50  0001 C CNN
-F 4 "-" H 2250 4150 50  0001 C CNN "Farnell"
+F 4 "" H 2250 4150 50  0001 C CNN "Farnell"
 F 5 "ST485EBDR" H 2250 4150 50  0001 C CNN "Manufacturer nr"
 	1    2250 4150
@@
 F 2 "Package_SO:SOIC-8_3.9x4.9mm_P1.27mm" H 4900 3250 50  0001 C CNN
 F 3 "http://www.st.com/resource/en/datasheet/st485eb.pdf" H 4900 4200 50  0001 C CNN
-F 4 "-" H 4900 4150 50  0001 C CNN "Farnell"
+F 4 "" H 4900 4150 50  0001 C CNN "Farnell"
 F 5 "ST485EBDR" H 4900 4150 50  0001 C CNN "Manufacturer nr"
 	1    4900 4150
@@
 F 2 "Package_SO:SOIC-8_3.9x4.9mm_P1.27mm" H 2250 4750 50  0001 C CNN
 F 3 "http://www.st.com/resource/en/datasheet/st485eb.pdf" H 2250 5700 50  0001 C CNN
-F 4 "-" H 2250 5650 50  0001 C CNN "Farnell"
+F 4 "" H 2250 5650 50  0001 C CNN "Farnell"
 F 5 "ST485EBDR" H 2250 5650 50  0001 C CNN "Manufacturer nr"
 	1    2250 5650
@@
 F 2 "Capacitor_SMD:C_1206_3216Metric" H 1138 4050 50  0001 C CNN
 F 3 "http://www.farnell.com/datasheets/1901289.pdf?_ga=2.262491141.804204398.1540810031-466615820.1533907205&_gac=1.154756810.1540810031.CjwKCAjw39reBRBJEiwAO1m0OUdqKKSX6YgNsFqfn4kAD7vSQS5JfvsNobbwGFQV72towt0oHUutJhoC7b8QAvD_BwE" H 1100 4200 50  0001 C CNN
-F 4 "1414715" H 1100 4200 50  0001 C CNN "Farnell"
-F 5 "C1206C104K5RACTU" H 1100 4200 50  0001 C CNN "Manufacturer nr"
+F 4 "2896646" H 1100 4200 50  0001 C CNN "Farnell"
+F 5 "VJ1206Y104KXXPW1BC" H 1100 4200 50  0001 C CNN "Manufacturer nr"
 	1    1100 4200
 	1    0    0    -1
@@
 F 2 "Capacitor_SMD:C_1206_3216Metric" H 3788 4050 50  0001 C CNN
 F 3 "http://www.farnell.com/datasheets/1901289.pdf?_ga=2.262491141.804204398.1540810031-466615820.1533907205&_gac=1.154756810.1540810031.CjwKCAjw39reBRBJEiwAO1m0OUdqKKSX6YgNsFqfn4kAD7vSQS5JfvsNobbwGFQV72towt0oHUutJhoC7b8QAvD_BwE" H 3750 4200 50  0001 C CNN
-F 4 "1414715" H 3750 4200 50  0001 C CNN "Farnell"
-F 5 "C1206C104K5RACTU" H 3750 4200 50  0001 C CNN "Manufacturer nr"
+F 4 "2896646" H 3750 4200 50  0001 C CNN "Farnell"
+F 5 "VJ1206Y104KXXPW1BC" H 3750 4200 50  0001 C CNN "Manufacturer nr"
 	1    3750 4200
 	1    0    0    -1
@@
 F 2 "Capacitor_SMD:C_1206_3216Metric" H 1138 5550 50  0001 C CNN
 F 3 "http://www.farnell.com/datasheets/1901289.pdf?_ga=2.262491141.804204398.1540810031-466615820.1533907205&_gac=1.154756810.1540810031.CjwKCAjw39reBRBJEiwAO1m0OUdqKKSX6YgNsFqfn4kAD7vSQS5JfvsNobbwGFQV72towt0oHUutJhoC7b8QAvD_BwE" H 1100 5700 50  0001 C CNN
-F 4 "1414715" H 1100 5700 50  0001 C CNN "Farnell"
-F 5 "C1206C104K5RACTU" H 1100 5700 50  0001 C CNN "Manufacturer nr"
+F 4 "2896646" H 1100 5700 50  0001 C CNN "Farnell"
+F 5 "VJ1206Y104KXXPW1BC" H 1100 5700 50  0001 C CNN "Manufacturer nr"
 	1    1100 5700
 	1    0    0    -1
