File: KiCad/BackplanePCB_solder2/BackplanePCB_solder.sch (KiCad schematic (older format))
At the start: 29 parts, among them J1 Conn_02x05_Odd_Even, J10 Conn_01x03, J11 Conn_01x03, J12 Conn_01x03, J13 Conn_01x03, J14 Conn_01x03, J15 Conn_01x03, J16 DB15_Female_MountingHoles, J17 DB15_Female_MountingHoles, J18 Conn_01x03, J19 DB15_Female_MountingHoles, J2 Conn_02x05_Odd_Even, J20 DB15_Female_MountingHoles, J21 DB15_Female_MountingHoles, J22 DB15_Female_MountingHoles, J23 DB15_Female_MountingHoles, J24 DB15_Female_MountingHoles, J3 PowerBug+15V, J4 PowerBug_GND, J5 Conn_01x03, J6 Conn_01x03, J7 Conn_01x03, J8 DB15_Female_MountingHoles, J9 DB15_Female_MountingHoles

Commit message: Updating design according to findings on proto (LEFT  config). Still some spces between sub -d screws is NOK.
Changed lines of the file:
@@
 +15V
 Text Label 3350 3250 0    50   ~ 0
-ID_1
+ID_10
 Text Label 3350 2050 0    50   ~ 0
 PWMO2_1
@@
 +15V
 Text Label 5000 3250 0    50   ~ 0
-ID_2
+ID_9
 Text Label 5000 2050 0    50   ~ 0
 PWMO2_2
@@
 +15V
 Text Label 6600 3250 0    50   ~ 0
-ID_3
+ID_8
 Text Label 6600 2050 0    50   ~ 0
 PWMO2_3
@@
 +15V
 Text Label 8150 3250 0    50   ~ 0
-ID_4
+ID_7
 Text Label 8150 2050 0    50   ~ 0
 PWMO2_4
@@
 +15V
 Text Label 9750 3250 0    50   ~ 0
-ID_5
+ID_6
 Text Label 9750 2050 0    50   ~ 0
 PWMO2_5
@@
 +15V
 Text Label 3350 5550 0    50   ~ 0
-ID_6
+ID_5
 Text Label 3350 4350 0    50   ~ 0
 PWMO2_6
@@
 +15V
 Text Label 5000 5550 0    50   ~ 0
-ID_7
+ID_4
 Text Label 5000 4350 0    50   ~ 0
 PWMO2_7
@@
 +15V
 Text Label 6600 5550 0    50   ~ 0
-ID_8
+ID_3
 Text Label 6600 4350 0    50   ~ 0
 PWMO2_8
@@
 +15V
 Text Label 8150 5550 0    50   ~ 0
-ID_9
+ID_2
 Text Label 8150 4350 0    50   ~ 0
 PWMO2_9
@@
 +15V
 Text Label 9750 5550 0    50   ~ 0
-ID_10
+ID_1
 Text Label 9750 4350 0    50   ~ 0
 PWMO2_10
@@
 Wire Wire Line
 	6000 6350 6400 6350
+Text Label 3150 6850 0    50   ~ 0
+GND
+Text Label 3150 7350 0    50   ~ 0
+GND
+Text Label 4100 6350 0    50   ~ 0
+GND
+Text Label 4100 6850 0    50   ~ 0
+GND
+Text Label 4100 7350 0    50   ~ 0
+GND
+Text Label 5050 6350 0    50   ~ 0
+GND
+Text Label 5050 6850 0    50   ~ 0
+GND
+Text Label 5050 7350 0    50   ~ 0
+GND
+Text Label 6000 6350 0    50   ~ 0
+GND
 Wire Bus Line
 	5900 6050 5900 6550
@@
 Wire Bus Line
 	3050 1950 3050 3750
-Text Label 3150 6850 0    50   ~ 0
-GND
-Text Label 3150 7350 0    50   ~ 0
-GND
-Text Label 4100 6350 0    50   ~ 0
-GND
-Text Label 4100 6850 0    50   ~ 0
-GND
-Text Label 4100 7350 0    50   ~ 0
-GND
-Text Label 5050 6350 0    50   ~ 0
-GND
-Text Label 5050 6850 0    50   ~ 0
-GND
-Text Label 5050 7350 0    50   ~ 0
-GND
-Text Label 6000 6350 0    50   ~ 0
-GND
 $EndSCHEMATC

Commit message: Revert to working version of commit on 16-10-18
Changed lines of the file:
@@
 +15V
 Text Label 3350 3250 0    50   ~ 0
-ID_10
+ID_1
 Text Label 3350 2050 0    50   ~ 0
 PWMO2_1
@@
 +15V
 Text Label 5000 3250 0    50   ~ 0
-ID_9
+ID_2
 Text Label 5000 2050 0    50   ~ 0
 PWMO2_2
@@
 +15V
 Text Label 6600 3250 0    50   ~ 0
-ID_8
+ID_3
 Text Label 6600 2050 0    50   ~ 0
 PWMO2_3
@@
 +15V
 Text Label 8150 3250 0    50   ~ 0
-ID_7
+ID_4
 Text Label 8150 2050 0    50   ~ 0
 PWMO2_4
@@
 +15V
 Text Label 9750 3250 0    50   ~ 0
-ID_6
+ID_5
 Text Label 9750 2050 0    50   ~ 0
 PWMO2_5
@@
 +15V
 Text Label 3350 5550 0    50   ~ 0
-ID_5
+ID_6
 Text Label 3350 4350 0    50   ~ 0
 PWMO2_6
@@
 +15V
 Text Label 5000 5550 0    50   ~ 0
-ID_4
+ID_7
 Text Label 5000 4350 0    50   ~ 0
 PWMO2_7
@@
 +15V
 Text Label 6600 5550 0    50   ~ 0
-ID_3
+ID_8
 Text Label 6600 4350 0    50   ~ 0
 PWMO2_8
@@
 +15V
 Text Label 8150 5550 0    50   ~ 0
-ID_2
+ID_9
 Text Label 8150 4350 0    50   ~ 0
 PWMO2_9
@@
 +15V
 Text Label 9750 5550 0    50   ~ 0
-ID_1
+ID_10
 Text Label 9750 4350 0    50   ~ 0
 PWMO2_10
@@
 Wire Wire Line
 	6000 6350 6400 6350
+Wire Bus Line
+	5900 6050 5900 6550
+Wire Bus Line
+	3050 6050 3050 7450
+Wire Bus Line
+	4000 6050 4000 7550
+Wire Bus Line
+	4950 6050 4950 7550
+Wire Bus Line
+	800  1150 800  3750
+Wire Bus Line
+	2650 1750 2650 3750
+Wire Bus Line
+	800  3750 800  7450
+Wire Bus Line
+	9450 4250 9450 6050
+Wire Bus Line
+	7850 4250 7850 6050
+Wire Bus Line
+	6300 4250 6300 6050
+Wire Bus Line
+	4700 4250 4700 6050
+Wire Bus Line
+	3050 4250 3050 6050
+Wire Bus Line
+	9450 1950 9450 3750
+Wire Bus Line
+	7850 1950 7850 3750
+Wire Bus Line
+	6300 1950 6300 3750
+Wire Bus Line
+	4700 1950 4700 3750
+Wire Bus Line
+	3050 1950 3050 3750
 Text Label 3150 6850 0    50   ~ 0
 GND
@@
 Text Label 6000 6350 0    50   ~ 0
 GND
-Wire Bus Line
-	5900 6050 5900 6550
-Wire Bus Line
-	3050 6050 3050 7450
-Wire Bus Line
-	4000 6050 4000 7550
-Wire Bus Line
-	4950 6050 4950 7550
-Wire Bus Line
-	800  1150 800  3750
-Wire Bus Line
-	2650 1750 2650 3750
-Wire Bus Line
-	800  3750 800  7450
-Wire Bus Line
-	9450 4250 9450 6050
-Wire Bus Line
-	7850 4250 7850 6050
-Wire Bus Line
-	6300 4250 6300 6050
-Wire Bus Line
-	4700 4250 4700 6050
-Wire Bus Line
-	3050 4250 3050 6050
-Wire Bus Line
-	9450 1950 9450 3750
-Wire Bus Line
-	7850 1950 7850 3750
-Wire Bus Line
-	6300 1950 6300 3750
-Wire Bus Line
-	4700 1950 4700 3750
-Wire Bus Line
-	3050 1950 3050 3750
 $EndSCHEMATC
