File: KiCad/BackplanePCB_solder2/BackplanePCB_solder.sch (KiCad schematic (older format))
At the start: 29 parts, among them J1 Conn_02x05_Odd_Even, J10 Conn_01x03, J11 Conn_01x03, J12 Conn_01x03, J13 Conn_01x03, J14 Conn_01x03, J15 Conn_01x03, J16 DB15_Female_MountingHoles, J17 DB15_Female_MountingHoles, J18 Conn_01x03, J19 DB15_Female_MountingHoles, J2 Conn_02x05_Odd_Even, J20 DB15_Female_MountingHoles, J21 DB15_Female_MountingHoles, J22 DB15_Female_MountingHoles, J23 DB15_Female_MountingHoles, J24 DB15_Female_MountingHoles, J3 PowerBug+15V, J4 PowerBug_GND, J5 Conn_01x03, J6 Conn_01x03, J7 Conn_01x03, J8 DB15_Female_MountingHoles, J9 DB15_Female_MountingHoles

Commit message: Backplane PCB updates
Changed lines of the file:
@@
 Text Label 3350 2850 0    50   ~ 0
 SYNC_B
+Text Label 3350 2550 0    50   ~ 0
+TX_A
+Text Label 3350 2450 0    50   ~ 0
+TX_B
 Text Label 3350 2750 0    50   ~ 0
-TX_A
+RX_A
 Text Label 3350 2650 0    50   ~ 0
-TX_B
-Text Label 3350 2550 0    50   ~ 0
-RX_A
-Text Label 3350 2450 0    50   ~ 0
 RX_B
 Entry Wire Line
@@
 +15V
 Text Label 3350 3250 0    50   ~ 0
-ID_1
+ID_10
 Text Label 3350 2050 0    50   ~ 0
 PWMO2_1
@@
 Text Label 5000 2850 0    50   ~ 0
 SYNC_B
+Text Label 5000 2550 0    50   ~ 0
+TX_A
+Text Label 5000 2450 0    50   ~ 0
+TX_B
 Text Label 5000 2750 0    50   ~ 0
-TX_A
+RX_A
 Text Label 5000 2650 0    50   ~ 0
-TX_B
-Text Label 5000 2550 0    50   ~ 0
-RX_A
-Text Label 5000 2450 0    50   ~ 0
 RX_B
 Text Label 5000 3650 0    50   ~ 0
@@
 +15V
 Text Label 5000 3250 0    50   ~ 0
-ID_2
+ID_9
 Text Label 5000 2050 0    50   ~ 0
 PWMO2_2
@@
 Text Label 6600 2850 0    50   ~ 0
 SYNC_B
+Text Label 6600 2550 0    50   ~ 0
+TX_A
+Text Label 6600 2450 0    50   ~ 0
+TX_B
 Text Label 6600 2750 0    50   ~ 0
-TX_A
+RX_A
 Text Label 6600 2650 0    50   ~ 0
-TX_B
-Text Label 6600 2550 0    50   ~ 0
-RX_A
-Text Label 6600 2450 0    50   ~ 0
 RX_B
 Text Label 6600 3650 0    50   ~ 0
@@
 +15V
 Text Label 6600 3250 0    50   ~ 0
-ID_3
+ID_8
 Text Label 6600 2050 0    50   ~ 0
 PWMO2_3
@@
 Text Label 8150 2850 0    50   ~ 0
 SYNC_B
+Text Label 8150 2550 0    50   ~ 0
+TX_A
+Text Label 8150 2450 0    50   ~ 0
+TX_B
 Text Label 8150 2750 0    50   ~ 0
-TX_A
+RX_A
 Text Label 8150 2650 0    50   ~ 0
-TX_B
-Text Label 8150 2550 0    50   ~ 0
-RX_A
-Text Label 8150 2450 0    50   ~ 0
 RX_B
 Text Label 8150 3650 0    50   ~ 0
@@
 +15V
 Text Label 8150 3250 0    50   ~ 0
-ID_4
+ID_7
 Text Label 8150 2050 0    50   ~ 0
 PWMO2_4
@@
 Text Label 9750 2850 0    50   ~ 0
 SYNC_B
+Text Label 9750 2550 0    50   ~ 0
+TX_A
+Text Label 9750 2450 0    50   ~ 0
+TX_B
 Text Label 9750 2750 0    50   ~ 0
-TX_A
+RX_A
 Text Label 9750 2650 0    50   ~ 0
-TX_B
-Text Label 9750 2550 0    50   ~ 0
-RX_A
-Text Label 9750 2450 0    50   ~ 0
 RX_B
 Text Label 9750 3650 0    50   ~ 0
@@
 +15V
 Text Label 9750 3250 0    50   ~ 0
-ID_5
+ID_6
 Text Label 9750 2050 0    50   ~ 0
 PWMO2_5
@@
 Text Label 3350 5150 0    50   ~ 0
 SYNC_B
+Text Label 3350 4850 0    50   ~ 0
+TX_A
+Text Label 3350 4750 0    50   ~ 0
+TX_B
 Text Label 3350 5050 0    50   ~ 0
-TX_A
+RX_A
 Text Label 3350 4950 0    50   ~ 0
-TX_B
-Text Label 3350 4850 0    50   ~ 0
-RX_A
-Text Label 3350 4750 0    50   ~ 0
 RX_B
 Text Label 3350 5950 0    50   ~ 0
@@
 +15V
 Text Label 3350 5550 0    50   ~ 0
-ID_6
+ID_5
 Text Label 3350 4350 0    50   ~ 0
 PWMO2_6
@@
 Text Label 5000 5150 0    50   ~ 0
 SYNC_B
+Text Label 5000 4850 0    50   ~ 0
+TX_A
+Text Label 5000 4750 0    50   ~ 0
+TX_B
 Text Label 5000 5050 0    50   ~ 0
-TX_A
+RX_A
 Text Label 5000 4950 0    50   ~ 0
-TX_B
-Text Label 5000 4850 0    50   ~ 0
-RX_A
-Text Label 5000 4750 0    50   ~ 0
 RX_B
 Text Label 5000 5950 0    50   ~ 0
@@
 +15V
 Text Label 5000 5550 0    50   ~ 0
-ID_7
+ID_4
 Text Label 5000 4350 0    50   ~ 0
 PWMO2_7
@@
 Text Label 6600 5150 0    50   ~ 0
 SYNC_B
+Text Label 6600 4850 0    50   ~ 0
+TX_A
+Text Label 6600 4750 0    50   ~ 0
+TX_B
 Text Label 6600 5050 0    50   ~ 0
-TX_A
+RX_A
 Text Label 6600 4950 0    50   ~ 0
-TX_B
-Text Label 6600 4850 0    50   ~ 0
-RX_A
-Text Label 6600 4750 0    50   ~ 0
 RX_B
 Text Label 6600 5950 0    50   ~ 0
@@
 +15V
 Text Label 6600 5550 0    50   ~ 0
-ID_8
+ID_3
 Text Label 6600 4350 0    50   ~ 0
 PWMO2_8
@@
 Text Label 8150 5150 0    50   ~ 0
 SYNC_B
+Text Label 8150 4850 0    50   ~ 0
+TX_A
+Text Label 8150 4750 0    50   ~ 0
+TX_B
 Text Label 8150 5050 0    50   ~ 0
-TX_A
+RX_A
 Text Label 8150 4950 0    50   ~ 0
-TX_B
-Text Label 8150 4850 0    50   ~ 0
-RX_A
-Text Label 8150 4750 0    50   ~ 0
 RX_B
 Text Label 8150 5950 0    50   ~ 0
@@
 +15V
 Text Label 8150 5550 0    50   ~ 0
-ID_9
+ID_2
 Text Label 8150 4350 0    50   ~ 0
 PWMO2_9
@@
 Text Label 9750 5150 0    50   ~ 0
 SYNC_B
+Text Label 9750 4850 0    50   ~ 0
+TX_A
+Text Label 9750 4750 0    50   ~ 0
+TX_B
 Text Label 9750 5050 0    50   ~ 0
-TX_A
+RX_A
 Text Label 9750 4950 0    50   ~ 0
-TX_B
-Text Label 9750 4850 0    50   ~ 0
-RX_A
-Text Label 9750 4750 0    50   ~ 0
 RX_B
 Text Label 9750 5950 0    50   ~ 0
@@
 +15V
 Text Label 9750 5550 0    50   ~ 0
-ID_10
+ID_1
 Text Label 9750 4350 0    50   ~ 0
 PWMO2_10
@@
 Wire Wire Line
 	6000 6350 6400 6350
+Text Label 3150 6850 0    50   ~ 0
+GND
+Text Label 3150 7350 0    50   ~ 0
+GND
+Text Label 4100 6350 0    50   ~ 0
+GND
+Text Label 4100 6850 0    50   ~ 0
+GND
+Text Label 4100 7350 0    50   ~ 0
+GND
+Text Label 5050 6350 0    50   ~ 0
+GND
+Text Label 5050 6850 0    50   ~ 0
+GND
+Text Label 5050 7350 0    50   ~ 0
+GND
+Text Label 6000 6350 0    50   ~ 0
+GND
 Wire Bus Line
 	5900 6050 5900 6550
@@
 Wire Bus Line
 	3050 1950 3050 3750
-Text Label 3150 6850 0    50   ~ 0
-GND
-Text Label 3150 7350 0    50   ~ 0
-GND
-Text Label 4100 6350 0    50   ~ 0
-GND
-Text Label 4100 6850 0    50   ~ 0
-GND
-Text Label 4100 7350 0    50   ~ 0
-GND
-Text Label 5050 6350 0    50   ~ 0
-GND
-Text Label 5050 6850 0    50   ~ 0
-GND
-Text Label 5050 7350 0    50   ~ 0
-GND
-Text Label 6000 6350 0    50   ~ 0
-GND
 $EndSCHEMATC
