File: KiCad/BackplanePCB_solder2/BackplanePCB_solder.kicad_pcb_LEFT.kicad_pcb (KiCad board)
At the start: 2 copper layers, 280 x 59 mm, 76 parts, among them J1 Conn_02x05_Odd_Even, J10 Conn_01x03, J11 Conn_01x03, J12 Conn_01x03, J16 DB15_Female_MountingHoles, J19 DB15_Female_MountingHoles, J21 DB15_Female_MountingHoles, J23 DB15_Female_MountingHoles, J25 Conn_01x06, J3 PowerBug+15V, J4 PowerBug_GND, J5 Conn_01x03, J6 Conn_01x03, J7 Conn_01x03, J8 DB15_Female_MountingHoles, J9 DB15_Female_MountingHoles, Q1 Q_NMOS_GSD, U1 ST485EBDR, U2 ST485EBDR, U3 ST485EBDR, U4 KA78M05_TO252, U5 ST485EBDR, U6 PIC16F18854-SO

Commit message: updated BackplanePCB_solder2 PCB for prototyping and production.
Routing:
- net ID_7: track 130.2 -> 131.6 mm
- net ID_9: track 129.7 -> 131.0 mm
- net GND: track 263.3 -> 262.4 mm
- net ID_10: track 136.0 -> 136.7 mm
- net Net-(C18-Pad1): track 17.6 -> 16.9 mm
Other:
- rule via_min_drill: 0.3 -> 0.4
- rule via_min_size: 0.6 -> 0.8

Commit message: Backplane PCB updates
Parts:
- moved R15 1.49 mm to (177.3, 175.7)
- moved R16 1.35 mm to (177.3, 177.1)
Routing:
- net Net-(R16-Pad1): track 2.50 -> 7.84 mm
- net Net-(R15-Pad1): track 2.56 -> 3.68 mm
