File: KiCad/MCP6N11 piggy back/MCP6N11_piggy_back.sch (KiCad schematic (older format))
At the start: 19 parts, among them J1 Conn_01x02_Male, J2 Conn_01x01_Male, J4 Conn_01x02_Male, J5 Conn_01x02_Male, U1 MCP6N11

Commit message: updated MCP6N11 piggy back/MCP6N11_piggy_back.sch
Parts:
- R1, R2: value 4k99 -> 9k10
- R8: value 1k -> 100k
Other:
- note added: "see page 9, Gmin = 1 and is 1 when Rf = 0 Ohm and Rg = open"
Changed lines of the file:
@@
 P 3350 3250
 F 0 "R1" V 3430 3250 50  0000 C CNN
-F 1 "4k99" V 3350 3250 50  0000 C CNN
+F 1 "9k10" V 3350 3250 50  0000 C CNN
 F 2 "Resistor_SMD:R_1206_3216Metric" V 3280 3250 50  0001 C CNN
 F 3 "~" H 3350 3250 50  0001 C CNN
@@
 P 3350 3650
 F 0 "R2" V 3430 3650 50  0000 C CNN
-F 1 "4k99" V 3350 3650 50  0000 C CNN
+F 1 "9k10" V 3350 3650 50  0000 C CNN
 F 2 "Resistor_SMD:R_1206_3216Metric" V 3280 3650 50  0001 C CNN
 F 3 "~" H 3350 3650 50  0001 C CNN
@@
 P 6150 4050
 F 0 "R8" V 6230 4050 50  0000 C CNN
-F 1 "1k" V 6150 4050 50  0000 C CNN
+F 1 "100k" V 6150 4050 50  0000 C CNN
 F 2 "Resistor_SMD:R_1206_3216Metric" V 6080 4050 50  0001 C CNN
 F 3 "~" H 6150 4050 50  0001 C CNN
@@
 Wire Wire Line
 	5200 4000 5200 4250
+Text Notes 5850 4350 0    50   ~ 0
+see page 9, Gmin = 1 and is 1 when Rf = 0 Ohm and Rg = open
 $EndSCHEMATC

Commit message: fault in schemtic regarding Rf and Rg
Connections:
- wire segments 66 -> 65
Changed lines of the file:
@@
 L Device:R R7
 U 1 1 5BB5BCC5
-P 5850 3800
-F 0 "R7" V 5930 3800 50  0000 C CNN
-F 1 "1k" V 5850 3800 50  0000 C CNN
-F 2 "Resistor_SMD:R_1206_3216Metric" V 5780 3800 50  0001 C CNN
-F 3 "~" H 5850 3800 50  0001 C CNN
-	1    5850 3800
-	0    -1   -1   0
+P 6150 3700
+F 0 "R7" V 6230 3700 50  0000 C CNN
+F 1 "1k" V 6150 3700 50  0000 C CNN
+F 2 "Resistor_SMD:R_1206_3216Metric" V 6080 3700 50  0001 C CNN
+F 3 "~" H 6150 3700 50  0001 C CNN
+	1    6150 3700
+	-1   0    0    1
 $EndComp
 $Comp
@@
 	0    -1   -1   0
 $EndComp
-Wire Wire Line
-	5850 3450 6150 3450
 $Comp
 L power:GND #PWR07
@@
 	3100 3500 3100 3650
 Wire Wire Line
-	5700 3800 5050 3800
-Wire Wire Line
-	5050 3800 5050 3350
-Wire Wire Line
 	5050 3350 5150 3350
 Wire Wire Line
-	6000 3800 6150 3800
-Wire Wire Line
-	6150 3800 6150 3450
-Connection ~ 6150 3450
-Wire Wire Line
-	6150 3450 6750 3450
-Wire Wire Line
-	6150 3900 6150 3800
-Connection ~ 6150 3800
-Wire Wire Line
 	6150 4200 6150 4250
 Wire Wire Line
@@
 Wire Wire Line
 	5550 4250 5550 4000
-Text Notes 5800 3950 0    50   ~ 0
+Text Notes 6200 3750 0    50   ~ 0
 Rf
 Text Notes 6200 4100 0    50   ~ 0
@@
 Text Notes 5850 4350 0    50   ~ 0
 see page 9, Gmin = 1 and is 1 when Rf = 0 Ohm and Rg = open
+Wire Wire Line
+	5850 3450 6150 3450
+Wire Wire Line
+	6150 3550 6150 3450
+Connection ~ 6150 3450
+Wire Wire Line
+	6150 3450 6750 3450
+Wire Wire Line
+	6150 3850 6150 3900
+Wire Wire Line
+	5050 3850 6150 3850
+Wire Wire Line
+	5050 3350 5050 3850
+Connection ~ 6150 3850
 $EndSCHEMATC
