File: KiCad/TrackModBusMaster_piggyback/TrackModBusMaster_piggyback.sch (KiCad schematic (older format))
At the start: 31 parts

Commit message: updating piggyback modbusmaster
Parts:
- added C14, C15, C16, C17: 22p, Capacitor_SMD:C_1206_3216Metric, symbol Device:C
- added C18: 2.2u, Capacitor_SMD:C_1206_3216Metric, symbol Device:C
- added D1, D4, D5: LED GR, LED_SMD:LED_1206_3216Metric, symbol Device:LED
- added D2: LED YE, LED_SMD:LED_1206_3216Metric, symbol Device:LED
- added D3: LED RD, LED_SMD:LED_1206_3216Metric, symbol Device:LED
- added J2: Conn_02x05_Odd_Even, Connector_IDC:IDC-Header_2x05_P2.54mm_Vertical, symbol Connector_Generic:Conn_02x05_Odd_Even
- added J4: Conn_01x08, Connector_PinHeader_2.54mm:PinHeader_1x08_P2.54mm_Vertical, symbol Connector_Generic:Conn_01x08
- added R12, R19, R20, R21, R26, R5: 4k7, Resistor_SMD:R_1206_3216Metric, symbol Device:R
- added R14, R15, R16, R17, R18: 301E, Resistor_SMD:R_1206_3216Metric, symbol Device:R
- added R22: 100k, Resistor_SMD:R_1206_3216Metric, symbol Device:R
- added R23: 10k, Resistor_SMD:R_1206_3216Metric, symbol Device:R
- added R24, R25: 470E, Resistor_SMD:R_1206_3216Metric, symbol Device:R
- added R7: 3k9, Resistor_SMD:R_1206_3216Metric, symbol Device:R
- added R8: 120E, Resistor_SMD:R_1206_3216Metric, symbol Device:R
- added R9: 1k00, Resistor_SMD:R_1206_3216Metric, symbol Device:R
- J1, J3: renamed from J?; footprint (none) -> Connector_PinHeader_2.54mm:PinHeader_2x08_P2.54mm_Vertical; symbol Connector_Generic:Conn_02x08_Top_Bottom -> Connector_Generic:Conn_02x08_Odd_Even
- J5: renamed from J?; footprint (none) -> Connector_PinHeader_2.54mm:PinHeader_1x08_P2.54mm_Vertical
- gave numbers to parts that had none: 28
Connections:
- net labels added: Reset_Out, Rx_A, Rx_B, SCK1, SDI, SDO, SS1, Sync, Sync_A, Sync_B, Tx_En
- wire segments 169 -> 307
- no-connect marks 6 -> 22

Commit message: updated TrackModBusMaster_piggyback
Connections:
- net labels added: +3.3VP
- wire segments 307 -> 310
- no-connect marks 22 -> 21
Changed lines of the file:
@@
-	1    0    0    -1
-$EndComp
-$Comp
-L power:+3.3V #PWR07
-U 1 1 5BCE517A
-P 2650 700
-F 0 "#PWR07" H 2650 550 50  0001 C CNN
-F 1 "+3.3V" H 2650 840 50  0000 C CNN
-F 2 "" H 2650 700 50  0001 C CNN
-F 3 "" H 2650 700 50  0001 C CNN
-	1    2650 700
 	1    0    0    -1
 $EndComp
@@
 Wire Wire Line
 	3350 1350 2650 1350
-Wire Wire Line
-	2650 1350 2650 700
 Wire Wire Line
 	3350 1450 2650 1450
@@
 Wire Wire Line
 	5750 5250 5900 5250
-Text GLabel 3250 2000 0    50   Input ~ 0
+Text GLabel 3150 2400 0    50   Input ~ 0
 Reset_A
-Text GLabel 3950 2000 2    50   Input ~ 0
+Text GLabel 4050 2400 2    50   Input ~ 0
 Reset_B
 $Comp
@@
 	1    0    0    -1
 $EndComp
-Text GLabel 3950 2100 2    50   Input ~ 0
+Text GLabel 4050 2100 2    50   Input ~ 0
 Tx_B
-Text GLabel 3250 2100 0    50   Input ~ 0
+Text GLabel 3150 2100 0    50   Input ~ 0
 Tx_A
-Text GLabel 3250 2200 0    50   Output ~ 0
+Text GLabel 3150 2000 0    50   Output ~ 0
 Rx_A
-Text GLabel 3950 2200 2    50   Output ~ 0
+Text GLabel 4050 2000 2    50   Output ~ 0
 Rx_B
-Text GLabel 3250 2300 0    50   Input ~ 0
+Text GLabel 3150 2300 0    50   Input ~ 0
 Sync_A
-Text GLabel 3950 2300 2    50   Input ~ 0
+Text GLabel 4050 2300 2    50   Input ~ 0
 Sync_B
-$Comp
-L power:GND #PWR014
-U 1 1 5BBA9943
-P 3250 2450
-F 0 "#PWR014" H 3250 2200 50  0001 C CNN
-F 1 "GND" H 3250 2300 50  0000 C CNN
-F 2 "" H 3250 2450 50  0001 C CNN
-F 3 "" H 3250 2450 50  0001 C CNN
-	1    3250 2450
-	1    0    0    -1
-$EndComp
-$Comp
-L power:GND #PWR020
-U 1 1 5BBA9990
-P 3950 2450
-F 0 "#PWR020" H 3950 2200 50  0001 C CNN
-F 1 "GND" H 3950 2300 50  0000 C CNN
-F 2 "" H 3950 2450 50  0001 C CNN
-F 3 "" H 3950 2450 50  0001 C CNN
-	1    3950 2450
-	1    0    0    -1
-$EndComp
-Wire Wire Line
-	3250 2000 3350 2000
-Wire Wire Line
-	3250 2100 3350 2100
-Wire Wire Line
-	3350 2200 3250 2200
-Wire Wire Line
-	3250 2300 3350 2300
-Wire Wire Line
-	3350 2400 3250 2400
-Wire Wire Line
-	3250 2400 3250 2450
-Wire Wire Line
-	3850 2400 3950 2400
-Wire Wire Line
-	3950 2400 3950 2450
-Wire Wire Line
-	3950 2300 3850 2300
-Wire Wire Line
-	3850 2200 3950 2200
-Wire Wire Line
-	3950 2100 3850 2100
-Wire Wire Line
-	3850 2000 3950 2000
 $Comp
 L power:+3.3V #PWR022
@@
 NoConn ~ 5150 950
 NoConn ~ 5150 850
-NoConn ~ 5150 750
+$Comp
+L power:+3.3V #PWR0101
+U 1 1 5BBCC540
+P 5200 700
+F 0 "#PWR0101" H 5200 550 50  0001 C CNN
+F 1 "+3.3V" H 5200 840 50  0000 C CNN
+F 2 "" H 5200 700 50  0001 C CNN
+F 3 "" H 5200 700 50  0001 C CNN
+	1    5200 700
+	1    0    0    -1
+$EndComp
+Wire Wire Line
+	5200 700  5200 750
+Wire Wire Line
+	5200 750  5150 750
+$Comp
+L power:+3.3VP #PWR0102
+U 1 1 5BC6E62D
+P 2650 650
+F 0 "#PWR0102" H 2800 600 50  0001 C CNN
+F 1 "+3.3VP" H 2650 750 50  0000 C CNN
+F 2 "" H 2650 650 50  0001 C CNN
+F 3 "" H 2650 650 50  0001 C CNN
+	1    2650 650
+	1    0    0    -1
+$EndComp
+Wire Wire Line
+	2650 650  2650 1350
+$Comp
+L power:GND #PWR020
+U 1 1 5BBA9990
+P 3950 2450
+F 0 "#PWR020" H 3950 2200 50  0001 C CNN
+F 1 "GND" H 3950 2300 50  0000 C CNN
+F 2 "" H 3950 2450 50  0001 C CNN
+F 3 "" H 3950 2450 50  0001 C CNN
+	1    3950 2450
+	1    0    0    -1
+$EndComp
+$Comp
+L power:GND #PWR014
+U 1 1 5BBA9943
+P 3250 2450
+F 0 "#PWR014" H 3250 2200 50  0001 C CNN
+F 1 "GND" H 3250 2300 50  0000 C CNN
+F 2 "" H 3250 2450 50  0001 C CNN
+F 3 "" H 3250 2450 50  0001 C CNN
+	1    3250 2450
+	1    0    0    -1
+$EndComp
+Wire Wire Line
+	3150 2000 3350 2000
+Wire Wire Line
+	3350 2100 3150 2100
+Wire Wire Line
+	3150 2300 3350 2300
+Wire Wire Line
+	3350 2400 3150 2400
+Wire Wire Line
+	3250 2450 3250 2200
+Wire Wire Line
+	3250 2200 3350 2200
+Wire Wire Line
+	3850 2200 3950 2200
+Wire Wire Line
+	3950 2200 3950 2450
+Wire Wire Line
+	4050 2400 3850 2400
+Wire Wire Line
+	3850 2300 4050 2300
+Wire Wire Line
+	4050 2100 3850 2100
+Wire Wire Line
+	3850 2000 4050 2000
+Wire Wire Line
+	3150 4450 3150 4500
 $EndSCHEMATC

Commit message: Finished TrackModBusMaster_piggyback
Connections:
- wire segments 310 -> 312
- no-connect marks 21 -> 20
Changed lines of the file:
@@
 L Connector_Generic:Conn_02x08_Odd_Even J1
 U 1 1 5BCE4FC3
-P 3550 1050
-F 0 "J1" H 3600 1450 50  0000 C CNN
-F 1 "Conn_02x08_Top_Bottom" H 3600 1550 50  0000 C CNN
-F 2 "Connector_PinHeader_2.54mm:PinHeader_2x08_P2.54mm_Vertical" H 3550 1050 50  0001 C CNN
-F 3 "~" H 3550 1050 50  0001 C CNN
-	1    3550 1050
+P 3150 1050
+F 0 "J1" H 3200 1450 50  0000 C CNN
+F 1 "Conn_02x08_Top_Bottom" H 3200 1550 50  0000 C CNN
+F 2 "Connector_PinHeader_2.54mm:PinHeader_2x08_P2.54mm_Vertical" H 3150 1050 50  0001 C CNN
+F 3 "~" H 3150 1050 50  0001 C CNN
+	1    3150 1050
 	1    0    0    -1
 $EndComp
@@
 L power:GND #PWR011
 U 1 1 5BCE50C5
-P 3050 1550
-F 0 "#PWR011" H 3050 1300 50  0001 C CNN
-F 1 "GND" H 3050 1400 50  0000 C CNN
-F 2 "" H 3050 1550 50  0001 C CNN
-F 3 "" H 3050 1550 50  0001 C CNN
-	1    3050 1550
+P 2650 1500
+F 0 "#PWR011" H 2650 1250 50  0001 C CNN
+F 1 "GND" H 2650 1350 50  0000 C CNN
+F 2 "" H 2650 1500 50  0001 C CNN
+F 3 "" H 2650 1500 50  0001 C CNN
+	1    2650 1500
 	1    0    0    -1
 $EndComp
@@
 L power:+5V #PWR010
 U 1 1 5BCE5123
-P 2900 700
-F 0 "#PWR010" H 2900 550 50  0001 C CNN
-F 1 "+5V" H 2900 840 50  0000 C CNN
-F 2 "" H 2900 700 50  0001 C CNN
-F 3 "" H 2900 700 50  0001 C CNN
-	1    2900 700
-	1    0    0    -1
-$EndComp
-Wire Wire Line
-	3050 1550 3050 1250
-Wire Wire Line
-	3050 750  3350 750
-Wire Wire Line
-	3350 850  3050 850
-Connection ~ 3050 850
-Wire Wire Line
-	3050 850  3050 750
-Wire Wire Line
-	3350 950  2900 950
-Wire Wire Line
-	2900 950  2900 700
-Wire Wire Line
-	3350 1050 2900 1050
-Wire Wire Line
-	2900 1050 2900 950
-Connection ~ 2900 950
-Wire Wire Line
-	3350 1150 3050 1150
-Connection ~ 3050 1150
-Wire Wire Line
-	3050 1150 3050 850
-Wire Wire Line
-	3350 1250 3050 1250
-Connection ~ 3050 1250
-Wire Wire Line
-	3050 1250 3050 1150
-Wire Wire Line
-	3350 1350 2650 1350
-Wire Wire Line
-	3350 1450 2650 1450
-Wire Wire Line
-	2650 1450 2650 1350
-Connection ~ 2650 1350
+P 2500 700
+F 0 "#PWR010" H 2500 550 50  0001 C CNN
+F 1 "+5V" H 2500 840 50  0000 C CNN
+F 2 "" H 2500 700 50  0001 C CNN
+F 3 "" H 2500 700 50  0001 C CNN
+	1    2500 700
+	1    0    0    -1
+$EndComp
+Wire Wire Line
+	2650 750  2950 750
+Wire Wire Line
+	2950 850  2650 850
+Connection ~ 2650 850
+Wire Wire Line
+	2650 850  2650 750
+Wire Wire Line
+	2950 950  2500 950
+Wire Wire Line
+	2500 950  2500 700
+Wire Wire Line
+	2950 1050 2500 1050
+Wire Wire Line
+	2500 1050 2500 950
+Connection ~ 2500 950
+Wire Wire Line
+	2950 1150 2650 1150
+Connection ~ 2650 1150
+Wire Wire Line
+	2650 1150 2650 850
+Wire Wire Line
+	2950 1250 2650 1250
+Wire Wire Line
+	2650 1250 2650 1150
+Wire Wire Line
+	2950 1350 2250 1350
+Wire Wire Line
+	2950 1450 2250 1450
+Wire Wire Line
+	2250 1450 2250 1350
+Connection ~ 2250 1350
 $Comp
 L MCU_Microchip_PIC16:PIC16F18854-SO U6
@@
 Wire Wire Line
 	7450 3200 7950 3200
-Text GLabel 3950 1350 2    50   Input ~ 0
+Text GLabel 3550 1350 2    50   Input ~ 0
 SCK1
-Text GLabel 3950 1150 2    50   Input ~ 0
+Text GLabel 3550 1150 2    50   Input ~ 0
 SS1
-Text GLabel 3950 950  2    50   Input ~ 0
+Text GLabel 3550 950  2    50   Input ~ 0
 SDO
-Text GLabel 3950 750  2    50   Output ~ 0
+Text GLabel 3550 750  2    50   Output ~ 0
 SDI
-Text GLabel 4550 600  0    50   Output ~ 0
+Text GLabel 4150 600  0    50   Output ~ 0
 Reset_Out
 $Comp
 L power:GND #PWR021
 U 1 1 5C082EC8
-P 3900 1500
-F 0 "#PWR021" H 3900 1250 50  0001 C CNN
-F 1 "GND" H 3900 1350 50  0000 C CNN
-F 2 "" H 3900 1500 50  0001 C CNN
-F 3 "" H 3900 1500 50  0001 C CNN
-	1    3900 1500
+P 3500 1500
+F 0 "#PWR021" H 3500 1250 50  0001 C CNN
+F 1 "GND" H 3500 1350 50  0000 C CNN
+F 2 "" H 3500 1500 50  0001 C CNN
+F 3 "" H 3500 1500 50  0001 C CNN
+	1    3500 1500
 	1    0    0    -1
 $EndComp
@@
 L Connector_Generic:Conn_02x08_Odd_Even J3
 U 1 1 5BCE4FFE
-P 4850 1050
-F 0 "J3" H 4900 1450 50  0000 C CNN
-F 1 "Conn_02x08_Top_Bottom" V 4900 50  50  0000 C CNN
-F 2 "Connector_PinHeader_2.54mm:PinHeader_2x08_P2.54mm_Vertical" H 4850 1050 50  0001 C CNN
-F 3 "~" H 4850 1050 50  0001 C CNN
-	1    4850 1050
-	1    0    0    -1
-$EndComp
-Wire Wire Line
-	4550 600  4650 600
-Wire Wire Line
-	4650 600  4650 750
-Wire Wire Line
-	3900 1500 3900 1450
-Wire Wire Line
-	3900 850  3850 850
-Wire Wire Line
-	3850 1050 3900 1050
-Connection ~ 3900 1050
-Wire Wire Line
-	3900 1050 3900 850
-Wire Wire Line
-	3850 1250 3900 1250
-Connection ~ 3900 1250
-Wire Wire Line
-	3900 1250 3900 1050
-Wire Wire Line
-	3850 1450 3900 1450
-Connection ~ 3900 1450
-Wire Wire Line
-	3900 1450 3900 1250
-NoConn ~ 4650 1450
-NoConn ~ 4650 1350
-NoConn ~ 4650 1250
-NoConn ~ 4650 1150
-NoConn ~ 4650 1050
-NoConn ~ 4650 950
-NoConn ~ 4650 850
-Wire Wire Line
-	3950 750  3850 750
-Wire Wire Line
-	3850 950  3950 950
-Wire Wire Line
-	3950 1150 3850 1150
-Wire Wire Line
-	3850 1350 3950 1350
+P 4500 1050
+F 0 "J3" H 4550 1450 50  0000 C CNN
+F 1 "Conn_02x08_Top_Bottom" V 4550 50  50  0000 C CNN
+F 2 "Connector_PinHeader_2.54mm:PinHeader_2x08_P2.54mm_Vertical" H 4500 1050 50  0001 C CNN
+F 3 "~" H 4500 1050 50  0001 C CNN
+	1    4500 1050
+	1    0    0    -1
+$EndComp
+Wire Wire Line
+	4300 600  4300 750
+Wire Wire Line
+	3500 1500 3500 1450
+Wire Wire Line
+	3500 850  3450 850
+Wire Wire Line
+	3450 1050 3500 1050
+Connection ~ 3500 1050
+Wire Wire Line
+	3500 1050 3500 850
+Wire Wire Line
+	3450 1250 3500 1250
+Connection ~ 3500 1250
+Wire Wire Line
+	3500 1250 3500 1050
+Wire Wire Line
+	3450 1450 3500 1450
+Connection ~ 3500 1450
+Wire Wire Line
+	3500 1450 3500 1250
+Wire Wire Line
+	3550 750  3450 750
+Wire Wire Line
+	3450 950  3550 950
+Wire Wire Line
+	3550 1150 3450 1150
+Wire Wire Line
+	3450 1350 3550 1350
 $Comp
 L Device:R R26
@@
 	1    0    0    -1
 $EndComp
-NoConn ~ 5150 1450
-NoConn ~ 5150 1350
-NoConn ~ 5150 1250
-NoConn ~ 5150 1150
-NoConn ~ 5150 1050
-NoConn ~ 5150 950
-NoConn ~ 5150 850
 $Comp
 L power:+3.3V #PWR0101
 U 1 1 5BBCC540
-P 5200 700
-F 0 "#PWR0101" H 5200 550 50  0001 C CNN
-F 1 "+3.3V" H 5200 840 50  0000 C CNN
-F 2 "" H 5200 700 50  0001 C CNN
-F 3 "" H 5200 700 50  0001 C CNN
-	1    5200 700
-	1    0    0    -1
-$EndComp
-Wire Wire Line
-	5200 700  5200 750
-Wire Wire Line
-	5200 750  5150 750
+P 4850 700
+F 0 "#PWR0101" H 4850 550 50  0001 C CNN
+F 1 "+3.3V" H 4850 840 50  0000 C CNN
+F 2 "" H 4850 700 50  0001 C CNN
+F 3 "" H 4850 700 50  0001 C CNN
+	1    4850 700
+	1    0    0    -1
+$EndComp
+Wire Wire Line
+	4850 700  4850 750
+Wire Wire Line
+	4850 750  4800 750
 $Comp
 L power:+3.3VP #PWR0102
 U 1 1 5BC6E62D
-P 2650 650
-F 0 "#PWR0102" H 2800 600 50  0001 C CNN
-F 1 "+3.3VP" H 2650 750 50  0000 C CNN
-F 2 "" H 2650 650 50  0001 C CNN
-F 3 "" H 2650 650 50  0001 C CNN
-	1    2650 650
-	1    0    0    -1
-$EndComp
-Wire Wire Line
-	2650 650  2650 1350
+P 2250 650
+F 0 "#PWR0102" H 2400 600 50  0001 C CNN
+F 1 "+3.3VP" H 2250 750 50  0000 C CNN
+F 2 "" H 2250 650 50  0001 C CNN
+F 3 "" H 2250 650 50  0001 C CNN
+	1    2250 650
+	1    0    0    -1
+$EndComp
+Wire Wire Line
+	2250 650  2250 1350
 $Comp
 L power:GND #PWR020
@@
 Wire Wire Line
 	3150 4450 3150 4500
+Wire Wire Line
+	4150 600  4300 600
+NoConn ~ 4800 950
+NoConn ~ 4800 1050
+NoConn ~ 4800 1150
+NoConn ~ 4800 1250
+NoConn ~ 4800 1350
+NoConn ~ 4800 1450
+NoConn ~ 4300 1450
+NoConn ~ 4300 1350
+NoConn ~ 4300 1250
+NoConn ~ 4300 1150
+NoConn ~ 4300 1050
+NoConn ~ 4300 950
+Wire Wire Line
+	2650 1500 2650 1250
+Connection ~ 2650 1250
+$Comp
+L power:GND #PWR?
+U 1 1 5BD9464F
+P 4200 1500
+F 0 "#PWR?" H 4200 1250 50  0001 C CNN
+F 1 "GND" H 4200 1350 50  0000 C CNN
+F 2 "" H 4200 1500 50  0001 C CNN
+F 3 "" H 4200 1500 50  0001 C CNN
+	1    4200 1500
+	1    0    0    -1
+$EndComp
+NoConn ~ 4800 850
+Wire Wire Line
+	4300 850  4200 850
+Wire Wire Line
+	4200 850  4200 1500
 $EndSCHEMATC

Commit message: update on schematic and pcb
Parts:
- added C19: 100u, Capacitor_THT:CP_Radial_D6.3mm_P2.50mm, symbol Device:CP
Connections:
- wire segments 312 -> 314
Changed lines of the file:
@@
 Connection ~ 2650 1250
 $Comp
-L power:GND #PWR?
+L power:GND #PWR033
 U 1 1 5BD9464F
 P 4200 1500
-F 0 "#PWR?" H 4200 1250 50  0001 C CNN
+F 0 "#PWR033" H 4200 1250 50  0001 C CNN
 F 1 "GND" H 4200 1350 50  0000 C CNN
 F 2 "" H 4200 1500 50  0001 C CNN
@@
 Wire Wire Line
 	4200 850  4200 1500
+$Comp
+L Device:CP C19
+U 1 1 5BBF833B
+P 1750 1200
+F 0 "C19" H 1775 1300 50  0000 L CNN
+F 1 "100u" H 1775 1100 50  0000 L CNN
+F 2 "Capacitor_THT:CP_Radial_D6.3mm_P2.50mm" H 1788 1050 50  0001 C CNN
+F 3 "~" H 1750 1200 50  0001 C CNN
+	1    1750 1200
+	1    0    0    -1
+$EndComp
+$Comp
+L power:+5V #PWR07
+U 1 1 5BBF83FC
+P 1750 1000
+F 0 "#PWR07" H 1750 850 50  0001 C CNN
+F 1 "+5V" H 1750 1140 50  0000 C CNN
+F 2 "" H 1750 1000 50  0001 C CNN
+F 3 "" H 1750 1000 50  0001 C CNN
+	1    1750 1000
+	1    0    0    -1
+$EndComp
+$Comp
+L power:GND #PWR032
+U 1 1 5BBF854F
+P 1750 1400
+F 0 "#PWR032" H 1750 1150 50  0001 C CNN
+F 1 "GND" H 1750 1250 50  0000 C CNN
+F 2 "" H 1750 1400 50  0001 C CNN
+F 3 "" H 1750 1400 50  0001 C CNN
+	1    1750 1400
+	1    0    0    -1
+$EndComp
+Wire Wire Line
+	1750 1000 1750 1050
+Wire Wire Line
+	1750 1350 1750 1400
 $EndSCHEMATC

Commit message: updated pcb according to motherboard (EthernetTarget)
Connections:
- net labels added: +5VP
- wire segments 314 -> 327
- no-connect marks 20 -> 14
Changed lines of the file:
@@
 L power:+3.3V #PWR0101
 U 1 1 5BBCC540
-P 4850 700
-F 0 "#PWR0101" H 4850 550 50  0001 C CNN
-F 1 "+3.3V" H 4850 840 50  0000 C CNN
-F 2 "" H 4850 700 50  0001 C CNN
-F 3 "" H 4850 700 50  0001 C CNN
-	1    4850 700
+P 5000 700
+F 0 "#PWR0101" H 5000 550 50  0001 C CNN
+F 1 "+3.3V" H 5000 840 50  0000 C CNN
+F 2 "" H 5000 700 50  0001 C CNN
+F 3 "" H 5000 700 50  0001 C CNN
+	1    5000 700
 	1    0    0    -1
 $EndComp
-Wire Wire Line
-	4850 700  4850 750
-Wire Wire Line
-	4850 750  4800 750
 $Comp
 L power:+3.3VP #PWR0102
@@
 Wire Wire Line
 	4150 600  4300 600
-NoConn ~ 4800 950
-NoConn ~ 4800 1050
-NoConn ~ 4800 1150
-NoConn ~ 4800 1250
-NoConn ~ 4800 1350
-NoConn ~ 4800 1450
 NoConn ~ 4300 1450
 NoConn ~ 4300 1350
@@
 	2650 1500 2650 1250
 Connection ~ 2650 1250
-$Comp
-L power:GND #PWR033
-U 1 1 5BD9464F
-P 4200 1500
-F 0 "#PWR033" H 4200 1250 50  0001 C CNN
-F 1 "GND" H 4200 1350 50  0000 C CNN
-F 2 "" H 4200 1500 50  0001 C CNN
-F 3 "" H 4200 1500 50  0001 C CNN
-	1    4200 1500
-	1    0    0    -1
-$EndComp
-NoConn ~ 4800 850
-Wire Wire Line
-	4300 850  4200 850
-Wire Wire Line
-	4200 850  4200 1500
 $Comp
 L Device:CP C19
@@
 Wire Wire Line
 	1750 1350 1750 1400
+$Comp
+L power:GND #PWR?
+U 1 1 5BBFD925
+P 4900 1500
+F 0 "#PWR?" H 4900 1250 50  0001 C CNN
+F 1 "GND" H 4900 1350 50  0000 C CNN
+F 2 "" H 4900 1500 50  0001 C CNN
+F 3 "" H 4900 1500 50  0001 C CNN
+	1    4900 1500
+	1    0    0    -1
+$EndComp
+Wire Wire Line
+	4800 850  4900 850
+Wire Wire Line
+	4900 850  4900 1150
+Wire Wire Line
+	4800 1150 4900 1150
+Connection ~ 4900 1150
+Wire Wire Line
+	4900 1150 4900 1250
+Wire Wire Line
+	4800 1250 4900 1250
+Connection ~ 4900 1250
+Wire Wire Line
+	4900 1250 4900 1500
+Wire Wire Line
+	4800 750  4900 750
+Wire Wire Line
+	4900 750  4900 850
+Connection ~ 4900 850
+Wire Wire Line
+	4800 1350 5000 1350
+Wire Wire Line
+	5000 1350 5000 700
+Wire Wire Line
+	4800 1450 5000 1450
+Wire Wire Line
+	5000 1450 5000 1350
+Connection ~ 5000 1350
+NoConn ~ 4300 850
+$Comp
+L power:+5VP #PWR?
+U 1 1 5BCB023D
+P 5250 700
+F 0 "#PWR?" H 5250 550 50  0001 C CNN
+F 1 "+5VP" H 5250 850 50  0000 C CNN
+F 2 "" H 5250 700 50  0001 C CNN
+F 3 "" H 5250 700 50  0001 C CNN
+	1    5250 700
+	1    0    0    -1
+$EndComp
+Wire Wire Line
+	5250 700  5050 700
+Wire Wire Line
+	5050 700  5050 950
+Wire Wire Line
+	5050 950  4800 950
+Wire Wire Line
+	4800 1050 5050 1050
+Wire Wire Line
+	5050 1050 5050 950
+Connection ~ 5050 950
 $EndSCHEMATC

Commit message: Updated TrackModBusMaster_piggyback.sch and layout. completed component list to generate BOM.
Parts:
- added C20: 100n, Capacitor_SMD:C_1206_3216Metric, symbol Device:C
- added R27: 60E, Resistor_SMD:R_1206_3216Metric, symbol Device:R
- added R28: NP, Resistor_SMD:R_0603_1608Metric, symbol Device:R
- C1, C12, C18, C2, C3, C8, C9: value 2.2u -> 4.7u; Farnell (none) -> 2320886; Manufacturer nr (none) -> MC1206B475K250CT
- C10, C11, C13, C4, C5, C6, C7: Farnell (none) -> 1414715; Manufacturer nr (none) -> C1206C104K5RACTU
- C14, C15, C16, C17: Farnell (none) -> 2896606; Manufacturer nr (none) -> VJ1206A220JXACW1BC
- C19: value 100u -> 220u; Farnell (none) -> 2346568; Manufacturer nr (none) -> 16PX220MEFC6.3X11
- D1, D4, D5: Farnell (none) -> 2426215; Manufacturer nr (none) -> KPH-1608SGC
- D2: Farnell (none) -> 2426218; Manufacturer nr (none) -> KPH-1608YC
- D3: Farnell (none) -> 2426211; Manufacturer nr (none) -> KPH-1608EC
- Q1: value BVSS123LT1G -> NTR5103NT1G; Farnell (none) -> 2724423; Manufacturer nr (none) -> NTR5103NT1G
- R1, R10, R11, R13, R2, R3: value 1E -> 0E; Farnell (none) -> 1100137; Manufacturer nr (none) -> WCR1206-R005JI
- R12, R19, R20, R21, R26, R5: value 4k7 -> 4k99; Farnell (none) -> 2695161; Manufacturer nr (none) -> MCWR12X4991FTL
- R14, R15, R16, R17, R18: value 301E -> 300E; Farnell (none) -> 1100176; Manufacturer nr (none) -> WCR1206-300RFI
- R22: value 100k -> 110k; Farnell (none) -> 1100246; Manufacturer nr (none) -> WCR1206-110KFI
- R23, R6: Farnell (none) -> 1100218; Manufacturer nr (none) -> WCR1206-10KFI
- R24, R25: Farnell (none) -> 1100183; Manufacturer nr (none) -> WCR1206-470RFI
- R4: value 100E -> 1k; Farnell (none) -> 1100192; Manufacturer nr (none) -> WCR1206-1K0FI
- R7: value 3k9 -> 1k; Farnell (none) -> 1100192; Manufacturer nr (none) -> WCR1206-1K0FI
- R8: value 120E -> 60E; Farnell (none) -> 1100159; Manufacturer nr (none) -> WCR1206-62RFI
- R9: value 1k00 -> 1k; Farnell (none) -> 1100192; Manufacturer nr (none) -> WCR1206-1K0FI
- U1, U2, U3, U4, U5: Farnell (none) -> -; Manufacturer nr (none) -> ST485EBDR
- U6: value PIC16F18854-SO -> PIC18F25K40; Farnell (none) -> 2564200; Manufacturer nr (none) -> PIC18F25K40-I/SO
Connections:
- wire segments 327 -> 335

Commit message: Updated Led's of TrackModBusMaster_piggyback.
Parts:
- D1, D2, D3, D4, D5: footprint LED_SMD:LED_1206_3216Metric -> Diode_SMD:LED_0.8x0.8
Changed lines of the file:
@@
 F 0 "D1" H 7800 2350 50  0000 C CNN
 F 1 "LED GR" H 7550 2400 50  0000 C CNN
-F 2 "LED_SMD:LED_1206_3216Metric" H 8050 2400 50  0001 C CNN
+F 2 "Diode_SMD:LED_0.8x0.8" H 8050 2400 50  0001 C CNN
 F 3 "http://www.farnell.com/datasheets/2045940.pdf?_ga=2.245392706.792852979.1526285019-1651149783.1519657816" H 8050 2400 50  0001 C CNN
 F 4 "2426215" H 8050 2400 50  0001 C CNN "Farnell"
@@
 F 0 "D2" H 7800 2450 50  0000 C CNN
 F 1 "LED YE" H 7550 2500 50  0000 C CNN
-F 2 "LED_SMD:LED_1206_3216Metric" H 8050 2500 50  0001 C CNN
+F 2 "Diode_SMD:LED_0.8x0.8" H 8050 2500 50  0001 C CNN
 F 3 "http://www.farnell.com/datasheets/2046217.pdf?_ga=2.214478033.792852979.1526285019-1651149783.1519657816" H 8050 2500 50  0001 C CNN
 F 4 "2426218" H 8050 2500 50  0001 C CNN "Farnell"
@@
 F 0 "D3" H 7800 2550 50  0000 C CNN
 F 1 "LED RD" H 7550 2600 50  0000 C CNN
-F 2 "LED_SMD:LED_1206_3216Metric" H 8050 2600 50  0001 C CNN
+F 2 "Diode_SMD:LED_0.8x0.8" H 8050 2600 50  0001 C CNN
 F 3 "http://www.farnell.com/datasheets/2046367.pdf?_ga=2.218710495.792852979.1526285019-1651149783.1519657816" H 8050 2600 50  0001 C CNN
 F 4 "2426211" H 8050 2600 50  0001 C CNN "Farnell"
@@
 F 0 "D4" H 7800 2650 50  0000 C CNN
 F 1 "LED GR" H 7550 2700 50  0000 C CNN
-F 2 "LED_SMD:LED_1206_3216Metric" H 8050 2700 50  0001 C CNN
+F 2 "Diode_SMD:LED_0.8x0.8" H 8050 2700 50  0001 C CNN
 F 3 "http://www.farnell.com/datasheets/2045940.pdf?_ga=2.245392706.792852979.1526285019-1651149783.1519657816" H 8050 2700 50  0001 C CNN
 F 4 "2426215" H 8050 2700 50  0001 C CNN "Farnell"
@@
 F 0 "D5" H 7800 2750 50  0000 C CNN
 F 1 "LED GR" H 7550 2800 50  0000 C CNN
-F 2 "LED_SMD:LED_1206_3216Metric" H 8050 2800 50  0001 C CNN
+F 2 "Diode_SMD:LED_0.8x0.8" H 8050 2800 50  0001 C CNN
 F 3 "http://www.farnell.com/datasheets/2045940.pdf?_ga=2.245392706.792852979.1526285019-1651149783.1519657816" H 8050 2800 50  0001 C CNN
 F 4 "2426215" H 8050 2800 50  0001 C CNN "Farnell"
