File: KiCad/TrackModBusMaster_piggyback/TrackModBusMaster_piggyback.sch (KiCad schematic (older format))
At the start: 65 parts, among them J1 Conn_02x08_Top_Bottom, J2 Conn_02x05_Odd_Even, J3 Conn_02x08_Top_Bottom, J4 Conn_01x08, J5 Conn_01x08, Q1 NTR5103NT1G, U1 ST485EBDR, U2 ST485EBDR, U3 ST485EBDR, U4 ST485EBDR, U5 ST485EBDR, U6 PIC18F25K40

Commit message: Updated all schematics and layouts. Updated all component lists and csv files. Created ShopCartAll.csv from farnell big order for these 4 boards. Created new gerber files in the board-named directories to be send to PCB farmer.
Parts:
- C10, C11, C13, C20, C4, C5, C6, C7: Farnell 1414715 -> 2896646; Manufacturer nr C1206C104K5RACTU -> VJ1206Y104KXXPW1BC
- R28, U1, U2, U3, U4, U5: Farnell - -> (none)
Changed lines of the file:
@@
 F 2 "Capacitor_SMD:C_1206_3216Metric" H 6738 1300 50  0001 C CNN
 F 3 "http://www.farnell.com/datasheets/1901289.pdf?_ga=2.262491141.804204398.1540810031-466615820.1533907205&_gac=1.154756810.1540810031.CjwKCAjw39reBRBJEiwAO1m0OUdqKKSX6YgNsFqfn4kAD7vSQS5JfvsNobbwGFQV72towt0oHUutJhoC7b8QAvD_BwE" H 6700 1450 50  0001 C CNN
-F 4 "1414715" H 6700 1450 50  0001 C CNN "Farnell"
-F 5 "C1206C104K5RACTU" H 6700 1450 50  0001 C CNN "Manufacturer nr"
+F 4 "2896646" H 6700 1450 50  0001 C CNN "Farnell"
+F 5 "VJ1206Y104KXXPW1BC" H 6700 1450 50  0001 C CNN "Manufacturer nr"
 	1    6700 1450
 	1    0    0    -1
@@
 F 2 "Package_SO:SOIC-8_3.9x4.9mm_P1.27mm" H 1850 2700 50  0001 C CNN
 F 3 "http://www.st.com/resource/en/datasheet/st485eb.pdf" H 1850 3650 50  0001 C CNN
-F 4 "-" H 1850 3600 50  0001 C CNN "Farnell"
+F 4 "" H 1850 3600 50  0001 C CNN "Farnell"
 F 5 "ST485EBDR" H 1850 3600 50  0001 C CNN "Manufacturer nr"
 	1    1850 3600
@@
 F 2 "Resistor_SMD:R_0603_1608Metric" V 2680 3250 50  0001 C CNN
 F 3 "http://www.farnell.com/datasheets/2331353.pdf?_ga=2.229119068.13702668.1544197496-523844734.1542029203&_gac=1.216280482.1543322461.EAIaIQobChMIof7Tlcz03gIVkuJ3Ch1UVwqwEAAYASAAEgK8PvD_BwE" H 2750 3250 50  0001 C CNN
-F 4 "-" V 2750 3250 50  0001 C CNN "Farnell"
+F 4 "" V 2750 3250 50  0001 C CNN "Farnell"
 F 5 "-" V 2750 3250 50  0001 C CNN "Manufacturer nr"
 	1    2750 3250
@@
 F 2 "Capacitor_SMD:C_1206_3216Metric" H 3488 5300 50  0001 C CNN
 F 3 "http://www.farnell.com/datasheets/1901289.pdf?_ga=2.262491141.804204398.1540810031-466615820.1533907205&_gac=1.154756810.1540810031.CjwKCAjw39reBRBJEiwAO1m0OUdqKKSX6YgNsFqfn4kAD7vSQS5JfvsNobbwGFQV72towt0oHUutJhoC7b8QAvD_BwE" H 3450 5450 50  0001 C CNN
-F 4 "1414715" H 3450 5450 50  0001 C CNN "Farnell"
-F 5 "C1206C104K5RACTU" H 3450 5450 50  0001 C CNN "Manufacturer nr"
+F 4 "2896646" H 3450 5450 50  0001 C CNN "Farnell"
+F 5 "VJ1206Y104KXXPW1BC" H 3450 5450 50  0001 C CNN "Manufacturer nr"
 	1    3450 5450
 	1    0    0    -1
@@
 F 2 "Capacitor_SMD:C_1206_3216Metric" H 938 3450 50  0001 C CNN
 F 3 "http://www.farnell.com/datasheets/1901289.pdf?_ga=2.262491141.804204398.1540810031-466615820.1533907205&_gac=1.154756810.1540810031.CjwKCAjw39reBRBJEiwAO1m0OUdqKKSX6YgNsFqfn4kAD7vSQS5JfvsNobbwGFQV72towt0oHUutJhoC7b8QAvD_BwE" H 900 3600 50  0001 C CNN
-F 4 "1414715" H 900 3600 50  0001 C CNN "Farnell"
-F 5 "C1206C104K5RACTU" H 900 3600 50  0001 C CNN "Manufacturer nr"
+F 4 "2896646" H 900 3600 50  0001 C CNN "Farnell"
+F 5 "VJ1206Y104KXXPW1BC" H 900 3600 50  0001 C CNN "Manufacturer nr"
 	1    900  3600
 	1    0    0    -1
@@
 F 2 "Capacitor_SMD:C_1206_3216Metric" H 2988 3550 50  0001 C CNN
 F 3 "http://www.farnell.com/datasheets/1901289.pdf?_ga=2.262491141.804204398.1540810031-466615820.1533907205&_gac=1.154756810.1540810031.CjwKCAjw39reBRBJEiwAO1m0OUdqKKSX6YgNsFqfn4kAD7vSQS5JfvsNobbwGFQV72towt0oHUutJhoC7b8QAvD_BwE" H 2950 3700 50  0001 C CNN
-F 4 "1414715" H 2950 3700 50  0001 C CNN "Farnell"
-F 5 "C1206C104K5RACTU" H 2950 3700 50  0001 C CNN "Manufacturer nr"
+F 4 "2896646" H 2950 3700 50  0001 C CNN "Farnell"
+F 5 "VJ1206Y104KXXPW1BC" H 2950 3700 50  0001 C CNN "Manufacturer nr"
 	1    2950 3700
 	1    0    0    -1
@@
 F 2 "Capacitor_SMD:C_1206_3216Metric" H 938 4900 50  0001 C CNN
 F 3 "http://www.farnell.com/datasheets/1901289.pdf?_ga=2.262491141.804204398.1540810031-466615820.1533907205&_gac=1.154756810.1540810031.CjwKCAjw39reBRBJEiwAO1m0OUdqKKSX6YgNsFqfn4kAD7vSQS5JfvsNobbwGFQV72towt0oHUutJhoC7b8QAvD_BwE" H 900 5050 50  0001 C CNN
-F 4 "1414715" H 900 5050 50  0001 C CNN "Farnell"
-F 5 "C1206C104K5RACTU" H 900 5050 50  0001 C CNN "Manufacturer nr"
+F 4 "2896646" H 900 5050 50  0001 C CNN "Farnell"
+F 5 "VJ1206Y104KXXPW1BC" H 900 5050 50  0001 C CNN "Manufacturer nr"
 	1    900  5050
 	1    0    0    -1
@@
 F 2 "Capacitor_SMD:C_1206_3216Metric" H 938 6350 50  0001 C CNN
 F 3 "http://www.farnell.com/datasheets/1901289.pdf?_ga=2.262491141.804204398.1540810031-466615820.1533907205&_gac=1.154756810.1540810031.CjwKCAjw39reBRBJEiwAO1m0OUdqKKSX6YgNsFqfn4kAD7vSQS5JfvsNobbwGFQV72towt0oHUutJhoC7b8QAvD_BwE" H 900 6500 50  0001 C CNN
-F 4 "1414715" H 900 6500 50  0001 C CNN "Farnell"
-F 5 "C1206C104K5RACTU" H 900 6500 50  0001 C CNN "Manufacturer nr"
+F 4 "2896646" H 900 6500 50  0001 C CNN "Farnell"
+F 5 "VJ1206Y104KXXPW1BC" H 900 6500 50  0001 C CNN "Manufacturer nr"
 	1    900  6500
 	1    0    0    -1
@@
 F 2 "Capacitor_SMD:C_1206_3216Metric" H 4088 4900 50  0001 C CNN
 F 3 "http://www.farnell.com/datasheets/1901289.pdf?_ga=2.262491141.804204398.1540810031-466615820.1533907205&_gac=1.154756810.1540810031.CjwKCAjw39reBRBJEiwAO1m0OUdqKKSX6YgNsFqfn4kAD7vSQS5JfvsNobbwGFQV72towt0oHUutJhoC7b8QAvD_BwE" H 4050 5050 50  0001 C CNN
-F 4 "1414715" H 4050 5050 50  0001 C CNN "Farnell"
-F 5 "C1206C104K5RACTU" H 4050 5050 50  0001 C CNN "Manufacturer nr"
+F 4 "2896646" H 4050 5050 50  0001 C CNN "Farnell"
+F 5 "VJ1206Y104KXXPW1BC" H 4050 5050 50  0001 C CNN "Manufacturer nr"
 	1    4050 5050
 	1    0    0    -1
@@
 F 2 "Capacitor_SMD:C_1206_3216Metric" H 4088 6350 50  0001 C CNN
 F 3 "http://www.farnell.com/datasheets/1901289.pdf?_ga=2.262491141.804204398.1540810031-466615820.1533907205&_gac=1.154756810.1540810031.CjwKCAjw39reBRBJEiwAO1m0OUdqKKSX6YgNsFqfn4kAD7vSQS5JfvsNobbwGFQV72towt0oHUutJhoC7b8QAvD_BwE" H 4050 6500 50  0001 C CNN
-F 4 "1414715" H 4050 6500 50  0001 C CNN "Farnell"
-F 5 "C1206C104K5RACTU" H 4050 6500 50  0001 C CNN "Manufacturer nr"
+F 4 "2896646" H 4050 6500 50  0001 C CNN "Farnell"
+F 5 "VJ1206Y104KXXPW1BC" H 4050 6500 50  0001 C CNN "Manufacturer nr"
 	1    4050 6500
 	1    0    0    -1
@@
 F 2 "Package_SO:SOIC-8_3.9x4.9mm_P1.27mm" H 1850 4150 50  0001 C CNN
 F 3 "http://www.st.com/resource/en/datasheet/st485eb.pdf" H 1850 5100 50  0001 C CNN
-F 4 "-" H 1850 5050 50  0001 C CNN "Farnell"
+F 4 "" H 1850 5050 50  0001 C CNN "Farnell"
 F 5 "ST485EBDR" H 1850 5050 50  0001 C CNN "Manufacturer nr"
 	1    1850 5050
@@
 F 2 "Package_SO:SOIC-8_3.9x4.9mm_P1.27mm" H 1850 5600 50  0001 C CNN
 F 3 "http://www.st.com/resource/en/datasheet/st485eb.pdf" H 1850 6550 50  0001 C CNN
-F 4 "-" H 1850 6500 50  0001 C CNN "Farnell"
+F 4 "" H 1850 6500 50  0001 C CNN "Farnell"
 F 5 "ST485EBDR" H 1850 6500 50  0001 C CNN "Manufacturer nr"
 	1    1850 6500
@@
 F 2 "Package_SO:SOIC-8_3.9x4.9mm_P1.27mm" H 5000 4150 50  0001 C CNN
 F 3 "http://www.st.com/resource/en/datasheet/st485eb.pdf" H 5000 5100 50  0001 C CNN
-F 4 "-" H 5000 5050 50  0001 C CNN "Farnell"
+F 4 "" H 5000 5050 50  0001 C CNN "Farnell"
 F 5 "ST485EBDR" H 5000 5050 50  0001 C CNN "Manufacturer nr"
 	1    5000 5050
@@
 F 2 "Package_SO:SOIC-8_3.9x4.9mm_P1.27mm" H 5000 5600 50  0001 C CNN
 F 3 "http://www.st.com/resource/en/datasheet/st485eb.pdf" H 5000 6550 50  0001 C CNN
-F 4 "-" H 5000 6500 50  0001 C CNN "Farnell"
+F 4 "" H 5000 6500 50  0001 C CNN "Farnell"
 F 5 "ST485EBDR" H 5000 6500 50  0001 C CNN "Manufacturer nr"
 	1    5000 6500
@@
 Connection ~ 3450 5250
 $Comp
-L power:GND #PWR?
+L power:GND #PWR0103
 U 1 1 5C35772C
 P 3450 5650
-F 0 "#PWR?" H 3450 5400 50  0001 C CNN
+F 0 "#PWR0103" H 3450 5400 50  0001 C CNN
 F 1 "GND" H 3450 5500 50  0000 C CNN
 F 2 "" H 3450 5650 50  0001 C CNN
