File: KiCad/TrackModBusMaster_piggyback/TrackModBusMaster_piggyback.kicad_pcb (KiCad board)
At the start: 2 copper layers, 40 x 77 mm, 66 parts, among them J1 Conn_02x08_Top_Bottom, J2 Conn_02x05_Odd_Even, J3 Conn_02x08_Top_Bottom, J4 Conn_01x08, J5 Conn_01x08, Q1 NTR5103NT1G, U1 ST485EBDR, U2 ST485EBDR, U3 ST485EBDR, U4 ST485EBDR, U5 ST485EBDR, U6 PIC18F25K40

Commit message: some minor changes
Routing:
- net Rx: track 18.0 -> 16.9 mm
Changed lines of the file:
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@@
   (general
     (thickness 1.6)
-    (drawings 52)
-    (tracks 497)
+    (drawings 53)
+    (tracks 495)
     (zones 0)
     (modules 66)
@@
     (descr "CP, Radial series, Radial, pin pitch=2.50mm, , diameter=6.3mm, Electrolytic Capacitor")
     (tags "CP Radial series Radial pin pitch 2.50mm  diameter 6.3mm Electrolytic Capacitor")
-    (fp_text reference C19 (at -2 -3.292) (layer F.SilkS)
+    (fp_text reference C19 (at 4.7244 3.2512) (layer F.SilkS)
       (effects (font (size 1 1) (thickness 0.15)))
     )
@@
     )
   )
+  (gr_text . (at 134.5946 111.6076) (layer F.SilkS)
+    (effects (font (size 2 2) (thickness 0.5)))
+  )
   (gr_text 9 (at 133.858 98.806 90) (layer F.SilkS)
     (effects (font (size 2 2) (thickness 0.5)))
@@
     (effects (font (size 2 2) (thickness 0.5)))
   )
-  (gr_text . (at 135.128 42.418) (layer F.SilkS)
+  (gr_text . (at 134.62 42.7482) (layer F.SilkS)
     (effects (font (size 2 2) (thickness 0.5)))
   )
@@
     (effects (font (size 2 2) (thickness 0.5)))
   )
-  (gr_text . (at 129.159 68.326) (layer F.SilkS)
+  (gr_text . (at 129.1844 69.1642) (layer F.SilkS)
     (effects (font (size 2 2) (thickness 0.5)))
   )
@@
   (segment (start 117.348 67.186) (end 117.348 68.072) (width 0.5) (layer F.Cu) (net 47))
   (segment (start 117.348 68.072) (end 118.745 69.469) (width 0.5) (layer F.Cu) (net 47))
-  (segment (start 128.435 84.202) (end 128.436 84.201) (width 0.5) (layer F.Cu) (net 48))
-  (segment (start 127.635 84.202) (end 128.435 84.202) (width 0.5) (layer F.Cu) (net 48))
-  (segment (start 128.436 84.201) (end 129.159 84.201) (width 0.5) (layer F.Cu) (net 48))
-  (via (at 129.159 84.201) (size 0.8) (drill 0.4) (layers F.Cu B.Cu) (net 48))
-  (segment (start 129.159 84.201) (end 129.159 83.635315) (width 0.5) (layer B.Cu) (net 48))
-  (segment (start 129.159 83.635315) (end 129.159 72.644) (width 0.5) (layer B.Cu) (net 48))
-  (segment (start 129.159 72.644) (end 129.159 70.485) (width 0.5) (layer B.Cu) (net 48))
-  (segment (start 129.159 70.485) (end 128.651 69.977) (width 0.5) (layer B.Cu) (net 48))
-  (via (at 128.651 69.977) (size 0.8) (drill 0.4) (layers F.Cu B.Cu) (net 48))
-  (segment (start 128.651 69.977) (end 130.65 69.977) (width 0.5) (layer F.Cu) (net 48))
+  (via (at 128.9558 71.247) (size 0.8) (drill 0.4) (layers F.Cu B.Cu) (net 48))
+  (segment (start 128.9558 70.485) (end 128.9558 71.247) (width 0.5) (layer F.Cu) (net 48))
+  (segment (start 130.65 69.977) (end 129.4638 69.977) (width 0.5) (layer F.Cu) (net 48))
+  (segment (start 129.4638 69.977) (end 128.9558 70.485) (width 0.5) (layer F.Cu) (net 48))
+  (via (at 128.9558 84.1502) (size 0.8) (drill 0.4) (layers F.Cu B.Cu) (net 48))
+  (segment (start 128.9558 71.247) (end 128.9558 84.1502) (width 0.5) (layer B.Cu) (net 48))
+  (segment (start 127.635 84.202) (end 128.904 84.202) (width 0.5) (layer F.Cu) (net 48))
+  (segment (start 128.904 84.202) (end 128.9558 84.1502) (width 0.5) (layer F.Cu) (net 48))
   (segment (start 125.095 82.702) (end 125.095 84.202) (width 0.5) (layer F.Cu) (net 49))
   (segment (start 127.152 80.645) (end 125.095 82.702) (width 0.5) (layer F.Cu) (net 49))

Commit message: Final checks and updates, PCB's ordered.
Routing:
- net GND: track 253.7 -> 248.5 mm
Other:
- board text added: "<ICSP"
Changed lines of the file:
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@@
   (general
     (thickness 1.6)
-    (drawings 53)
+    (drawings 54)
     (tracks 495)
     (zones 0)
@@
   )
   (setup
-    (last_trace_width 0.25)
+    (last_trace_width 0.5)
     (user_trace_width 0.25)
     (user_trace_width 0.5)
@@
     (tags resistor)
     (attr smd)
-    (fp_text reference R10 (at 0 -1.778) (layer F.SilkS)
+    (fp_text reference R10 (at -3.048 0 90) (layer F.SilkS)
       (effects (font (size 1 1) (thickness 0.15)))
     )
@@
     (tags "SOIC 1.27")
     (attr smd)
-    (fp_text reference U2 (at 4.191 -3.429) (layer F.SilkS)
+    (fp_text reference U2 (at -3.048 3.302) (layer F.SilkS)
       (effects (font (size 1 1) (thickness 0.15)))
     )
@@
     (tags "SOIC 1.27")
     (attr smd)
-    (fp_text reference U3 (at 4.826 -1.905) (layer F.SilkS)
+    (fp_text reference U3 (at 0 3.556) (layer F.SilkS)
       (effects (font (size 1 1) (thickness 0.15)))
     )
@@
     (tags "SOIC 1.27")
     (attr smd)
-    (fp_text reference U5 (at 2.667 -3.429) (layer F.SilkS)
+    (fp_text reference U5 (at -0.127 3.429) (layer F.SilkS)
       (effects (font (size 1 1) (thickness 0.15)))
     )
@@
     )
   )
+  (gr_text <ICSP (at 106.68 108.458 90) (layer B.SilkS)
+    (effects (font (size 1.5 1.5) (thickness 0.3)) (justify mirror))
+  )
   (gr_text . (at 134.5946 111.6076) (layer F.SilkS)
     (effects (font (size 2 2) (thickness 0.5)))
@@
   (via (at 132.08 110.617) (size 0.8) (drill 0.4) (layers F.Cu B.Cu) (net 2))
   (segment (start 131.737 110.617) (end 132.08 110.617) (width 0.5) (layer F.Cu) (net 2))
-  (via (at 132.588 83.185) (size 0.8) (drill 0.4) (layers F.Cu B.Cu) (net 2))
-  (segment (start 137.569 83.185) (end 133.153685 83.185) (width 0.5) (layer F.Cu) (net 2))
-  (segment (start 133.153685 83.185) (end 132.588 83.185) (width 0.5) (layer F.Cu) (net 2))
-  (segment (start 140.109 80.645) (end 137.569 83.185) (width 0.5) (layer F.Cu) (net 2))
-  (segment (start 141.384 80.645) (end 140.109 80.645) (width 0.5) (layer F.Cu) (net 2))
   (via (at 115.824 103.886006) (size 0.8) (drill 0.4) (layers F.Cu B.Cu) (net 2))
   (segment (start 115.824 102.365) (end 115.824 103.886006) (width 0.5) (layer F.Cu) (net 2))
@@
   (segment (start 109.728 56.388) (end 107.188 56.388) (width 0.5) (layer F.Cu) (net 2))
   (segment (start 107.188 56.388) (end 106.172 56.388) (width 0.5) (layer F.Cu) (net 2))
+  (via (at 137.414 78.994) (size 0.8) (drill 0.4) (layers F.Cu B.Cu) (net 2))
+  (segment (start 141.384 80.645) (end 139.827 80.645) (width 0.5) (layer F.Cu) (net 2))
+  (segment (start 138.176 78.994) (end 137.414 78.994) (width 0.5) (layer F.Cu) (net 2))
+  (segment (start 139.827 80.645) (end 138.176 78.994) (width 0.5) (layer F.Cu) (net 2))
   (segment (start 135.512 65.126) (end 135.446 65.192) (width 0.5) (layer F.Cu) (net 3))
   (segment (start 135.512 62.738) (end 135.512 65.126) (width 0.5) (layer F.Cu) (net 3))
@@
   (segment (start 114.176 106.807) (end 116.172 106.807) (width 0.5) (layer F.Cu) (net 41))
   (segment (start 112.906 108.077) (end 114.176 106.807) (width 0.5) (layer F.Cu) (net 41))
-  (segment (start 133.093 79.375) (end 132.588 78.87) (width 0.5) (layer F.Cu) (net 42))
-  (segment (start 135.984 79.375) (end 133.093 79.375) (width 0.5) (layer F.Cu) (net 42))
   (segment (start 126.365 83.502) (end 127.913002 81.953998) (width 0.5) (layer F.Cu) (net 42))
   (segment (start 137.795 80.711) (end 136.459 79.375) (width 0.5) (layer F.Cu) (net 42))
@@
   (segment (start 126.365 84.202) (end 126.365 83.502) (width 0.5) (layer F.Cu) (net 42))
   (segment (start 127.913002 81.953998) (end 137.248002 81.953998) (width 0.5) (layer F.Cu) (net 42))
+  (segment (start 132.588 78.87) (end 133.988 78.87) (width 0.5) (layer F.Cu) (net 42))
+  (segment (start 134.493 79.375) (end 135.984 79.375) (width 0.5) (layer F.Cu) (net 42))
+  (segment (start 133.988 78.87) (end 134.493 79.375) (width 0.5) (layer F.Cu) (net 42))
   (segment (start 113.665 73.533) (end 113.665 74.802) (width 0.5) (layer F.Cu) (net 43))
   (segment (start 109.474 69.342) (end 113.665 73.533) (width 0.5) (layer F.Cu) (net 43))
