File: KiCad/ModeltrainWagonLight2/Modelwagonlight.sch (KiCad schematic (older format))
At the start: 17 parts, among them J1 Conn_01x01, J2 Conn_01x01, J3 Conn_01x01, J4 Conn_01x01, U1 LP2951DR

Commit message: Redrawn Modelwagonlight schematic and layout.
Parts:
- removed C1, C2: 22uF, Capacitors_THT:CP_Radial_D6.3mm_P2.50mm, symbol device:CP
- removed R6: NP, Resistors_SMD:R_1206, symbol device:R
- added C1, C2: 22u, Capacitor_SMD:C_1206_3216Metric, symbol device:C
- C3, C4: footprint Capacitors_SMD:C_1206 -> Capacitor_SMD:C_0603_1608Metric
- D1, D2: footprint Diodes_SMD:D_SOD-123 -> Diode_SMD:D_SOD-123
- R1: footprint Resistors_SMD:R_1206 -> Resistor_SMD:R_1206_3216Metric
- R4, R5: footprint Resistors_SMD:R_1206 -> Resistor_SMD:R_0603_1608Metric
- U1: footprint SMD_Packages:SOIC-8-N -> Package_SO:SOIC-8_3.9x4.9mm_P1.27mm
Connections:
- net labels added: GND
- wire segments 58 -> 56
Changed lines of the file:
@@
 F 0 "D1" H 5100 4050 50  0000 C CNN
 F 1 "STPS0540Z" H 5100 3850 50  0000 C CNN
-F 2 "Diodes_SMD:D_SOD-123" H 5100 3950 50  0001 C CNN
+F 2 "Diode_SMD:D_SOD-123" H 5100 3950 50  0001 C CNN
 F 3 "http://www.farnell.com/datasheets/2307147.pdf?_ga=2.156369662.418749504.1544431297-523844734.1542029203&_gac=1.55988569.1544607905.Cj0KCQiAgMPgBRDDARIsAOh3uyLPfvJVUZkf7WxE18rn4hxFId_d7BLsoZhKQT-s5UnN8AQpoENdC_QaAjuvEALw_wcB" H 5100 3950 50  0001 C CNN
 F 4 "1175677" H 5100 3950 50  0001 C CNN "Farnell"
@@
 F 0 "R1" V 4530 3950 50  0000 C CNN
 F 1 "47E" V 4450 3950 50  0000 C CNN
-F 2 "Resistors_SMD:R_1206" V 4380 3950 50  0001 C CNN
+F 2 "Resistor_SMD:R_1206_3216Metric" V 4380 3950 50  0001 C CNN
 F 3 "http://www.farnell.com/datasheets/2331353.pdf?_ga=2.124196682.13702668.1544197496-523844734.1542029203&_gac=1.140706310.1543322461.EAIaIQobChMIof7Tlcz03gIVkuJ3Ch1UVwqwEAAYASAAEgK8PvD_BwE" H 4450 3950 50  0001 C CNN
 F 4 "1100156" V 4450 3950 50  0001 C CNN "Farnell"
@@
 F 0 "R4" V 9130 4250 50  0000 C CNN
 F 1 "470E" V 9050 4250 50  0000 C CNN
-F 2 "Resistors_SMD:R_1206" V 8980 4250 50  0001 C CNN
+F 2 "Resistor_SMD:R_0603_1608Metric" V 8980 4250 50  0001 C CNN
 F 3 "http://www.farnell.com/datasheets/2331353.pdf?_ga=2.192410474.13702668.1544197496-523844734.1542029203&_gac=1.212666656.1543322461.EAIaIQobChMIof7Tlcz03gIVkuJ3Ch1UVwqwEAAYASAAEgK8PvD_BwE" H 9050 4250 50  0001 C CNN
 F 4 "1100183" V 9050 4250 50  0001 C CNN "Farnell"
@@
 F 0 "R5" V 9330 4250 50  0000 C CNN
 F 1 "NP" V 9250 4250 50  0000 C CNN
-F 2 "Resistors_SMD:R_1206" V 9180 4250 50  0001 C CNN
+F 2 "Resistor_SMD:R_0603_1608Metric" V 9180 4250 50  0001 C CNN
 F 3 "" H 9250 4250 50  0001 C CNN
 	1    9250 4250
 	-1   0    0    1
 $EndComp
-$Comp
-L device:R R6
-U 1 1 5ABB5D36
-P 9450 4250
-F 0 "R6" V 9530 4250 50  0000 C CNN
-F 1 "NP" V 9450 4250 50  0000 C CNN
-F 2 "Resistors_SMD:R_1206" V 9380 4250 50  0001 C CNN
-F 3 "" H 9450 4250 50  0001 C CNN
-	1    9450 4250
-	-1   0    0    1
-$EndComp
 Wire Wire Line
 	5600 3950 5600 4150
@@
 	5600 4650 5600 4450
 Connection ~ 5600 4650
-$Comp
-L device:CP C1
-U 1 1 5ABB8BA8
-P 5600 4300
-F 0 "C1" H 5625 4400 50  0000 L CNN
-F 1 "22uF" H 5625 4200 50  0000 L CNN
-F 2 "Capacitors_THT:CP_Radial_D6.3mm_P2.50mm" H 5638 4150 50  0001 C CNN
-F 3 "http://www.farnell.com/datasheets/1662440.pdf?_ga=2.122364238.418749504.1544431297-523844734.1542029203&_gac=1.125792376.1544607905.Cj0KCQiAgMPgBRDDARIsAOh3uyLPfvJVUZkf7WxE18rn4hxFId_d7BLsoZhKQT-s5UnN8AQpoENdC_QaAjuvEALw_wcB" H 5600 4300 50  0001 C CNN
-F 4 "9452397" H 5600 4300 50  0001 C CNN "Farnell"
-F 5 "MCUMHR35V226M6.3X5" H 5600 4300 50  0001 C CNN "Manufacturer nr"
-	1    5600 4300
-	1    0    0    -1
-$EndComp
 $Comp
 L Modelwagonlight-rescue:Conn_01x01 J1
@@
 F 0 "U1" H 7450 4550 60  0000 C CNN
 F 1 "LP2951DR" H 7450 4650 60  0000 C CNN
-F 2 "SMD_Packages:SOIC-8-N" H 7450 4250 60  0001 C CNN
+F 2 "Package_SO:SOIC-8_3.9x4.9mm_P1.27mm" H 7450 4250 60  0001 C CNN
 F 3 "http://www.ti.com/general/docs/lit/getliterature.tsp?genericPartNumber=LP2951&fileType=pdf" H 7450 4250 60  0001 C CNN
 F 4 "2781769" H 7450 4250 50  0001 C CNN "Farnell"
@@
 Connection ~ 9050 3900
 Wire Wire Line
-	9450 3900 9450 4100
-Connection ~ 9250 3900
-Wire Wire Line
 	8700 4650 8700 4400
 Connection ~ 6800 4650
@@
 	9250 4650 9250 4400
 Connection ~ 9050 4650
-Wire Wire Line
-	9450 4650 9450 4400
-Connection ~ 9250 4650
 Wire Wire Line
 	5250 3950 5300 3950
@@
 F 0 "C3" H 6475 4400 50  0000 L CNN
 F 1 "100n" H 6475 4200 50  0000 L CNN
-F 2 "Capacitors_SMD:C_1206" H 6488 4150 50  0001 C CNN
+F 2 "Capacitor_SMD:C_0603_1608Metric" H 6488 4150 50  0001 C CNN
 F 3 "http://www.farnell.com/datasheets/1901289.pdf?_ga=2.262491141.804204398.1540810031-466615820.1533907205&_gac=1.154756810.1540810031.CjwKCAjw39reBRBJEiwAO1m0OUdqKKSX6YgNsFqfn4kAD7vSQS5JfvsNobbwGFQV72towt0oHUutJhoC7b8QAvD_BwE" H 6450 4300 50  0001 C CNN
 F 4 "2896646" H 6450 4300 50  0001 C CNN "Farnell"
@@
 	9050 3900 9250 3900
 Wire Wire Line
-	9250 3900 9450 3900
-Wire Wire Line
 	6800 4650 8050 4650
 Wire Wire Line
@@
 	9050 4650 9250 4650
 Wire Wire Line
-	9250 4650 9450 4650
-Wire Wire Line
 	6800 4300 6800 4400
 Wire Wire Line
@@
 	6600 4100 6800 4100
 Wire Wire Line
-	6450 4650 6800 4650
-$Comp
-L device:CP C2
-U 1 1 5C10E3DF
-P 8700 4250
-F 0 "C2" H 8725 4350 50  0000 L CNN
-F 1 "22uF" H 8725 4150 50  0000 L CNN
-F 2 "Capacitors_THT:CP_Radial_D6.3mm_P2.50mm" H 8738 4100 50  0001 C CNN
-F 3 "http://www.farnell.com/datasheets/1662440.pdf?_ga=2.122364238.418749504.1544431297-523844734.1542029203&_gac=1.125792376.1544607905.Cj0KCQiAgMPgBRDDARIsAOh3uyLPfvJVUZkf7WxE18rn4hxFId_d7BLsoZhKQT-s5UnN8AQpoENdC_QaAjuvEALw_wcB" H 8700 4250 50  0001 C CNN
-F 4 "9452397" H 8700 4250 50  0001 C CNN "Farnell"
-F 5 "MCUMHR35V226M6.3X5" H 8700 4250 50  0001 C CNN "Manufacturer nr"
-	1    8700 4250
-	1    0    0    -1
-$EndComp
+	6450 4650 6700 4650
 $Comp
 L device:C C4
@@
 F 0 "C4" H 8425 4350 50  0000 L CNN
 F 1 "100n" H 8425 4150 50  0000 L CNN
-F 2 "Capacitors_SMD:C_1206" H 8438 4100 50  0001 C CNN
+F 2 "Capacitor_SMD:C_0603_1608Metric" H 8438 4100 50  0001 C CNN
 F 3 "http://www.farnell.com/datasheets/1901289.pdf?_ga=2.262491141.804204398.1540810031-466615820.1533907205&_gac=1.154756810.1540810031.CjwKCAjw39reBRBJEiwAO1m0OUdqKKSX6YgNsFqfn4kAD7vSQS5JfvsNobbwGFQV72towt0oHUutJhoC7b8QAvD_BwE" H 8400 4250 50  0001 C CNN
 F 4 "2896646" H 8400 4250 50  0001 C CNN "Farnell"
@@
 F 0 "D2" H 5100 4400 50  0000 C CNN
 F 1 "STPS0540Z" H 5100 4200 50  0000 C CNN
-F 2 "Diodes_SMD:D_SOD-123" H 5100 4300 50  0001 C CNN
+F 2 "Diode_SMD:D_SOD-123" H 5100 4300 50  0001 C CNN
 F 3 "http://www.farnell.com/datasheets/2307147.pdf?_ga=2.156369662.418749504.1544431297-523844734.1542029203&_gac=1.55988569.1544607905.Cj0KCQiAgMPgBRDDARIsAOh3uyLPfvJVUZkf7WxE18rn4hxFId_d7BLsoZhKQT-s5UnN8AQpoENdC_QaAjuvEALw_wcB" H 5100 4300 50  0001 C CNN
 F 4 "1175677" H 5100 4300 50  0001 C CNN "Farnell"
@@
 	1    0    0    -1
 $EndComp
+$Comp
+L device:C C1
+U 1 1 5C1828A9
+P 5600 4300
+F 0 "C1" H 5625 4400 50  0000 L CNN
+F 1 "22u" H 5625 4200 50  0000 L CNN
+F 2 "Capacitor_SMD:C_1206_3216Metric" H 5638 4150 50  0001 C CNN
+F 3 "http://www.farnell.com/datasheets/2079197.pdf?_ga=2.237228869.453305454.1544563035-1187106011.1538513614&_gac=1.262713726.1544645790.Cj0KCQiAgMPgBRDDARIsAOh3uyJWgmg4Jmz9qsKK7EVWh3ooL0QXFRR6pElfBGS6pZkWxoBnou2jGrYaAp9cEALw_wcB" H 5600 4300 50  0001 C CNN
+F 4 "2611953" H 5600 4300 50  0001 C CNN "Farnell"
+F 5 "GRM31CR61E226ME15L" H 5600 4300 50  0001 C CNN "Manufacturer nr"
+	1    5600 4300
+	1    0    0    -1
+$EndComp
+$Comp
+L device:C C2
+U 1 1 5C182A5F
+P 8700 4250
+F 0 "C2" H 8725 4350 50  0000 L CNN
+F 1 "22u" H 8725 4150 50  0000 L CNN
+F 2 "Capacitor_SMD:C_1206_3216Metric" H 8738 4100 50  0001 C CNN
+F 3 "http://www.farnell.com/datasheets/2079197.pdf?_ga=2.237228869.453305454.1544563035-1187106011.1538513614&_gac=1.262713726.1544645790.Cj0KCQiAgMPgBRDDARIsAOh3uyJWgmg4Jmz9qsKK7EVWh3ooL0QXFRR6pElfBGS6pZkWxoBnou2jGrYaAp9cEALw_wcB" H 8700 4250 50  0001 C CNN
+F 4 "2611953" H 8700 4250 50  0001 C CNN "Farnell"
+F 5 "GRM31CR61E226ME15L" H 8700 4250 50  0001 C CNN "Manufacturer nr"
+	1    8700 4250
+	1    0    0    -1
+$EndComp
+$Comp
+L power:GND #PWR?
+U 1 1 5C1839A0
+P 6700 4900
+F 0 "#PWR?" H 6700 4650 50  0001 C CNN
+F 1 "GND" H 6705 4727 50  0000 C CNN
+F 2 "" H 6700 4900 50  0001 C CNN
+F 3 "" H 6700 4900 50  0001 C CNN
+	1    6700 4900
+	1    0    0    -1
+$EndComp
+Wire Wire Line
+	6700 4900 6700 4650
+Connection ~ 6700 4650
+Wire Wire Line
+	6700 4650 6800 4650
 $EndSCHEMATC
